Commit message: add collision, inertial and joint dynamics

File: universal_robot_description/urdf/robot.urdf.xacro (robot description, xacro)
@@ -4,9 +4,13 @@
   <property name="shoulder_height" value="0.1" />
   <property name="shoulder_offset" value="0.1" />
+  <property name="shoulder_radius" value="0.1" />
   <property name="upper_arm_length" value="0.5" />
+  <property name="upper_arm_radius" value="0.05" />
   <property name="forearm_length" value="0.5" />
+  <property name="forearm_radius" value="0.03" />
   <property name="wrist_1_length" value="0.1" />
   <property name="wrist_2_length" value="0.1" />
   <property name="wrist_3_length" value="0.1" />
+  <property name="wrist_radius" value="0.03" />
   <link name="base_link" />
   <joint name="shoulder_pan_joint" type="revolute">
@@ -16,12 +20,23 @@
     <axis xyz="0.0 0.0 1.0" />
     <limit lower="-${pi}" upper="${pi}" effort="10.0" velocity="1.0"/>
+    <dynamics damping="0.1" friction="0.1"/>
   </joint>
   <link name="shoulder_link">
     <visual>
       <geometry>
-        <cylinder length="${shoulder_height}" radius="0.1"/>
+        <cylinder length="${shoulder_height}" radius="${shoulder_radius}"/>
       </geometry>
       <origin xyz="0.0 0.0 ${-shoulder_height/2.0}" rpy="0.0 0.0 0.0" />
     </visual>
+    <collision>
+      <geometry>
+        <cylinder length="${shoulder_height}" radius="${shoulder_radius}"/>
+      </geometry>
+      <origin xyz="0.0 0.0 ${-shoulder_height/2.0}" rpy="0.0 0.0 0.0" />
+    </collision>
+    <inertial>
+      <mass value="10" />
+      <inertia ixx="1.0" ixy="0.0" ixz="0.0" iyy="1.0" iyz="0.0" izz="1.0"/>
+    </inertial>
   </link>
   <joint name="shoulder_lift_joint" type="revolute">
@@ -31,12 +46,23 @@
     <axis xyz="0.0 1.0 0.0" />
     <limit lower="-${pi}" upper="${pi}" effort="10.0" velocity="1.0"/>
+    <dynamics damping="0.1" friction="0.1"/>
   </joint>
   <link name="upper_arm_link">
     <visual>
       <geometry>
-        <cylinder length="${upper_arm_length}" radius="0.05"/>
+        <cylinder length="${upper_arm_length}" radius="${upper_arm_radius}"/>
       </geometry>
       <origin xyz="0.0 0.0 ${upper_arm_length/2.0}" rpy="0.0 0.0 0.0" />
     </visual>
+    <collision>
+      <geometry>
+        <cylinder length="${upper_arm_length}" radius="${upper_arm_radius}"/>
+      </geometry>
+      <origin xyz="0.0 0.0 ${upper_arm_length/2.0}" rpy="0.0 0.0 0.0" />
+    </collision>
+    <inertial>
+      <mass value="10" />
+      <inertia ixx="1.0" ixy="0.0" ixz="0.0" iyy="1.0" iyz="0.0" izz="1.0"/>
+    </inertial>
   </link>
   <joint name="elbow_joint" type="revolute">
@@ -46,12 +72,23 @@
     <axis xyz="0.0 -1.0 0.0" />
     <limit lower="-${pi}" upper="${pi}" effort="10.0" velocity="1.0"/>
+    <dynamics damping="0.1" friction="0.1"/>
   </joint>
   <link name="forearm_link">
     <visual>
       <geometry>
-        <cylinder length="${forearm_length}" radius="0.05"/>
+        <cylinder length="${forearm_length}" radius="${forearm_radius}"/>
       </geometry>
       <origin xyz="0.0 0.0 ${forearm_length/2.0}" rpy="0.0 0.0 0.0" />
     </visual>
+    <collision>
+      <geometry>
+        <cylinder length="${forearm_length}" radius="${forearm_radius}"/>
+      </geometry>
+      <origin xyz="0.0 0.0 ${forearm_length/2.0}" rpy="0.0 0.0 0.0" />
+    </collision>
+    <inertial>
+      <mass value="10" />
+      <inertia ixx="1.0" ixy="0.0" ixz="0.0" iyy="1.0" iyz="0.0" izz="1.0"/>
+    </inertial>
   </link>
   <joint name="wrist_1_joint" type="revolute">
@@ -61,12 +98,23 @@
     <axis xyz="0.0 1.0 0.0" />
     <limit lower="-${pi}" upper="${pi}" effort="10.0" velocity="1.0"/>
+    <dynamics damping="0.1" friction="0.1"/>
   </joint>
   <link name="wrist_1_link">
     <visual>
       <geometry>
-        <cylinder length="${wrist_1_length}" radius="0.05"/>
+        <cylinder length="${wrist_1_length}" radius="${wrist_radius}"/>
       </geometry>
       <origin xyz="0.0 ${wrist_1_length/2.0} 0.0" rpy="-${pi/2.0} 0.0 0.0" />
     </visual>
+    <collision>
+      <geometry>
+        <cylinder length="${wrist_1_length}" radius="${wrist_radius}"/>
+      </geometry>
+      <origin xyz="0.0 ${wrist_1_length/2.0} 0.0" rpy="-${pi/2.0} 0.0 0.0" />
+    </collision>
+    <inertial>
+      <mass value="10" />
+      <inertia ixx="1.0" ixy="0.0" ixz="0.0" iyy="1.0" iyz="0.0" izz="1.0"/>
+    </inertial>
   </link>
   <joint name="wrist_2_joint" type="revolute">
@@ -76,12 +124,23 @@
     <axis xyz="0.0 0.0 1.0" />
     <limit lower="-${pi}" upper="${pi}" effort="10.0" velocity="1.0"/>
+    <dynamics damping="0.1" friction="0.1"/>
   </joint>
   <link name="wrist_2_link">
     <visual>
       <geometry>
-        <cylinder length="${wrist_2_length}" radius="0.05"/>
+        <cylinder length="${wrist_2_length}" radius="${wrist_radius}"/>
       </geometry>
       <origin xyz="0.0 0.0 ${wrist_2_length/2.0}" rpy="0.0 0.0 0.0" />
     </visual>
+    <collision>
+      <geometry>
+        <cylinder length="${wrist_2_length}" radius="${wrist_radius}"/>
+      </geometry>
+      <origin xyz="0.0 0.0 ${wrist_2_length/2.0}" rpy="0.0 0.0 0.0" />
+    </collision>
+    <inertial>
+      <mass value="10" />
+      <inertia ixx="1.0" ixy="0.0" ixz="0.0" iyy="1.0" iyz="0.0" izz="1.0"/>
+    </inertial>
   </link>
   <joint name="wrist_3_joint" type="revolute">
@@ -91,12 +150,23 @@
     <axis xyz="0.0 1.0 0.0" />
     <limit lower="-${pi}" upper="${pi}" effort="10.0" velocity="1.0"/>
+    <dynamics damping="0.1" friction="0.1"/>
   </joint>
   <link name="wrist_3_link">
     <visual>
       <geometry>
-        <cylinder length="${wrist_3_length}" radius="0.05"/>
+        <cylinder length="${wrist_3_length}" radius="${wrist_radius}"/>
       </geometry>
       <origin xyz="0.0 ${wrist_3_length/2.0} 0.0" rpy="${-pi/2.0} 0.0 0.0" />
     </visual>
+    <collision>
+      <geometry>
+        <cylinder length="${wrist_3_length}" radius="${wrist_radius}"/>
+      </geometry>
+      <origin xyz="0.0 ${wrist_3_length/2.0} 0.0" rpy="${-pi/2.0} 0.0 0.0" />
+    </collision>
+    <inertial>
+      <mass value="10" />
+      <inertia ixx="1.0" ixy="0.0" ixz="0.0" iyy="1.0" iyz="0.0" izz="1.0"/>
+    </inertial>
   </link>
   <joint name="ee_fixed_joint" type="fixed">
@@ -112,4 +182,14 @@
       <origin xyz="0.0 0.0 0.0" rpy="0.0 ${-pi/2.0} 0.0" />
     </visual>
+    <collision>
+      <geometry>
+        <cylinder length="0.01" radius="0.06"/>
+      </geometry>
+      <origin xyz="0.0 0.0 0.0" rpy="0.0 ${-pi/2.0} 0.0" />
+    </collision>
+    <inertial>
+      <mass value="10" />
+      <inertia ixx="1.0" ixy="0.0" ixz="0.0" iyy="1.0" iyz="0.0" izz="1.0"/>
+    </inertial>
   </link>
 </robot>

Commit message: can be loaded in gazebo

File: universal_robot_description/urdf/robot.urdf.xacro (robot description, xacro)
@@ -13,5 +13,10 @@
   <property name="wrist_3_length" value="0.1" />
   <property name="wrist_radius" value="0.03" />
-  <link name="base_link" />
+  <link name="base_link" >
+    <inertial>
+      <mass value="10" />
+      <inertia ixx="1.0" ixy="0.0" ixz="0.0" iyy="1.0" iyz="0.0" izz="1.0"/>
+    </inertial>
+  </link>
   <joint name="shoulder_pan_joint" type="revolute">
     <parent link="base_link" />
@@ -193,3 +198,6 @@
     </inertial>
   </link>
+  <gazebo reference="universal_robot">
+    <material>Gazebo/Blue</material>
+  </gazebo>
 </robot>

Commit message: Add correct dimensions to urdf

File: universal_robot_description/urdf/robot.urdf.xacro (robot description, xacro)
@@ -1,15 +1,37 @@
 <?xml version="1.0"?>
+<!--
+DH for UR5:
+a = [0.00000, -0.42500, -0.39225,  0.00000,  0.00000,  0.0000]
+d = [0.089159,  0.00000,  0.00000,  0.10915,  0.09465,  0.0823]
+alpha = [ 1.570796327, 0, 0, 1.570796327, -1.570796327, 0 ]
+q_home_offset = [0, -1.570796327, 0, -1.570796327, 0, 0]
+joint_direction = [-1, -1, 1, 1, 1, 1]
+mass = [3.7000, 8.3930, 2.2750, 1.2190, 1.2190, 0.1879]
+center_of_mass = [ [0, -0.02561, 0.00193], [0.2125, 0, 0.11336], [0.11993, 0.0, 0.0265], [0, -0.0018, 0.01634], [0, 0.0018,0.01634], [0, 0, -0.001159] ]
+-->
 <robot name="universal_robot">
-  <property name="pi" value="3.14" />
+  <property name="pi" value="3.14159265" />
+  <property name="shoulder_mass" value="3.7000" />
+  <property name="upper_arm_mass" value="8.3930" />
+  <property name="forearm_mass" value="2.2750" />
+  <property name="wrist_1_mass" value="1.2190" />
+  <property name="wrist_2_mass" value="1.2190" />
+  <property name="wrist_3_mass" value="0.1879" />
+  <property name="shoulder_cog" value="0.0 0.00193 -0.02561" />
+  <property name="upper_arm_cog" value="0.0 -0.024201 0.2125" /> <!-- 0.11336 - 0.089159 =  -->
+  <property name="forearm_cog" value="0.0 0.0265 0.11993" /> <!-- 0.119 is not half of 0.39225 ?? -->
+  <property name="wrist_1_cog" value="0.0 0.110949 0.01634" /> <!-- 0.0018 + 0.10915 = 0.110949 -->
+  <property name="wrist_2_cog" value="0.0 0.0018 0.11099" />  <!-- 0.01634 + 0.09465 = 0.11099-->
+  <property name="wrist_3_cog" value="0.0 0.001159 0.0" />
   <property name="shoulder_height" value="0.1" />
-  <property name="shoulder_offset" value="0.1" />
+  <property name="shoulder_offset" value="0.089159" />
+  <property name="upper_arm_length" value="0.42500" />
+  <property name="forearm_length" value="0.39225" />
+  <property name="wrist_1_length" value="0.10915" />
+  <property name="wrist_2_length" value="0.09465" />
+  <property name="wrist_3_length" value="0.0823" />
   <property name="shoulder_radius" value="0.1" />
-  <property name="upper_arm_length" value="0.5" />
   <property name="upper_arm_radius" value="0.05" />
-  <property name="forearm_length" value="0.5" />
   <property name="forearm_radius" value="0.03" />
-  <property name="wrist_1_length" value="0.1" />
-  <property name="wrist_2_length" value="0.1" />
-  <property name="wrist_3_length" value="0.1" />
   <property name="wrist_radius" value="0.03" />
   <link name="base_link" >
@@ -41,6 +63,7 @@
     </collision>
     <inertial>
-      <mass value="10" />
-      <inertia ixx="1.0" ixy="0.0" ixz="0.0" iyy="1.0" iyz="0.0" izz="1.0"/>
+      <mass value="${shoulder_mass}" />
+      <inertia ixx="1.0" ixy="0.0" ixz="0.0" iyy="1.0" iyz="0.0" izz="1.0"/>
+      <origin xyz="${shoulder_cog}" rpy="0.0 0.0 0.0" />
     </inertial>
   </link>
@@ -67,6 +90,7 @@
     </collision>
     <inertial>
-      <mass value="10" />
-      <inertia ixx="1.0" ixy="0.0" ixz="0.0" iyy="1.0" iyz="0.0" izz="1.0"/>
+      <mass value="${upper_arm_mass}" />
+      <inertia ixx="1.0" ixy="0.0" ixz="0.0" iyy="1.0" iyz="0.0" izz="1.0"/>
+      <origin xyz="${upper_arm_cog}" rpy="0.0 0.0 0.0" />
     </inertial>
   </link>
@@ -93,5 +117,6 @@
     </collision>
     <inertial>
-      <mass value="10" />
+      <mass value="${forearm_mass}" />
+      <origin xyz="${forearm_cog}" rpy="0.0 0.0 0.0" />
       <inertia ixx="1.0" ixy="0.0" ixz="0.0" iyy="1.0" iyz="0.0" izz="1.0"/>
     </inertial>
@@ -119,5 +144,6 @@
     </collision>
     <inertial>
-      <mass value="10" />
+      <mass value="${wrist_1_mass}" />
+      <origin xyz="${wrist_1_cog}" rpy="0.0 0.0 0.0" />
       <inertia ixx="1.0" ixy="0.0" ixz="0.0" iyy="1.0" iyz="0.0" izz="1.0"/>
     </inertial>
@@ -145,5 +171,6 @@
     </collision>
     <inertial>
-      <mass value="10" />
+      <mass value="${wrist_2_mass}" />
+      <origin xyz="${wrist_2_cog}" rpy="0.0 0.0 0.0" />
       <inertia ixx="1.0" ixy="0.0" ixz="0.0" iyy="1.0" iyz="0.0" izz="1.0"/>
     </inertial>
@@ -171,5 +198,6 @@
     </collision>
     <inertial>
-      <mass value="10" />
+      <mass value="${wrist_3_mass}" />
+      <origin xyz="${wrist_3_cog}" rpy="0.0 0.0 0.0" />
       <inertia ixx="1.0" ixy="0.0" ixz="0.0" iyy="1.0" iyz="0.0" izz="1.0"/>
     </inertial>
@@ -193,8 +221,4 @@
       <origin xyz="0.0 0.0 0.0" rpy="0.0 ${-pi/2.0} 0.0" />
     </collision>
-    <inertial>
-      <mass value="10" />
-      <inertia ixx="1.0" ixy="0.0" ixz="0.0" iyy="1.0" iyz="0.0" izz="1.0"/>
-    </inertial>
   </link>
   <gazebo reference="universal_robot">

Commit message: no more magic numbers

File: universal_robot_description/urdf/robot.urdf.xacro (robot description, xacro)
@@ -12,4 +12,5 @@
 <robot name="universal_robot">
   <property name="pi" value="3.14159265" />
+  <property name="base_mass" value="10.0" /> <!-- not form spec -->
   <property name="shoulder_mass" value="3.7000" />
   <property name="upper_arm_mass" value="8.3930" />
@@ -24,5 +25,5 @@
   <property name="wrist_2_cog" value="0.0 0.0018 0.11099" />  <!-- 0.01634 + 0.09465 = 0.11099-->
   <property name="wrist_3_cog" value="0.0 0.001159 0.0" />
-  <property name="shoulder_height" value="0.1" />
+  <property name="shoulder_height" value="0.1" />  <!-- not form spec -->
   <property name="shoulder_offset" value="0.089159" />
   <property name="upper_arm_length" value="0.42500" />
@@ -31,11 +32,11 @@
   <property name="wrist_2_length" value="0.09465" />
   <property name="wrist_3_length" value="0.0823" />
-  <property name="shoulder_radius" value="0.1" />
-  <property name="upper_arm_radius" value="0.05" />
-  <property name="forearm_radius" value="0.03" />
-  <property name="wrist_radius" value="0.03" />
+  <property name="shoulder_radius" value="0.1" />  <!-- not form spec -->
+  <property name="upper_arm_radius" value="0.05" />  <!-- not form spec -->
+  <property name="forearm_radius" value="0.03" />  <!-- not form spec -->
+  <property name="wrist_radius" value="0.03" />  <!-- not form spec -->
   <link name="base_link" >
     <inertial>
-      <mass value="10" />
+      <mass value="${base_mass}" />
       <inertia ixx="1.0" ixy="0.0" ixz="0.0" iyy="1.0" iyz="0.0" izz="1.0"/>
     </inertial>
@@ -211,5 +212,5 @@
     <visual>
       <geometry>
-        <cylinder length="0.01" radius="0.06"/>
+        <cylinder length="0.01" radius="${wrist_radius * 1.25}"/>
       </geometry>
       <origin xyz="0.0 0.0 0.0" rpy="0.0 ${-pi/2.0} 0.0" />
@@ -217,5 +218,5 @@
     <collision>
       <geometry>
-        <cylinder length="0.01" radius="0.06"/>
+        <cylinder length="0.01" radius="${wrist_radius * 1.25}"/>
       </geometry>
       <origin xyz="0.0 0.0 0.0" rpy="0.0 ${-pi/2.0} 0.0" />

Commit message: put in correct joint offsets and joint directions

File: universal_robot_description/urdf/robot.urdf.xacro (robot description, xacro)
@@ -72,5 +72,5 @@
     <parent link="shoulder_link" />
     <child link = "upper_arm_link" />
-    <origin xyz="0.0 ${shoulder_offset} 0.0" rpy="0.0 0.0 0.0" />
+    <origin xyz="0.0 ${shoulder_offset} 0.0" rpy="0.0 ${pi / 2.0} 0.0" />
     <axis xyz="0.0 1.0 0.0" />
     <limit lower="-${pi}" upper="${pi}" effort="10.0" velocity="1.0"/>
@@ -100,5 +100,5 @@
     <child link = "forearm_link" />
     <origin xyz="0.0 ${-shoulder_offset} ${upper_arm_length}" rpy="0.0 0.0 0.0" />
-    <axis xyz="0.0 -1.0 0.0" />
+    <axis xyz="0.0 1.0 0.0" />
     <limit lower="-${pi}" upper="${pi}" effort="10.0" velocity="1.0"/>
     <dynamics damping="0.1" friction="0.1"/>
@@ -126,5 +126,5 @@
     <parent link="forearm_link" />
     <child link = "wrist_1_link" />
-    <origin xyz="0.0 0.0 ${forearm_length}" rpy="0.0 0.0 0.0" />
+    <origin xyz="0.0 0.0 ${forearm_length}" rpy="0.0 ${pi / 2.0} 0.0" />
     <axis xyz="0.0 1.0 0.0" />
     <limit lower="-${pi}" upper="${pi}" effort="10.0" velocity="1.0"/>

Commit message: update joint limits

File: universal_robot_description/urdf/robot.urdf.xacro (robot description, xacro)
@@ -47,5 +47,5 @@
     <origin xyz="0.0 0.0 ${shoulder_height}" rpy="0.0 0.0 0.0" />
     <axis xyz="0.0 0.0 1.0" />
-    <limit lower="-${pi}" upper="${pi}" effort="10.0" velocity="1.0"/>
+    <limit lower="${-2.0 * pi}" upper="${2.0 * pi}" effort="10.0" velocity="1.0"/>
     <dynamics damping="0.1" friction="0.1"/>
   </joint>
@@ -74,5 +74,5 @@
     <origin xyz="0.0 ${shoulder_offset} 0.0" rpy="0.0 ${pi / 2.0} 0.0" />
     <axis xyz="0.0 1.0 0.0" />
-    <limit lower="-${pi}" upper="${pi}" effort="10.0" velocity="1.0"/>
+    <limit lower="${-2.0 * pi}" upper="${2.0 * pi}" effort="10.0" velocity="1.0"/>
     <dynamics damping="0.1" friction="0.1"/>
   </joint>
@@ -101,5 +101,5 @@
     <origin xyz="0.0 ${-shoulder_offset} ${upper_arm_length}" rpy="0.0 0.0 0.0" />
     <axis xyz="0.0 1.0 0.0" />
-    <limit lower="-${pi}" upper="${pi}" effort="10.0" velocity="1.0"/>
+    <limit lower="${-2.0 * pi}" upper="${2.0 * pi}" effort="10.0" velocity="1.0"/>
     <dynamics damping="0.1" friction="0.1"/>
   </joint>
@@ -128,5 +128,5 @@
     <origin xyz="0.0 0.0 ${forearm_length}" rpy="0.0 ${pi / 2.0} 0.0" />
     <axis xyz="0.0 1.0 0.0" />
-    <limit lower="-${pi}" upper="${pi}" effort="10.0" velocity="1.0"/>
+    <limit lower="${-2.0 * pi}" upper="${2.0 * pi}" effort="10.0" velocity="1.0"/>
     <dynamics damping="0.1" friction="0.1"/>
   </joint>
@@ -136,5 +136,5 @@
         <cylinder length="${wrist_1_length}" radius="${wrist_radius}"/>
       </geometry>
-      <origin xyz="0.0 ${wrist_1_length/2.0} 0.0" rpy="-${pi/2.0} 0.0 0.0" />
+      <origin xyz="0.0 ${wrist_1_length/2.0} 0.0" rpy="${-pi/2.0} 0.0 0.0" />
     </visual>
     <collision>
@@ -142,5 +142,5 @@
         <cylinder length="${wrist_1_length}" radius="${wrist_radius}"/>
       </geometry>
-      <origin xyz="0.0 ${wrist_1_length/2.0} 0.0" rpy="-${pi/2.0} 0.0 0.0" />
+      <origin xyz="0.0 ${wrist_1_length/2.0} 0.0" rpy="${-pi/2.0} 0.0 0.0" />
     </collision>
     <inertial>
@@ -155,5 +155,5 @@
     <origin xyz="0.0 ${wrist_1_length} 0.0" rpy="0.0 0.0 0.0" />
     <axis xyz="0.0 0.0 1.0" />
-    <limit lower="-${pi}" upper="${pi}" effort="10.0" velocity="1.0"/>
+    <limit lower="${-2.0 * pi}" upper="${2.0 * pi}" effort="10.0" velocity="1.0"/>
     <dynamics damping="0.1" friction="0.1"/>
   </joint>
@@ -182,5 +182,5 @@
     <origin xyz="0.0 0.0 ${wrist_3_length}" rpy="0.0 0.0 0.0" />
     <axis xyz="0.0 1.0 0.0" />
-    <limit lower="-${pi}" upper="${pi}" effort="10.0" velocity="1.0"/>
+    <limit lower="${-2.0 * pi}" upper="${2.0 * pi}" effort="10.0" velocity="1.0"/>
     <dynamics damping="0.1" friction="0.1"/>
   </joint>

Commit message: update joint velocity limits

File: universal_robot_description/urdf/robot.urdf.xacro (robot description, xacro)
@@ -47,5 +47,5 @@
     <origin xyz="0.0 0.0 ${shoulder_height}" rpy="0.0 0.0 0.0" />
     <axis xyz="0.0 0.0 1.0" />
-    <limit lower="${-2.0 * pi}" upper="${2.0 * pi}" effort="10.0" velocity="1.0"/>
+    <limit lower="${-2.0 * pi}" upper="${2.0 * pi}" effort="10.0" velocity="${pi}"/>
     <dynamics damping="0.1" friction="0.1"/>
   </joint>
@@ -74,5 +74,5 @@
     <origin xyz="0.0 ${shoulder_offset} 0.0" rpy="0.0 ${pi / 2.0} 0.0" />
     <axis xyz="0.0 1.0 0.0" />
-    <limit lower="${-2.0 * pi}" upper="${2.0 * pi}" effort="10.0" velocity="1.0"/>
+    <limit lower="${-2.0 * pi}" upper="${2.0 * pi}" effort="10.0" velocity="${pi}"/>
     <dynamics damping="0.1" friction="0.1"/>
   </joint>
@@ -101,5 +101,5 @@
     <origin xyz="0.0 ${-shoulder_offset} ${upper_arm_length}" rpy="0.0 0.0 0.0" />
     <axis xyz="0.0 1.0 0.0" />
-    <limit lower="${-2.0 * pi}" upper="${2.0 * pi}" effort="10.0" velocity="1.0"/>
+    <limit lower="${-2.0 * pi}" upper="${2.0 * pi}" effort="10.0" velocity="${pi}"/>
     <dynamics damping="0.1" friction="0.1"/>
   </joint>
@@ -128,5 +128,5 @@
     <origin xyz="0.0 0.0 ${forearm_length}" rpy="0.0 ${pi / 2.0} 0.0" />
     <axis xyz="0.0 1.0 0.0" />
-    <limit lower="${-2.0 * pi}" upper="${2.0 * pi}" effort="10.0" velocity="1.0"/>
+    <limit lower="${-2.0 * pi}" upper="${2.0 * pi}" effort="10.0" velocity="${pi}"/>
     <dynamics damping="0.1" friction="0.1"/>
   </joint>
@@ -155,5 +155,5 @@
     <origin xyz="0.0 ${wrist_1_length} 0.0" rpy="0.0 0.0 0.0" />
     <axis xyz="0.0 0.0 1.0" />
-    <limit lower="${-2.0 * pi}" upper="${2.0 * pi}" effort="10.0" velocity="1.0"/>
+    <limit lower="${-2.0 * pi}" upper="${2.0 * pi}" effort="10.0" velocity="${pi}"/>
     <dynamics damping="0.1" friction="0.1"/>
   </joint>
@@ -182,5 +182,5 @@
     <origin xyz="0.0 0.0 ${wrist_3_length}" rpy="0.0 0.0 0.0" />
     <axis xyz="0.0 1.0 0.0" />
-    <limit lower="${-2.0 * pi}" upper="${2.0 * pi}" effort="10.0" velocity="1.0"/>
+    <limit lower="${-2.0 * pi}" upper="${2.0 * pi}" effort="10.0" velocity="${pi}"/>
     <dynamics damping="0.1" friction="0.1"/>
   </joint>
