Commit message: rename package to ur5

File: ur5_description/urdf/robot.urdf.xacro (robot description, xacro)
@@ -87,5 +87,5 @@
     <visual>
       <geometry>
-       <mesh filename="package://universal_robot_description/meshes/UpperArm.dae" />
+       <mesh filename="package://ur5_description/meshes/UpperArm.dae" />
       </geometry>
       <origin xyz="0.0 0.0 0.0" rpy="0.0 0.0 0.0" />

Commit message: added all meshes and completed collision model

File: ur5_description/urdf/robot.urdf.xacro (robot description, xacro)
@@ -28,16 +28,16 @@
 <!-- Kinematic model -->
   <property name="shoulder_height" value="0.089159" />
-  <property name="shoulder_offset" value="0.13915" />  <!-- shoulder_offset - elbow_offset + wrrist_1_offset = 0.10915 -->
+  <property name="shoulder_offset" value="0.13585" />  <!-- shoulder_offset - elbow_offset + wrist_1_length = 0.10915 -->
   <property name="upper_arm_length" value="0.42500" />
-  <property name="elbow_offset" value="0.130" />       <!-- CAD measured -->
+  <property name="elbow_offset" value="0.1197" />       <!-- CAD measured -->
   <property name="forearm_length" value="0.39225" />
-  <property name="wrist_1_length" value="0.100" />     <!-- CAD measured -->
-  <property name="wrist_2_length" value="0.09465" />
+  <property name="wrist_1_length" value="0.093" />     <!-- CAD measured -->
+  <property name="wrist_2_length" value="0.09465" />   <!-- In CAD this distance is 0.930, but in the spec it is 0.09465 -->
   <property name="wrist_3_length" value="0.0823" />
   <property name="shoulder_radius" value="0.060" />   <!-- manually measured -->
   <property name="upper_arm_radius" value="0.054" />  <!-- manually measured -->
   <property name="elbow_radius" value="0.060" />      <!-- manually measured -->
-  <property name="forearm_radius" value="0.038" />    <!-- manually measured -->
-  <property name="wrist_radius" value="0.035" />      <!-- manually measured -->
+  <property name="forearm_radius" value="0.040" />    <!-- manually measured -->
+  <property name="wrist_radius" value="0.045" />      <!-- manually measured -->
 <!-- Collision model -->
   <property name="base_collision_length" value="0.160" />      <!-- manually measured -->
@@ -47,4 +47,10 @@
   <property name="elbow_collision_offset" value="0.035" />     <!-- manually measured -->
   <link name="base_link" >
+    <visual>
+      <geometry>
+        <mesh filename="package://ur5_description/meshes/Base.dae" />
+      </geometry>
+      <origin xyz="0.0 0.0 0.003" rpy="0.0 0.0 ${3.0 * pi / 4.0}" />
+    </visual>
     <inertial>
       <mass value="${base_mass}" />
@@ -63,13 +69,12 @@
     <visual>
       <geometry>
+        <mesh filename="package://ur5_description/meshes/Shoulder.dae" />
+      </geometry>
+    </visual>
+    <collision>
+      <geometry>
         <cylinder length="${base_collision_length}" radius="${shoulder_radius}"/>
       </geometry>
-      <origin xyz="0.0 0.0 ${base_collision_length / 2.0 - shoulder_height}" rpy="0.0 0.0 0.0" />
-    </visual>
-    <collision>
-      <geometry>
-        <cylinder length="${shoulder_height}" radius="${shoulder_radius}"/>
-      </geometry>
-      <origin xyz="0.0 0.0 ${-shoulder_height/2.0}" rpy="0.0 0.0 0.0" />
+      <origin xyz="0.0 0.0 ${-shoulder_height + (base_collision_length/2.0)}" rpy="0.0 0.0 0.0" />
     </collision>
     <inertial>
@@ -90,5 +95,5 @@
     <visual>
       <geometry>
-       <mesh filename="package://ur5_description/meshes/UpperArm.dae" />
+        <mesh filename="package://ur5_description/meshes/UpperArm.dae" />
       </geometry>
       <origin xyz="0.0 0.0 0.0" rpy="0.0 0.0 0.0" />
@@ -117,7 +122,6 @@
     <visual>
       <geometry>
-        <cylinder length="${forearm_length}" radius="${forearm_radius}"/>
-      </geometry>
-      <origin xyz="0.0 0.0 ${forearm_length/2.0}" rpy="0.0 0.0 0.0" />
+        <mesh filename="package://ur5_description/meshes/Forearm.dae" />
+      </geometry>
     </visual>
     <collision>
@@ -144,13 +148,13 @@
     <visual>
       <geometry>
-        <cylinder length="${wrist_1_length}" radius="${wrist_radius}"/>
-      </geometry>
-      <origin xyz="0.0 ${wrist_1_length/2.0} 0.0" rpy="${-pi/2.0} 0.0 0.0" />
-    </visual>
-    <collision>
-      <geometry>
-        <cylinder length="${wrist_1_length}" radius="${wrist_radius}"/>
-      </geometry>
-      <origin xyz="0.0 ${wrist_1_length/2.0} 0.0" rpy="${-pi/2.0} 0.0 0.0" />
+        <mesh filename="package://ur5_description/meshes/Wrist1.dae" />
+      </geometry>
+      <origin xyz="0.0 ${wrist_1_length} 0.0" rpy="0.0 ${pi / 2.0} 0.0" />
+    </visual>
+    <collision>
+      <geometry>
+        <cylinder length="${1.6*wrist_1_length}" radius="${wrist_radius}"/>
+      </geometry>
+      <origin xyz="0.0 ${0.25*wrist_1_length} 0.0" rpy="${-pi/2.0} 0.0 0.0" />
     </collision>
     <inertial>
@@ -171,13 +175,13 @@
     <visual>
       <geometry>
-        <cylinder length="${wrist_2_length}" radius="${wrist_radius}"/>
-      </geometry>
-      <origin xyz="0.0 0.0 ${wrist_2_length/2.0}" rpy="0.0 0.0 0.0" />
-    </visual>
-    <collision>
-      <geometry>
-        <cylinder length="${wrist_2_length}" radius="${wrist_radius}"/>
-      </geometry>
-      <origin xyz="0.0 0.0 ${wrist_2_length/2.0}" rpy="0.0 0.0 0.0" />
+        <mesh filename="package://ur5_description/meshes/Wrist2.dae" />
+      </geometry>
+      <origin xyz="0.0 0.0 ${wrist_2_length}" rpy="0.0 0.0 0.0" />
+    </visual>
+    <collision>
+      <geometry>
+        <cylinder length="${1.6*wrist_2_length}" radius="${wrist_radius}"/>
+      </geometry>
+      <origin xyz="0.0 0.0 ${0.25*wrist_2_length}" rpy="0.0 0.0 0.0" />
     </collision>
     <inertial>
@@ -190,5 +194,5 @@
     <parent link="wrist_2_link" />
     <child link = "wrist_3_link" />
-    <origin xyz="0.0 0.0 ${wrist_3_length}" rpy="0.0 0.0 0.0" />
+    <origin xyz="0.0 0.0 ${wrist_2_length}" rpy="0.0 0.0 0.0" />
     <axis xyz="0.0 1.0 0.0" />
     <limit lower="${-2.0 * pi}" upper="${2.0 * pi}" effort="10.0" velocity="${pi}"/>
@@ -198,13 +202,12 @@
     <visual>
       <geometry>
-        <cylinder length="${wrist_3_length}" radius="${wrist_radius}"/>
-      </geometry>
-      <origin xyz="0.0 ${wrist_3_length/2.0} 0.0" rpy="${-pi/2.0} 0.0 0.0" />
-    </visual>
-    <collision>
-      <geometry>
-        <cylinder length="${wrist_3_length}" radius="${wrist_radius}"/>
-      </geometry>
-      <origin xyz="0.0 ${wrist_3_length/2.0} 0.0" rpy="${-pi/2.0} 0.0 0.0" />
+        <mesh filename="package://ur5_description/meshes/Wrist3.dae" />
+      </geometry>
+    </visual>
+    <collision>
+      <geometry>
+        <cylinder length="${1.65*wrist_3_length}" radius="${wrist_radius}"/>
+      </geometry>
+      <origin xyz="0.0 ${0.15 * wrist_3_length} 0.0" rpy="${-pi/2.0} 0.0 0.0" />
     </collision>
     <inertial>
@@ -219,18 +222,5 @@
     <origin xyz="0.0 ${wrist_3_length} 0.0" rpy="0.0 0.0 ${pi/2.0}" />
   </joint>
-  <link name="ee_link">
-    <visual>
-      <geometry>
-        <cylinder length="0.01" radius="${wrist_radius * 1.25}"/>
-      </geometry>
-      <origin xyz="0.0 0.0 0.0" rpy="0.0 ${-pi/2.0} 0.0" />
-    </visual>
-    <collision>
-      <geometry>
-        <cylinder length="0.01" radius="${wrist_radius * 1.25}"/>
-      </geometry>
-      <origin xyz="0.0 0.0 0.0" rpy="0.0 ${-pi/2.0} 0.0" />
-    </collision>
-  </link>
+  <link name="ee_link" />
   <!-- Extra links for collision model -->
   <joint name="shoulder_collision_joint" type="fixed">
