Commit message: add prefix to urdf

File: ur5_description/urdf/model.urdf.xacro (robot description, xacro)
@@ -1,3 +1,4 @@
 <?xml version="1.0"?>
+<robot xmlns:xacro="http://ros.org/wiki/xacro" >
 <!--
 DH for UR5:
@@ -10,5 +11,4 @@
 center_of_mass = [ [0, -0.02561, 0.00193], [0.2125, 0, 0.11336], [0.11993, 0.0, 0.0265], [0, -0.0018, 0.01634], [0, 0.0018,0.01634], [0, 0, -0.001159] ]
 -->
-<robot>
   <property name="pi" value="3.14159265" />
 <!-- Inertia parameters -->
@@ -46,5 +46,6 @@
   <property name="elbow_collision_length" value="0.200" />     <!-- manually measured -->
   <property name="elbow_collision_offset" value="0.035" />     <!-- manually measured -->
-  <link name="base_link" >
+<xacro:macro name="ur5_robot" params="prefix">
+  <link name="${prefix}base_link" >
     <visual>
       <geometry>
@@ -59,6 +60,6 @@
   </link>
   <joint name="shoulder_pan_joint" type="revolute">
-    <parent link="base_link" />
-    <child link = "shoulder_link" />
+    <parent link="${prefix}base_link" />
+    <child link = "${prefix}shoulder_link" />
     <origin xyz="0.0 0.0 ${shoulder_height}" rpy="0.0 0.0 0.0" />
     <axis xyz="0.0 0.0 1.0" />
@@ -66,5 +67,5 @@
     <dynamics damping="0.1" friction="0.1"/>
   </joint>
-  <link name="shoulder_link">
+  <link name="${prefix}shoulder_link">
     <visual>
       <geometry>
@@ -85,6 +86,6 @@
   </link>
   <joint name="shoulder_lift_joint" type="revolute">
-    <parent link="shoulder_link" />
-    <child link = "upper_arm_link" />
+    <parent link="${prefix}shoulder_link" />
+    <child link = "${prefix}upper_arm_link" />
     <origin xyz="0.0 ${shoulder_offset} 0.0" rpy="0.0 ${pi / 2.0} 0.0" />
     <axis xyz="0.0 1.0 0.0" />
@@ -92,5 +93,5 @@
     <dynamics damping="0.1" friction="0.1"/>
   </joint>
-  <link name="upper_arm_link">
+  <link name="${prefix}upper_arm_link">
     <visual>
       <geometry>
@@ -112,6 +113,6 @@
   </link>
   <joint name="elbow_joint" type="revolute">
-    <parent link="upper_arm_link" />
-    <child link = "forearm_link" />
+    <parent link="${prefix}upper_arm_link" />
+    <child link = "${prefix}forearm_link" />
     <origin xyz="0.0 ${-elbow_offset} ${upper_arm_length}" rpy="0.0 0.0 0.0" />
     <axis xyz="0.0 1.0 0.0" />
@@ -119,5 +120,5 @@
     <dynamics damping="0.1" friction="0.1"/>
   </joint>
-  <link name="forearm_link">
+  <link name="${prefix}forearm_link">
     <visual>
       <geometry>
@@ -138,6 +139,6 @@
   </link>
   <joint name="wrist_1_joint" type="revolute">
-    <parent link="forearm_link" />
-    <child link = "wrist_1_link" />
+    <parent link="${prefix}forearm_link" />
+    <child link = "${prefix}wrist_1_link" />
     <origin xyz="0.0 0.0 ${forearm_length}" rpy="0.0 ${pi / 2.0} 0.0" />
     <axis xyz="0.0 1.0 0.0" />
@@ -145,5 +146,5 @@
     <dynamics damping="0.1" friction="0.1"/>
   </joint>
-  <link name="wrist_1_link">
+  <link name="${prefix}wrist_1_link">
     <visual>
       <geometry>
@@ -165,6 +166,6 @@
   </link>
   <joint name="wrist_2_joint" type="revolute">
-    <parent link="wrist_1_link" />
-    <child link = "wrist_2_link" />
+    <parent link="${prefix}wrist_1_link" />
+    <child link = "${prefix}wrist_2_link" />
     <origin xyz="0.0 ${wrist_1_length} 0.0" rpy="0.0 0.0 0.0" />
     <axis xyz="0.0 0.0 1.0" />
@@ -172,5 +173,5 @@
     <dynamics damping="0.1" friction="0.1"/>
   </joint>
-  <link name="wrist_2_link">
+  <link name="${prefix}wrist_2_link">
     <visual>
       <geometry>
@@ -192,6 +193,6 @@
   </link>
   <joint name="wrist_3_joint" type="revolute">
-    <parent link="wrist_2_link" />
-    <child link = "wrist_3_link" />
+    <parent link="${prefix}wrist_2_link" />
+    <child link = "${prefix}wrist_3_link" />
     <origin xyz="0.0 0.0 ${wrist_2_length}" rpy="0.0 0.0 0.0" />
     <axis xyz="0.0 1.0 0.0" />
@@ -199,5 +200,5 @@
     <dynamics damping="0.1" friction="0.1"/>
   </joint>
-  <link name="wrist_3_link">
+  <link name="${prefix}wrist_3_link">
     <visual>
       <geometry>
@@ -218,15 +219,15 @@
   </link>
   <joint name="ee_fixed_joint" type="fixed">
-    <parent link="wrist_3_link" />
-    <child link = "ee_link" />
+    <parent link="${prefix}wrist_3_link" />
+    <child link = "${prefix}ee_link" />
     <origin xyz="0.0 ${wrist_3_length} 0.0" rpy="0.0 0.0 ${pi/2.0}" />
   </joint>
-  <link name="ee_link" />
+  <link name="${prefix}ee_link" />
   <!-- Extra links for collision model -->
   <joint name="shoulder_collision_joint" type="fixed">
-    <parent link="upper_arm_link" />
-    <child link = "shoulder_collision_link" />
-  </joint>
-  <link name="shoulder_collision_link">
+    <parent link="${prefix}upper_arm_link" />
+    <child link = "${prefix}shoulder_collision_link" />
+  </joint>
+  <link name="${prefix}shoulder_collision_link">
     <collision>
       <geometry>
@@ -237,8 +238,8 @@
   </link>
   <joint name="elbow_collision_joint" type="fixed">
-    <parent link="upper_arm_link" />
-    <child link = "elbow_collision_link" />
-  </joint>
-  <link name="elbow_collision_link">
+    <parent link="${prefix}upper_arm_link" />
+    <child link = "${prefix}elbow_collision_link" />
+  </joint>
+  <link name="${prefix}elbow_collision_link">
     <collision>
       <geometry>
@@ -251,3 +252,4 @@
     <material>Gazebo/Blue</material>
   </gazebo>
+</xacro:macro>
 </robot>

File: ur5_description/urdf/robot.urdf.xacro (robot description, xacro)
@@ -1,4 +1,6 @@
 <?xml version="1.0"?>
-<robot name="ur5">
+<robot xmlns:xacro="http://ros.org/wiki/xacro"
+       name="ur5">
   <include filename="$(find ur5_description)/urdf/model.urdf.xacro" />
+  <xacro:ur5_robot prefix="" />
 </robot>

Commit message: apply prefix to joints too

File: ur5_description/urdf/model.urdf.xacro (robot description, xacro)
@@ -59,5 +59,5 @@
     </inertial>
   </link>
-  <joint name="shoulder_pan_joint" type="revolute">
+  <joint name="${prefix}shoulder_pan_joint" type="revolute">
     <parent link="${prefix}base_link" />
     <child link = "${prefix}shoulder_link" />
@@ -85,5 +85,5 @@
     </inertial>
   </link>
-  <joint name="shoulder_lift_joint" type="revolute">
+  <joint name="${prefix}shoulder_lift_joint" type="revolute">
     <parent link="${prefix}shoulder_link" />
     <child link = "${prefix}upper_arm_link" />
@@ -112,5 +112,5 @@
     </inertial>
   </link>
-  <joint name="elbow_joint" type="revolute">
+  <joint name="${prefix}elbow_joint" type="revolute">
     <parent link="${prefix}upper_arm_link" />
     <child link = "${prefix}forearm_link" />
@@ -138,5 +138,5 @@
     </inertial>
   </link>
-  <joint name="wrist_1_joint" type="revolute">
+  <joint name="${prefix}wrist_1_joint" type="revolute">
     <parent link="${prefix}forearm_link" />
     <child link = "${prefix}wrist_1_link" />
@@ -165,5 +165,5 @@
     </inertial>
   </link>
-  <joint name="wrist_2_joint" type="revolute">
+  <joint name="${prefix}wrist_2_joint" type="revolute">
     <parent link="${prefix}wrist_1_link" />
     <child link = "${prefix}wrist_2_link" />
@@ -192,5 +192,5 @@
     </inertial>
   </link>
-  <joint name="wrist_3_joint" type="revolute">
+  <joint name="${prefix}wrist_3_joint" type="revolute">
     <parent link="${prefix}wrist_2_link" />
     <child link = "${prefix}wrist_3_link" />
@@ -218,5 +218,5 @@
     </inertial>
   </link>
-  <joint name="ee_fixed_joint" type="fixed">
+  <joint name="${prefix}ee_fixed_joint" type="fixed">
     <parent link="${prefix}wrist_3_link" />
     <child link = "${prefix}ee_link" />
@@ -225,5 +225,5 @@
   <link name="${prefix}ee_link" />
   <!-- Extra links for collision model -->
-  <joint name="shoulder_collision_joint" type="fixed">
+  <joint name="${prefix}shoulder_collision_joint" type="fixed">
     <parent link="${prefix}upper_arm_link" />
     <child link = "${prefix}shoulder_collision_link" />
@@ -237,5 +237,5 @@
     </collision>
   </link>
-  <joint name="elbow_collision_joint" type="fixed">
+  <joint name="${prefix}elbow_collision_joint" type="fixed">
     <parent link="${prefix}upper_arm_link" />
     <child link = "${prefix}elbow_collision_link" />

Commit message: changed damping values for simulation

File: ur5_description/urdf/model.urdf.xacro (robot description, xacro)
@@ -69,5 +69,5 @@
     <axis xyz="0.0 0.0 1.0" />
     <limit lower="${-2.0 * pi}" upper="${2.0 * pi}" effort="10.0" velocity="${pi}"/>
-    <dynamics damping="0.1" friction="0.1"/>
+    <dynamics damping="10" friction="0.1"/>
   </joint>
   <link name="${prefix}shoulder_link">
@@ -95,5 +95,5 @@
     <axis xyz="0.0 1.0 0.0" />
     <limit lower="${-2.0 * pi}" upper="${2.0 * pi}" effort="10.0" velocity="${pi}"/>
-    <dynamics damping="0.1" friction="0.1"/>
+    <dynamics damping="10" friction="0.1"/>
   </joint>
   <link name="${prefix}upper_arm_link">
@@ -122,5 +122,5 @@
     <axis xyz="0.0 1.0 0.0" />
     <limit lower="${-2.0 * pi}" upper="${2.0 * pi}" effort="10.0" velocity="${pi}"/>
-    <dynamics damping="0.1" friction="0.1"/>
+    <dynamics damping="10" friction="0.1"/>
   </joint>
   <link name="${prefix}forearm_link">
@@ -148,5 +148,5 @@
     <axis xyz="0.0 1.0 0.0" />
     <limit lower="${-2.0 * pi}" upper="${2.0 * pi}" effort="10.0" velocity="${pi}"/>
-    <dynamics damping="0.1" friction="0.1"/>
+    <dynamics damping="10" friction="0.1"/>
   </joint>
   <link name="${prefix}wrist_1_link">
@@ -175,5 +175,5 @@
     <axis xyz="0.0 0.0 1.0" />
     <limit lower="${-2.0 * pi}" upper="${2.0 * pi}" effort="10.0" velocity="${pi}"/>
-    <dynamics damping="0.1" friction="0.1"/>
+    <dynamics damping="10" friction="0.1"/>
   </joint>
   <link name="${prefix}wrist_2_link">
@@ -202,5 +202,5 @@
     <axis xyz="0.0 1.0 0.0" />
     <limit lower="${-2.0 * pi}" upper="${2.0 * pi}" effort="10.0" velocity="${pi}"/>
-    <dynamics damping="0.1" friction="0.1"/>
+    <dynamics damping="10" friction="0.1"/>
   </joint>
   <link name="${prefix}wrist_3_link">

Commit message: Cleaning up joint axes in urdf.

File: ur5_description/urdf/model.urdf.xacro (robot description, xacro)
@@ -67,5 +67,5 @@
     <child link = "${prefix}shoulder_link" />
     <origin xyz="0.0 0.0 ${shoulder_height}" rpy="0.0 0.0 0.0" />
-    <axis xyz="0.0 0.0 1.0" />
+    <axis xyz="0 0 1" />
     <limit lower="${-2.0 * pi}" upper="${2.0 * pi}" effort="10.0" velocity="${pi}"/>
     <dynamics damping="10" friction="0.1"/>
@@ -93,5 +93,5 @@
     <child link = "${prefix}upper_arm_link" />
     <origin xyz="0.0 ${shoulder_offset} 0.0" rpy="0.0 ${pi / 2.0} 0.0" />
-    <axis xyz="0.0 1.0 0.0" />
+    <axis xyz="0 1 0" />
     <limit lower="${-2.0 * pi}" upper="${2.0 * pi}" effort="10.0" velocity="${pi}"/>
     <dynamics damping="10" friction="0.1"/>
@@ -120,5 +120,5 @@
     <child link = "${prefix}forearm_link" />
     <origin xyz="0.0 ${-elbow_offset} ${upper_arm_length}" rpy="0.0 0.0 0.0" />
-    <axis xyz="0.0 1.0 0.0" />
+    <axis xyz="0 1 0" />
     <limit lower="${-2.0 * pi}" upper="${2.0 * pi}" effort="10.0" velocity="${pi}"/>
     <dynamics damping="10" friction="0.1"/>
@@ -146,5 +146,5 @@
     <child link = "${prefix}wrist_1_link" />
     <origin xyz="0.0 0.0 ${forearm_length}" rpy="0.0 ${pi / 2.0} 0.0" />
-    <axis xyz="0.0 1.0 0.0" />
+    <axis xyz="0 1 0" />
     <limit lower="${-2.0 * pi}" upper="${2.0 * pi}" effort="10.0" velocity="${pi}"/>
     <dynamics damping="10" friction="0.1"/>
@@ -173,5 +173,5 @@
     <child link = "${prefix}wrist_2_link" />
     <origin xyz="0.0 ${wrist_1_length} 0.0" rpy="0.0 0.0 0.0" />
-    <axis xyz="0.0 0.0 1.0" />
+    <axis xyz="0 0 1" />
     <limit lower="${-2.0 * pi}" upper="${2.0 * pi}" effort="10.0" velocity="${pi}"/>
     <dynamics damping="10" friction="0.1"/>
@@ -200,5 +200,5 @@
     <child link = "${prefix}wrist_3_link" />
     <origin xyz="0.0 0.0 ${wrist_2_length}" rpy="0.0 0.0 0.0" />
-    <axis xyz="0.0 1.0 0.0" />
+    <axis xyz="0 1 0" />
     <limit lower="${-2.0 * pi}" upper="${2.0 * pi}" effort="10.0" velocity="${pi}"/>
     <dynamics damping="10" friction="0.1"/>
