Commit message: Renamed packages and new groovy version

File: ur_description/urdf/materials.urdf.xacro (robot description, xacro)
@@ -1,8 +1,8 @@
 <?xml version="1.0"?>
 <robot>
-  <material name="Blue">
+  <material name="UR/Blue">
     <color rgba="0.0 0.0 0.8 1.0"/>
   </material>
-  <material name="Grey">
+  <material name="UR/Grey">
     <color rgba="0.7 0.7 0.7 1.0"/>
   </material>

File: ur_description/urdf/ur10.urdf.xacro (robot description, xacro)
@@ -65,5 +65,5 @@
       </geometry>
       <origin xyz="0.0 0.0 0.003" rpy="0.0 0.0 ${3.0 * pi / 4.0}" />
-      <material name="Blue" />
+      <material name="UR/Blue" />
     </visual>
     <inertial>
@@ -85,5 +85,5 @@
         <mesh filename="package://ur_description/meshes/ur10/Shoulder.stl" />
       </geometry>
-      <material name="Grey" />
+      <material name="UR/Grey" />
     </visual>
     <collision>
@@ -113,5 +113,5 @@
       </geometry>
       <origin xyz="0.0 0.0 0.0" rpy="0.0 0.0 0.0" />
-      <material name="Blue" />
+      <material name="UR/Blue" />
     </visual>
     <collision>
@@ -140,5 +140,5 @@
         <mesh filename="package://ur_description/meshes/ur10/Forearm_new.stl" />
       </geometry>
-      <material name="Grey" />
+      <material name="UR/Grey" />
     </visual>
     <collision>
@@ -168,5 +168,5 @@
       </geometry>
       <origin xyz="0.0 ${wrist_1_length} 0.0" rpy="0.0 0 0.0" />
-      <material name="Blue" />
+      <material name="UR/Blue" />
     </visual>
     <collision>
@@ -196,5 +196,5 @@
       </geometry>
       <origin xyz="0.0 0.0 ${wrist_2_length}" rpy="0.0 0.0 0.0" />
-      <material name="Grey" />
+      <material name="UR/Grey" />
     </visual>
     <collision>
@@ -224,5 +224,5 @@
       </geometry>
       <origin xyz="0.0 ${wrist_3_length} 0.0" rpy="0.0 0.0 0" />
-      <material name="Blue" />
+      <material name="UR/Blue" />
     </visual>
     <collision>
@@ -274,5 +274,5 @@
   <xacro:ur10_arm_gazebo name="${name}" />
   <!--gazebo reference="universal_robot">
-    <material>Gazebo/Blue</material>
+    <material>Gazebo/UR/Blue</material>
   </gazebo-->
 </xacro:macro>

File: ur_description/urdf/ur10_robot.urdf.xacro (robot description, xacro)
@@ -1,7 +1,37 @@
 <?xml version="1.0"?>
-<robot xmlns:xacro="http://ros.org/wiki/xacro"
-       name="ur10">
-  <include filename="$(find ur_description)/urdf/ur10.gazebo.xacro" />
+<robot xmlns:sensor="http://playerstage.sourceforge.net/gazebo/xmlschema/#sensor"
+       xmlns:controller="http://playerstage.sourceforge.net/gazebo/xmlschema/#controller"
+       xmlns:interface="http://playerstage.sourceforge.net/gazebo/xmlschema/#interface"
+       xmlns:xacro="http://playerstage.sourceforge.net/gazebo/xmlschema/#interface"
+       name="ur10" >
+  <!-- common stuff -->
+  <include filename="$(find ur_description)/urdf/gazebo.urdf.xacro" />
+  <!--include filename="$(find ur_description)/urdf/materials.urdf.xacro" /-->
+  <!-- ur10 -->
   <include filename="$(find ur_description)/urdf/ur10.urdf.xacro" />
-  <xacro:ur10_robot prefix="" />
+  <!-- foot for arm -->
+	<link name="base_link">
+		<inertial>
+		   <origin xyz="0 0 -10" rpy="0 0 0"/>
+		   <mass value="1000.0"/>
+		   <inertia ixx="100.0"  ixy="0"  ixz="0" iyy="100.0" iyz="0" izz="100.0" />
+		</inertial>
+		<visual>
+		   <origin xyz="0 0 0.25" rpy="0 0 0" />
+		   <geometry>
+			  <cylinder radius="0.1" length="0.5"/>
+		   </geometry>
+		   <material name="Grey" />
+		</visual>
+		<collision>
+		   <origin xyz="0 0 0.25" rpy="0 0 0" />
+		   <geometry>
+			  <cylinder radius="0.1" length="0.5"/>
+		   </geometry>
+		</collision>
+	</link>
+  <!-- arm -->
+  <xacro:ur10_robot name="arm" parent="base_link">
+    <origin xyz="0 0 0.5" rpy="0 0 0" />
+  </xacro:ur10_robot>
 </robot>

File: ur_description/urdf/ur5_robot.urdf.xacro (robot description, xacro)
@@ -1,7 +1,15 @@
 <?xml version="1.0"?>
-<robot xmlns:xacro="http://ros.org/wiki/xacro"
-       name="ur5">
-  <include filename="$(find ur_description)/urdf/ur5.gazebo.xacro" />
+<robot xmlns:sensor="http://playerstage.sourceforge.net/gazebo/xmlschema/#sensor"
+       xmlns:controller="http://playerstage.sourceforge.net/gazebo/xmlschema/#controller"
+       xmlns:interface="http://playerstage.sourceforge.net/gazebo/xmlschema/#interface"
+       xmlns:xacro="http://playerstage.sourceforge.net/gazebo/xmlschema/#interface"
+       name="ur5" >
+  <!-- common stuff -->
+  <include filename="$(find ur_description)/urdf/gazebo.urdf.xacro" />
+  <include filename="$(find ur_description)/urdf/materials.urdf.xacro" />
+  <!-- ur5 -->
   <include filename="$(find ur_description)/urdf/ur5.urdf.xacro" />
-  <xacro:ur5_robot prefix="" />
+  <!-- arm -->
+  <xacro:ur5_robot prefix="arm_">
+  </xacro:ur5_robot>
 </robot>
