Commit message: minor changes on ur5 xacro files

File: ur_description/urdf/ur5.gazebo.xacro (robot description, xacro)
@@ -2,24 +2,10 @@
 <robot xmlns:sensor="http://playerstage.sourceforge.net/gazebo/xmlschema/#sensor"
        xmlns:controller="http://playerstage.sourceforge.net/gazebo/xmlschema/#controller"
-       xmlns:interface="http://playerstage.sourceforge.net/gazebo/xmlschema/#interface">
-  <gazebo>
-    <controller:gazebo_ros_controller_manager name="gazebo_ros_controller_manager" plugin="libgazebo_ros_controller_manager.so">
-      <alwaysOn>true</alwaysOn>
-      <updateRate>1000.0</updateRate>
-      <interface:audio name="gazebo_ros_controller_manager_dummy_iface" />
-    </controller:gazebo_ros_controller_manager>
-    <controller:gazebo_ros_power_monitor name="gazebo_ros_power_monitor_controller" plugin="libgazebo_ros_power_monitor.so">
-      <alwaysOn>true</alwaysOn>
-      <updateRate>1.0</updateRate>
-      <timeout>5</timeout>
-      <interface:audio name="power_monitor_dummy_interface" />
-      <powerStateTopic>power_state</powerStateTopic>
-      <powerStateRate>10.0</powerStateRate>
-      <fullChargeCapacity>87.78</fullChargeCapacity>
-      <dischargeRate>-474</dischargeRate>
-      <chargeRate>525</chargeRate>
-      <dischargeVoltage>15.52</dischargeVoltage>
-      <chargeVoltage>16.41</chargeVoltage>
-    </controller:gazebo_ros_power_monitor>
-  </gazebo>
+       xmlns:interface="http://playerstage.sourceforge.net/gazebo/xmlschema/#interface"
+       xmlns:xacro="http://ros.org/wiki/xacro">
+	<xacro:macro name="ur5_arm_gazebo" params="name">
+	  <gazebo reference="universal_robot">
+	    <material>Gazebo/Blue</material>
+	  </gazebo>
+	</xacro:macro>
 </robot>

File: ur_description/urdf/ur5.urdf.xacro (robot description, xacro)
@@ -5,14 +5,15 @@
        xmlns:xacro="http://ros.org/wiki/xacro">
 <include filename="$(find ur_description)/urdf/ur5.transmission.xacro" />
-<!--
-DH for UR5:
-a = [0.00000, -0.42500, -0.39225,  0.00000,  0.00000,  0.0000]
-d = [0.089159,  0.00000,  0.00000,  0.10915,  0.09465,  0.0823]
-alpha = [ 1.570796327, 0, 0, 1.570796327, -1.570796327, 0 ]
-q_home_offset = [0, -1.570796327, 0, -1.570796327, 0, 0]
-joint_direction = [-1, -1, 1, 1, 1, 1]
-mass = [3.7000, 8.3930, 2.2750, 1.2190, 1.2190, 0.1879]
-center_of_mass = [ [0, -0.02561, 0.00193], [0.2125, 0, 0.11336], [0.11993, 0.0, 0.0265], [0, -0.0018, 0.01634], [0, 0.0018,0.01634], [0, 0, -0.001159] ]
--->
+  <include filename="$(find ur_description)/urdf/ur5.gazebo.xacro" />
+		<!--
+		DH for UR5:
+		a = [0.00000, -0.42500, -0.39225,  0.00000,  0.00000,  0.0000]
+		d = [0.089159,  0.00000,  0.00000,  0.10915,  0.09465,  0.0823]
+		alpha = [ 1.570796327, 0, 0, 1.570796327, -1.570796327, 0 ]
+		q_home_offset = [0, -1.570796327, 0, -1.570796327, 0, 0]
+		joint_direction = [-1, -1, 1, 1, 1, 1]
+		mass = [3.7000, 8.3930, 2.2750, 1.2190, 1.2190, 0.1879]
+		center_of_mass = [ [0, -0.02561, 0.00193], [0.2125, 0, 0.11336], [0.11993, 0.0, 0.0265], [0, -0.0018, 0.01634], [0, 0.0018,0.01634], [0, 0, -0.001159] ]
+		-->
   <property name="pi" value="3.14159265" />
 <!-- Inertia parameters -->
@@ -51,16 +52,16 @@
   <property name="elbow_collision_offset" value="0.035" />     <!-- manually measured -->
 <xacro:macro name="ur5_robot" params="prefix">
-  <link name="${prefix}base_link" >
-    <visual>
-      <geometry>
-        <mesh filename="package://ur_description/meshes/ur5/Base.dae" />
-      </geometry>
-      <origin xyz="0.0 0.0 0.003" rpy="0.0 0.0 ${3.0 * pi / 4.0}" />
-    </visual>
-    <inertial>
-      <mass value="${base_mass}" />
-      <inertia ixx="1.0" ixy="0.0" ixz="0.0" iyy="1.0" iyz="0.0" izz="1.0"/>
-    </inertial>
-  </link>
+	<link name="${prefix}base_link" >
+		<visual>
+		  <geometry>
+		    <mesh filename="package://ur_description/meshes/ur5/Base.dae" />
+		  </geometry>
+		  <origin xyz="0.0 0.0 0.003" rpy="0.0 0.0 ${3.0 * pi / 4.0}" />
+		</visual>
+		<inertial>
+		  <mass value="${base_mass}" />
+		  <inertia ixx="1.0" ixy="0.0" ixz="0.0" iyy="1.0" iyz="0.0" izz="1.0"/>
+		</inertial>
+	</link>
   <joint name="${prefix}shoulder_pan_joint" type="revolute">
     <parent link="${prefix}base_link" />
@@ -256,7 +257,5 @@
   -->
   <xacro:ur5_arm_transmission name="${prefix}" />
-  <gazebo reference="universal_robot">
-    <material>Gazebo/Blue</material>
-  </gazebo>
+  <xacro:ur5_arm_gazebo name="${prefix}" />
 </xacro:macro>
 </robot>

File: ur_description/urdf/ur5_robot.urdf.xacro (robot description, xacro)
@@ -10,4 +10,31 @@
   <!-- ur5 -->
   <include filename="$(find ur_description)/urdf/ur5.urdf.xacro" />
+  <!-- foot for arm -->
+	<link name="base_link">
+		<inertial>
+		   <origin xyz="0 0 -10" rpy="0 0 0"/>
+		   <mass value="1000.0"/>
+		   <inertia ixx="100.0"  ixy="0"  ixz="0" iyy="100.0" iyz="0" izz="100.0" />
+		</inertial>
+		<visual>
+		   <origin xyz="0 0 0.25" rpy="0 0 0" />
+		   <geometry>
+			  <cylinder radius="0.1" length="0.5"/>
+		   </geometry>
+		   <material name="Grey" />
+		</visual>
+		<collision>
+		   <origin xyz="0 0 0.25" rpy="0 0 0" />
+		   <geometry>
+			  <cylinder radius="0.1" length="0.5"/>
+		   </geometry>
+		</collision>
+	</link>
+	<!-- joint between base_link and ur_base_link -->
+	<joint name="arm_base_joint" type="fixed" >
+		<origin xyz="0 0 0.5" rpy="0 0 0" />
+		<parent link="base_link" />
+		<child link="arm_base_link" />
+	</joint>
   <!-- arm -->
   <xacro:ur5_robot prefix="arm_">

Commit message: use same xacro params as ur10

File: ur_description/urdf/ur5.gazebo.xacro (robot description, xacro)
@@ -1,5 +1,5 @@
 <?xml version="1.0"?>
 <robot xmlns:xacro="http://www.ros.org/wiki/xacro">
-  <xacro:macro name="ur5_arm_gazebo" params="name">
+  <xacro:macro name="ur5_arm_gazebo" params="prefix">
     <gazebo reference="universal_robot">
       <material>Gazebo/Blue</material>

File: ur_description/urdf/ur5.urdf.xacro (robot description, xacro)
@@ -226,8 +226,6 @@
   </joint>
   <link name="${prefix}ee_link" />
-  <xacro:ur5_arm_transmission name="${prefix}" />
-  <gazebo reference="universal_robot">
-    <material>Gazebo/Blue</material>
-  </gazebo>
-</xacro:macro>
+  <xacro:ur5_arm_transmission prefix="${prefix}" />
+  <xacro:ur5_arm_gazebo prefix="${prefix}" />
+  </xacro:macro>
 </robot>
