Commit message: fixed typo in limits

File: ur_description/urdf/ur10_limited.urdf.xacro (robot description, xacro)
@@ -64,5 +64,5 @@
     <origin xyz="0.0 0.0 ${shoulder_height}" rpy="0.0 0.0 0.0" />
     <axis xyz="0.0 0.0 1.0" />
-    <limit lower="${pi}" upper="${pi}" effort="330.0" velocity="2.16"/>
+    <limit lower="${-pi}" upper="${pi}" effort="330.0" velocity="2.16"/>
     <dynamics damping="1.2" friction="0.0"/>
   </joint>
@@ -90,5 +90,5 @@
     <origin xyz="0.0 ${shoulder_offset} 0.0" rpy="0.0 ${pi / 2.0} 0.0" />
     <axis xyz="0.0 1.0 0.0" />
-    <limit lower="${pi}" upper="${pi}" effort="10.0" velocity="${pi}"/>
+    <limit lower="${-pi}" upper="${pi}" effort="10.0" velocity="${pi}"/>
     <dynamics damping="1.2" friction="0.0"/>
   </joint>
@@ -118,5 +118,5 @@
     <origin xyz="0.0 ${-elbow_offset} ${upper_arm_length}" rpy="0.0 0.0 0.0" />
     <axis xyz="0.0 1.0 0.0" />
-    <limit lower="${pi}" upper="${pi}" effort="150.0" velocity="${pi}"/>
+    <limit lower="${-pi}" upper="${pi}" effort="150.0" velocity="${pi}"/>
     <dynamics damping="0.6" friction="0.0"/>
   </joint>
@@ -144,5 +144,5 @@
     <origin xyz="0.0 0.0 ${forearm_length}" rpy="0.0 ${pi / 2.0} 0.0" />
     <axis xyz="0.0 1.0 0.0" />
-    <limit lower="${pi}" upper="${pi}" effort="54.0" velocity="${pi}"/>
+    <limit lower="${-pi}" upper="${pi}" effort="54.0" velocity="${pi}"/>
     <dynamics damping="0.6" friction="0.0"/>
   </joint>
@@ -172,5 +172,5 @@
     <origin xyz="0.0 ${wrist_1_length} 0.0" rpy="0.0 0.0 0.0" />
     <axis xyz="0.0 0.0 1.0" />
-    <limit lower="${pi}" upper="${pi}" effort="54.0" velocity="${pi}"/>
+    <limit lower="${-pi}" upper="${pi}" effort="54.0" velocity="${pi}"/>
     <dynamics damping="0.6" friction="0.0"/>
   </joint>
@@ -200,5 +200,5 @@
     <origin xyz="0.0 0.0 ${wrist_2_length}" rpy="0.0 0.0 0.0" />
     <axis xyz="0.0 1.0 0.0" />
-    <limit lower="${pi}" upper="${pi}" effort="54.0" velocity="${pi}"/>
+    <limit lower="${-pi}" upper="${pi}" effort="54.0" velocity="${pi}"/>
     <dynamics damping="0.6" friction="0.0"/>
   </joint>

File: ur_description/urdf/ur5_limited.urdf.xacro (robot description, xacro)
@@ -93,5 +93,5 @@
     <origin xyz="0.0 ${shoulder_offset} 0.0" rpy="0.0 ${pi / 2.0} 0.0" />
     <axis xyz="0 1 0" />
-    <limit lower="${pi}" upper="${pi}" effort="150.0" velocity="${pi}"/>
+    <limit lower="${-pi}" upper="${pi}" effort="150.0" velocity="${pi}"/>
     <dynamics damping="0.4" friction="0.0"/>
   </joint>
@@ -120,5 +120,5 @@
     <origin xyz="0.0 ${-elbow_offset} ${upper_arm_length}" rpy="0.0 0.0 0.0" />
     <axis xyz="0 1 0" />
-    <limit lower="${pi}" upper="${pi}" effort="150.0" velocity="${pi}"/>
+    <limit lower="${-pi}" upper="${pi}" effort="150.0" velocity="${pi}"/>
     <dynamics damping="0.4" friction="0.0"/>
   </joint>
