Commit message: update urdf files

File: ur_description/urdf/ur10_joint_limited_robot.urdf (robot description, URDF)
Before this commit: robot ur10, 8 links, 7 joints
Joints:
- joint elbow_joint: limit lower=-3.14159265 upper=3.14159265 effort=150.0 velocity=3.14159265 -> lower=-3.14159265 upper=3.14159265 effort=1000.0 velocity=3.14159265
- joint shoulder_lift_joint: limit lower=-3.14159265 upper=3.14159265 effort=10.0 velocity=3.14159265 -> lower=-3.14159265 upper=3.14159265 effort=1000.0 velocity=3.14159265
- joint shoulder_pan_joint: limit lower=-3.14159265 upper=3.14159265 effort=330.0 velocity=2.16 -> lower=-3.14159265 upper=3.14159265 effort=1000.0 velocity=2.16
- joint wrist_1_joint: limit lower=-3.14159265 upper=3.14159265 effort=54.0 velocity=3.14159265 -> lower=-3.14159265 upper=3.14159265 effort=1000.0 velocity=3.14159265
- joint wrist_2_joint: limit lower=-3.14159265 upper=3.14159265 effort=54.0 velocity=3.14159265 -> lower=-3.14159265 upper=3.14159265 effort=1000.0 velocity=3.14159265
- joint wrist_3_joint: limit lower=-3.14159265 upper=3.14159265 effort=54.0 velocity=3.14159265 -> lower=-3.14159265 upper=3.14159265 effort=1000.0 velocity=3.14159265

File: ur_description/urdf/ur10_robot.urdf (robot description, URDF)
Before this commit: robot ur10, 8 links, 7 joints
Joints:
- joint elbow_joint: limit lower=-6.2831853 upper=6.2831853 effort=150.0 velocity=3.14159265 -> lower=-6.2831853 upper=6.2831853 effort=1000.0 velocity=3.14159265
- joint shoulder_lift_joint: limit lower=-6.2831853 upper=6.2831853 effort=10.0 velocity=3.14159265 -> lower=-6.2831853 upper=6.2831853 effort=1000.0 velocity=3.14159265
- joint shoulder_pan_joint: limit lower=-6.2831853 upper=6.2831853 effort=330.0 velocity=2.16 -> lower=-6.2831853 upper=6.2831853 effort=1000.0 velocity=2.16
- joint wrist_1_joint: limit lower=-6.2831853 upper=6.2831853 effort=54.0 velocity=3.14159265 -> lower=-6.2831853 upper=6.2831853 effort=1000.0 velocity=3.14159265
- joint wrist_2_joint: limit lower=-6.2831853 upper=6.2831853 effort=54.0 velocity=3.14159265 -> lower=-6.2831853 upper=6.2831853 effort=1000.0 velocity=3.14159265
- joint wrist_3_joint: limit lower=-6.2831853 upper=6.2831853 effort=54.0 velocity=3.14159265 -> lower=-6.2831853 upper=6.2831853 effort=1000.0 velocity=3.14159265

File: ur_description/urdf/ur5_joint_limited_robot.urdf (robot description, URDF)
Before this commit: robot ur5, 8 links, 7 joints
Joints:
- joint elbow_joint: limit lower=-3.14159265 upper=3.14159265 effort=150.0 velocity=3.14159265 -> lower=-3.14159265 upper=3.14159265 effort=1000.0 velocity=3.14159265
- joint shoulder_lift_joint: limit lower=-3.14159265 upper=3.14159265 effort=150.0 velocity=3.14159265 -> lower=-3.14159265 upper=3.14159265 effort=1000.0 velocity=3.14159265
- joint shoulder_pan_joint: limit lower=-3.14159265 upper=3.14159265 effort=150.0 velocity=3.14159265 -> lower=-3.14159265 upper=3.14159265 effort=1000.0 velocity=3.14159265
- joint wrist_1_joint: limit lower=-3.14159265 upper=0.7853981625 effort=28.0 velocity=3.14159265 -> lower=-3.14159265 upper=0.7853981625 effort=1000.0 velocity=3.14159265
- joint wrist_2_joint: limit lower=-3.14159265 upper=3.14159265 effort=28.0 velocity=3.14159265 -> lower=-3.14159265 upper=3.14159265 effort=1000.0 velocity=3.14159265
- joint wrist_3_joint: limit lower=-3.14159265 upper=3.14159265 effort=28.0 velocity=3.14159265 -> lower=-3.14159265 upper=3.14159265 effort=1000.0 velocity=3.14159265

File: ur_description/urdf/ur5_robot.urdf (robot description, URDF)
Before this commit: robot ur5, 8 links, 7 joints
Joints:
- joint elbow_joint: limit lower=-6.2831853 upper=6.2831853 effort=150.0 velocity=3.14159265 -> lower=-6.2831853 upper=6.2831853 effort=1000.0 velocity=3.14159265
- joint shoulder_lift_joint: limit lower=-6.2831853 upper=6.2831853 effort=150.0 velocity=3.14159265 -> lower=-6.2831853 upper=6.2831853 effort=1000.0 velocity=3.14159265
- joint shoulder_pan_joint: limit lower=-6.2831853 upper=6.2831853 effort=150.0 velocity=3.14159265 -> lower=-6.2831853 upper=6.2831853 effort=1000.0 velocity=3.14159265
- joint wrist_1_joint: limit lower=-3.14159265 upper=0.7853981625 effort=28.0 velocity=3.14159265 -> lower=-3.14159265 upper=0.7853981625 effort=1000.0 velocity=3.14159265
- joint wrist_2_joint: limit lower=-3.14159265 upper=3.14159265 effort=28.0 velocity=3.14159265 -> lower=-3.14159265 upper=3.14159265 effort=1000.0 velocity=3.14159265
- joint wrist_3_joint: limit lower=-3.14159265 upper=3.14159265 effort=28.0 velocity=3.14159265 -> lower=-3.14159265 upper=3.14159265 effort=1000.0 velocity=3.14159265

Commit message: update urdf files

File: ur_description/urdf/ur10_joint_limited_robot.urdf (robot description, URDF)
Before this commit: robot ur10, 9 links, 8 joints
Links:
- link base_link: geometry collision mesh filename=package://ur_description/meshes/ur10/collision/Base.dae; visual mesh filename=package://ur_description/meshes/ur10/visual/Base.dae
- link forearm_link: geometry collision mesh filename=package://ur_description/meshes/ur10/collision/Forearm.dae; visual mesh filename=package://ur_description/meshes/ur10/visual/Forearm.dae
- link shoulder_link: geometry collision mesh filename=package://ur_description/meshes/ur10/collision/Shoulder.dae; visual mesh filename=package://ur_description/meshes/ur10/visual/Shoulder.dae
- link upper_arm_link: geometry collision mesh filename=package://ur_description/meshes/ur10/collision/UpperArm.dae; visual mesh filename=package://ur_description/meshes/ur10/visual/UpperArm.dae
- link wrist_1_link: geometry collision mesh filename=package://ur_description/meshes/ur10/collision/Wrist1.dae; visual mesh filename=package://ur_description/meshes/ur10/visual/Wrist1.dae
- link wrist_2_link: geometry collision mesh filename=package://ur_description/meshes/ur10/collision/Wrist2.dae; visual mesh filename=package://ur_description/meshes/ur10/visual/Wrist2.dae
- link wrist_3_link: geometry collision mesh filename=package://ur_description/meshes/ur10/collision/Wrist3.dae; visual mesh filename=package://ur_description/meshes/ur10/visual/Wrist3.dae
Joints:
- joint elbow_joint: axis 0.0 1.0 0.0 -> 0 1 0
- joint shoulder_lift_joint: axis 0.0 1.0 0.0 -> 0 1 0
- joint shoulder_pan_joint: axis 0.0 0.0 1.0 -> 0 0 1
- joint wrist_1_joint: axis 0.0 1.0 0.0 -> 0 1 0
- joint wrist_2_joint: axis 0.0 0.0 1.0 -> 0 0 1
- joint wrist_3_joint: axis 0.0 1.0 0.0 -> 0 1 0

File: ur_description/urdf/ur10_robot.urdf (robot description, URDF)
Before this commit: robot ur10, 9 links, 8 joints
Links:
- link base_link: geometry collision mesh filename=package://ur_description/meshes/ur10/collision/Base.dae; visual mesh filename=package://ur_description/meshes/ur10/visual/Base.dae
- link forearm_link: geometry collision mesh filename=package://ur_description/meshes/ur10/collision/Forearm.dae; visual mesh filename=package://ur_description/meshes/ur10/visual/Forearm.dae
- link shoulder_link: geometry collision mesh filename=package://ur_description/meshes/ur10/collision/Shoulder.dae; visual mesh filename=package://ur_description/meshes/ur10/visual/Shoulder.dae
- link upper_arm_link: geometry collision mesh filename=package://ur_description/meshes/ur10/collision/UpperArm.dae; visual mesh filename=package://ur_description/meshes/ur10/visual/UpperArm.dae
- link wrist_1_link: geometry collision mesh filename=package://ur_description/meshes/ur10/collision/Wrist1.dae; visual mesh filename=package://ur_description/meshes/ur10/visual/Wrist1.dae
- link wrist_2_link: geometry collision mesh filename=package://ur_description/meshes/ur10/collision/Wrist2.dae; visual mesh filename=package://ur_description/meshes/ur10/visual/Wrist2.dae
- link wrist_3_link: geometry collision mesh filename=package://ur_description/meshes/ur10/collision/Wrist3.dae; visual mesh filename=package://ur_description/meshes/ur10/visual/Wrist3.dae
Joints:
- joint elbow_joint: axis 0.0 1.0 0.0 -> 0 1 0
- joint shoulder_lift_joint: axis 0.0 1.0 0.0 -> 0 1 0
- joint shoulder_pan_joint: axis 0.0 0.0 1.0 -> 0 0 1
- joint wrist_1_joint: axis 0.0 1.0 0.0 -> 0 1 0
- joint wrist_2_joint: axis 0.0 0.0 1.0 -> 0 0 1
- joint wrist_3_joint: axis 0.0 1.0 0.0 -> 0 1 0

Commit message: re-generate urdf-files from latest xacro-files

File: ur_description/urdf/ur10_joint_limited_robot.urdf (robot description, URDF)
Before this commit: robot ur10, 9 links, 8 joints
Links:
- link base_link: geometry collision mesh filename=package://ur_description/meshes/ur10/collision/base.stl; visual mesh filename=package://ur_description/meshes/ur10/visual/Base.dae
- link ee_link: geometry collision box size=0.01 0.01 0.01
- link forearm_link: geometry collision mesh filename=package://ur_description/meshes/ur10/collision/forearm.stl; visual mesh filename=package://ur_description/meshes/ur10/visual/Forearm.dae
- link shoulder_link: geometry collision mesh filename=package://ur_description/meshes/ur10/collision/shoulder.stl; visual mesh filename=package://ur_description/meshes/ur10/visual/Shoulder.dae
- link upper_arm_link: geometry collision mesh filename=package://ur_description/meshes/ur10/collision/upper_arm.stl; visual mesh filename=package://ur_description/meshes/ur10/visual/UpperArm.dae
- link wrist_1_link: geometry collision mesh filename=package://ur_description/meshes/ur10/collision/wrist_1.stl; visual mesh filename=package://ur_description/meshes/ur10/visual/Wrist1.dae
- link wrist_2_link: geometry collision mesh filename=package://ur_description/meshes/ur10/collision/wrist_2.stl; visual mesh filename=package://ur_description/meshes/ur10/visual/Wrist2.dae
- link wrist_3_link: geometry collision mesh filename=package://ur_description/meshes/ur10/collision/wrist_3.stl; visual mesh filename=package://ur_description/meshes/ur10/visual/Wrist3.dae

File: ur_description/urdf/ur10_robot.urdf (robot description, URDF)
Before this commit: robot ur10, 9 links, 8 joints
Links:
- link base_link: geometry collision mesh filename=package://ur_description/meshes/ur10/collision/base.stl; visual mesh filename=package://ur_description/meshes/ur10/visual/Base.dae
- link ee_link: geometry collision box size=0.01 0.01 0.01
- link forearm_link: geometry collision mesh filename=package://ur_description/meshes/ur10/collision/forearm.stl; visual mesh filename=package://ur_description/meshes/ur10/visual/Forearm.dae
- link shoulder_link: geometry collision mesh filename=package://ur_description/meshes/ur10/collision/shoulder.stl; visual mesh filename=package://ur_description/meshes/ur10/visual/Shoulder.dae
- link upper_arm_link: geometry collision mesh filename=package://ur_description/meshes/ur10/collision/upper_arm.stl; visual mesh filename=package://ur_description/meshes/ur10/visual/UpperArm.dae
- link wrist_1_link: geometry collision mesh filename=package://ur_description/meshes/ur10/collision/wrist_1.stl; visual mesh filename=package://ur_description/meshes/ur10/visual/Wrist1.dae
- link wrist_2_link: geometry collision mesh filename=package://ur_description/meshes/ur10/collision/wrist_2.stl; visual mesh filename=package://ur_description/meshes/ur10/visual/Wrist2.dae
- link wrist_3_link: geometry collision mesh filename=package://ur_description/meshes/ur10/collision/wrist_3.stl; visual mesh filename=package://ur_description/meshes/ur10/visual/Wrist3.dae

File: ur_description/urdf/ur5_joint_limited_robot.urdf (robot description, URDF)
Before this commit: robot ur5, 9 links, 8 joints
Links:
- link base_link: geometry collision mesh filename=package://ur_description/meshes/ur5/collision/base.stl; visual mesh filename=package://ur_description/meshes/ur5/visual/Base.dae
- link ee_link: geometry collision box size=0.01 0.01 0.01
- link forearm_link: geometry collision mesh filename=package://ur_description/meshes/ur5/collision/forearm.stl; visual mesh filename=package://ur_description/meshes/ur5/visual/Forearm.dae
- link shoulder_link: geometry collision mesh filename=package://ur_description/meshes/ur5/collision/shoulder.stl; visual mesh filename=package://ur_description/meshes/ur5/visual/Shoulder.dae
- link upper_arm_link: geometry collision mesh filename=package://ur_description/meshes/ur5/collision/upper_arm.stl; visual mesh filename=package://ur_description/meshes/ur5/visual/UpperArm.dae
- link wrist_1_link: geometry collision mesh filename=package://ur_description/meshes/ur5/collision/wrist_1.stl; visual mesh filename=package://ur_description/meshes/ur5/visual/Wrist1.dae
- link wrist_2_link: geometry collision mesh filename=package://ur_description/meshes/ur5/collision/wrist_2.stl; visual mesh filename=package://ur_description/meshes/ur5/visual/Wrist2.dae
- link wrist_3_link: geometry collision mesh filename=package://ur_description/meshes/ur5/collision/wrist_3.stl; visual mesh filename=package://ur_description/meshes/ur5/visual/Wrist3.dae

File: ur_description/urdf/ur5_robot.urdf (robot description, URDF)
Before this commit: robot ur5, 9 links, 8 joints
Links:
- link base_link: geometry collision mesh filename=package://ur_description/meshes/ur5/collision/base.stl; visual mesh filename=package://ur_description/meshes/ur5/visual/Base.dae
- link ee_link: geometry collision box size=0.01 0.01 0.01
- link forearm_link: geometry collision mesh filename=package://ur_description/meshes/ur5/collision/forearm.stl; visual mesh filename=package://ur_description/meshes/ur5/visual/Forearm.dae
- link shoulder_link: geometry collision mesh filename=package://ur_description/meshes/ur5/collision/shoulder.stl; visual mesh filename=package://ur_description/meshes/ur5/visual/Shoulder.dae
- link upper_arm_link: geometry collision mesh filename=package://ur_description/meshes/ur5/collision/upper_arm.stl; visual mesh filename=package://ur_description/meshes/ur5/visual/UpperArm.dae
- link wrist_1_link: geometry collision mesh filename=package://ur_description/meshes/ur5/collision/wrist_1.stl; visual mesh filename=package://ur_description/meshes/ur5/visual/Wrist1.dae
- link wrist_2_link: geometry collision mesh filename=package://ur_description/meshes/ur5/collision/wrist_2.stl; visual mesh filename=package://ur_description/meshes/ur5/visual/Wrist2.dae
- link wrist_3_link: geometry collision mesh filename=package://ur_description/meshes/ur5/collision/wrist_3.stl; visual mesh filename=package://ur_description/meshes/ur5/visual/Wrist3.dae
