Commit message: use new transmission interfaces

File: ur_description/urdf/ur10.transmission.xacro (robot description, xacro)
@@ -2,33 +2,51 @@
 <robot xmlns:xacro="http://www.ros.org/wiki/xacro">
 	<xacro:macro name="ur10_arm_transmission" params="prefix">
-		<transmission name="shoulder_pan_trans" type="pr2_mechanism_model/SimpleTransmission">
-			<actuator name="shoulder_pan_motor"/>
+		<transmission name="${prefix}shoulder_pan_trans">
+			<type>transmission_interface/SimpleTransmission</type>
 			<joint name="${prefix}shoulder_pan_joint"/>
-			<mechanicalReduction>1</mechanicalReduction>
+			<actuator name="${prefix}shoulder_pan_motor">
+				<hardwareInterface>EffortJointInterface</hardwareInterface>
+				<mechanicalReduction>1</mechanicalReduction>
+			</actuator>
 		</transmission>
-		<transmission name="shoulder_lift_trans" type="pr2_mechanism_model/SimpleTransmission">
-			<actuator name="shoulder_lift_motor"/>
+		<transmission name="${prefix}shoulder_lift_trans">
+			<type>transmission_interface/SimpleTransmission</type>
 			<joint name="${prefix}shoulder_lift_joint"/>
-			<mechanicalReduction>1</mechanicalReduction>
+			<actuator name="${prefix}shoulder_lift_motor">
+				<hardwareInterface>EffortJointInterface</hardwareInterface>
+				<mechanicalReduction>1</mechanicalReduction>
+			</actuator>
 		</transmission>
-		<transmission name="elbow_trans" type="pr2_mechanism_model/SimpleTransmission">
-			<actuator name="elbow_motor"/>
+		<transmission name="${prefix}elbow_trans">
+			<type>transmission_interface/SimpleTransmission</type>
 			<joint name="${prefix}elbow_joint"/>
-			<mechanicalReduction>1</mechanicalReduction>
+			<actuator name="${prefix}elbow_motor">
+				<hardwareInterface>EffortJointInterface</hardwareInterface>
+				<mechanicalReduction>1</mechanicalReduction>
+			</actuator>
 		</transmission>
-		<transmission name="wrist_1_trans" type="pr2_mechanism_model/SimpleTransmission">
-			<actuator name="wrist_1_motor"/>
+		<transmission name="${prefix}wrist_1_trans">
+			<type>transmission_interface/SimpleTransmission</type>
 			<joint name="${prefix}wrist_1_joint"/>
-			<mechanicalReduction>1</mechanicalReduction>
+			<actuator name="${prefix}wrist_1_motor">
+				<hardwareInterface>EffortJointInterface</hardwareInterface>
+				<mechanicalReduction>1</mechanicalReduction>
+			</actuator>
 		</transmission>
-		<transmission name="wrist_2_trans" type="pr2_mechanism_model/SimpleTransmission">
-			<actuator name="wrist_2_motor"/>
+		<transmission name="${prefix}wrist_2_trans">
+			<type>transmission_interface/SimpleTransmission</type>
 			<joint name="${prefix}wrist_2_joint"/>
-			<mechanicalReduction>1</mechanicalReduction>
+			<actuator name="${prefix}wrist_2_motor">
+				<hardwareInterface>EffortJointInterface</hardwareInterface>
+				<mechanicalReduction>1</mechanicalReduction>
+			</actuator>
 		</transmission>
-		<transmission name="wrist_3_trans" type="pr2_mechanism_model/SimpleTransmission">
-			<actuator name="wrist_3_motor"/>
+		<transmission name="${prefix}wrist_3_trans">
+			<type>transmission_interface/SimpleTransmission</type>
 			<joint name="${prefix}wrist_3_joint"/>
-			<mechanicalReduction>1</mechanicalReduction>
+			<actuator name="${prefix}wrist_3_motor">
+				<hardwareInterface>EffortJointInterface</hardwareInterface>
+				<mechanicalReduction>1</mechanicalReduction>
+			</actuator>
 		</transmission>
 	</xacro:macro>

File: ur_description/urdf/ur5.transmission.xacro (robot description, xacro)
@@ -1,34 +1,52 @@
 <?xml version="1.0"?>
 <robot xmlns:xacro="http://www.ros.org/wiki/xacro">
-	<xacro:macro name="ur5_arm_transmission" params="name">
-		<transmission name="shoulder_pan_trans" type="pr2_mechanism_model/SimpleTransmission">
-			<actuator name="shoulder_pan_motor"/>
-			<joint name="${name}shoulder_pan_joint"/>
-			<mechanicalReduction>1</mechanicalReduction>
+	<xacro:macro name="ur5_arm_transmission" params="prefix">
+		<transmission name="${prefix}shoulder_pan_trans">
+			<type>transmission_interface/SimpleTransmission</type>
+			<joint name="${prefix}shoulder_pan_joint"/>
+			<actuator name="${prefix}shoulder_pan_motor">
+				<hardwareInterface>EffortJointInterface</hardwareInterface>
+				<mechanicalReduction>1</mechanicalReduction>
+			</actuator>
 		</transmission>
-		<transmission name="shoulder_lift_trans" type="pr2_mechanism_model/SimpleTransmission">
-			<actuator name="shoulder_lift_motor"/>
-			<joint name="${name}shoulder_lift_joint"/>
-			<mechanicalReduction>1</mechanicalReduction>
+		<transmission name="${prefix}shoulder_lift_trans">
+			<type>transmission_interface/SimpleTransmission</type>
+			<joint name="${prefix}shoulder_lift_joint"/>
+			<actuator name="${prefix}shoulder_lift_motor">
+				<hardwareInterface>EffortJointInterface</hardwareInterface>
+				<mechanicalReduction>1</mechanicalReduction>
+			</actuator>
 		</transmission>
-		<transmission name="elbow_trans" type="pr2_mechanism_model/SimpleTransmission">
-			<actuator name="elbow_motor"/>
-			<joint name="${name}elbow_joint"/>
-			<mechanicalReduction>1</mechanicalReduction>
+		<transmission name="${prefix}elbow_trans">
+			<type>transmission_interface/SimpleTransmission</type>
+			<joint name="${prefix}elbow_joint"/>
+			<actuator name="${prefix}elbow_motor">
+				<hardwareInterface>EffortJointInterface</hardwareInterface>
+				<mechanicalReduction>1</mechanicalReduction>
+			</actuator>
 		</transmission>
-		<transmission name="wrist_1_trans" type="pr2_mechanism_model/SimpleTransmission">
-			<actuator name="wrist_1_motor"/>
-			<joint name="${name}wrist_1_joint"/>
-			<mechanicalReduction>1</mechanicalReduction>
+		<transmission name="${prefix}wrist_1_trans">
+			<type>transmission_interface/SimpleTransmission</type>
+			<joint name="${prefix}wrist_1_joint"/>
+			<actuator name="${prefix}wrist_1_motor">
+				<hardwareInterface>EffortJointInterface</hardwareInterface>
+				<mechanicalReduction>1</mechanicalReduction>
+			</actuator>
 		</transmission>
-		<transmission name="wrist_2_trans" type="pr2_mechanism_model/SimpleTransmission">
-			<actuator name="wrist_2_motor"/>
-			<joint name="${name}wrist_2_joint"/>
-			<mechanicalReduction>1</mechanicalReduction>
+		<transmission name="${prefix}wrist_2_trans">
+			<type>transmission_interface/SimpleTransmission</type>
+			<joint name="${prefix}wrist_2_joint"/>
+			<actuator name="${prefix}wrist_2_motor">
+				<hardwareInterface>EffortJointInterface</hardwareInterface>
+				<mechanicalReduction>1</mechanicalReduction>
+			</actuator>
 		</transmission>
-		<transmission name="wrist_3_trans" type="pr2_mechanism_model/SimpleTransmission">
-			<actuator name="wrist_3_motor"/>
-			<joint name="${name}wrist_3_joint"/>
-			<mechanicalReduction>1</mechanicalReduction>
+		<transmission name="${prefix}wrist_3_trans">
+			<type>transmission_interface/SimpleTransmission</type>
+			<joint name="${prefix}wrist_3_joint"/>
+			<actuator name="${prefix}wrist_3_motor">
+				<hardwareInterface>EffortJointInterface</hardwareInterface>
+				<mechanicalReduction>1</mechanicalReduction>
+			</actuator>
 		</transmission>
 	</xacro:macro>

Commit message: various fixes

File: ur_description/urdf/ur10.transmission.xacro (robot description, xacro)
@@ -2,28 +2,28 @@
 <robot xmlns:xacro="http://www.ros.org/wiki/xacro">
   <xacro:macro name="ur10_arm_transmission" params="prefix">
-		<transmission name="${prefix}shoulder_pan_trans" type="sr_mechanism_model/SimpleTransmission">
-			<actuator name="${prefix}shoulder_pan_motor"/>
-			<joint name="${prefix}shoulder_pan_joint"/>
-		</transmission>
-		<transmission name="${prefix}shoulder_lift_trans" type="sr_mechanism_model/SimpleTransmission">
-			<actuator name="${prefix}shoulder_lift_motor"/>
-			<joint name="${prefix}shoulder_lift_joint"/>
-		</transmission>
-		<transmission name="${prefix}elbow_trans" type="sr_mechanism_model/SimpleTransmission">
-			<actuator name="${prefix}elbow_motor"/>
-			<joint name="${prefix}elbow_joint"/>
-		</transmission>
-		<transmission name="${prefix}wrist_1_trans" type="sr_mechanism_model/SimpleTransmission">
-			<actuator name="${prefix}wrist_1_motor"/>
-			<joint name="${prefix}wrist_1_joint"/>
-		</transmission>
-		<transmission name="${prefix}wrist_2_trans" type="sr_mechanism_model/SimpleTransmission">
-			<actuator name="${prefix}wrist_2_motor"/>
-			<joint name="${prefix}wrist_2_joint"/>
-		</transmission>
-		<transmission name="${prefix}wrist_3_trans" type="sr_mechanism_model/SimpleTransmission">
-			<actuator name="${prefix}wrist_3_motor"/>
-			<joint name="${prefix}wrist_3_joint"/>
-		</transmission>
+    <transmission name="${prefix}shoulder_pan_trans" type="sr_mechanism_model/NullTransmission">
+      <actuator name="${prefix}shoulder_pan_motor"/>
+      <joint name="${prefix}shoulder_pan_joint"/>
+    </transmission>
+    <transmission name="${prefix}shoulder_lift_trans" type="sr_mechanism_model/NullTransmission">
+      <actuator name="${prefix}shoulder_lift_motor"/>
+      <joint name="${prefix}shoulder_lift_joint"/>
+    </transmission>
+    <transmission name="${prefix}elbow_trans" type="sr_mechanism_model/NullTransmission">
+      <actuator name="${prefix}elbow_motor"/>
+      <joint name="${prefix}elbow_joint"/>
+    </transmission>
+    <transmission name="${prefix}wrist_1_trans" type="sr_mechanism_model/NullTransmission">
+      <actuator name="${prefix}wrist_1_motor"/>
+      <joint name="${prefix}wrist_1_joint"/>
+    </transmission>
+    <transmission name="${prefix}wrist_2_trans" type="sr_mechanism_model/NullTransmission">
+      <actuator name="${prefix}wrist_2_motor"/>
+      <joint name="${prefix}wrist_2_joint"/>
+    </transmission>
+    <transmission name="${prefix}wrist_3_trans" type="sr_mechanism_model/NullTransmission">
+      <actuator name="${prefix}wrist_3_motor"/>
+      <joint name="${prefix}wrist_3_joint"/>
+    </transmission>
   </xacro:macro>
 </robot>
