Commit message: Reorganized meshes to include both collision and visual messhes (like other ROS-I robots).  Modified urdf xacro to include new models.  Removed extra robot pedestal link from urdf (urdfs should only include the robot itself).

File: ur_description/urdf/ur5.urdf.xacro (robot description, xacro)
@@ -6,14 +6,14 @@
 <include filename="$(find ur_description)/urdf/ur5.transmission.xacro" />
   <include filename="$(find ur_description)/urdf/ur5.gazebo.xacro" />
-		<!--
-		DH for UR5:
-		a = [0.00000, -0.42500, -0.39225,  0.00000,  0.00000,  0.0000]
-		d = [0.089159,  0.00000,  0.00000,  0.10915,  0.09465,  0.0823]
-		alpha = [ 1.570796327, 0, 0, 1.570796327, -1.570796327, 0 ]
-		q_home_offset = [0, -1.570796327, 0, -1.570796327, 0, 0]
-		joint_direction = [-1, -1, 1, 1, 1, 1]
-		mass = [3.7000, 8.3930, 2.2750, 1.2190, 1.2190, 0.1879]
-		center_of_mass = [ [0, -0.02561, 0.00193], [0.2125, 0, 0.11336], [0.11993, 0.0, 0.0265], [0, -0.0018, 0.01634], [0, 0.0018,0.01634], [0, 0, -0.001159] ]
-		-->
+<!--
+DH for UR5:
+a = [0.00000, -0.42500, -0.39225,  0.00000,  0.00000,  0.0000]
+d = [0.089159,  0.00000,  0.00000,  0.10915,  0.09465,  0.0823]
+alpha = [ 1.570796327, 0, 0, 1.570796327, -1.570796327, 0 ]
+q_home_offset = [0, -1.570796327, 0, -1.570796327, 0, 0]
+joint_direction = [-1, -1, 1, 1, 1, 1]
+mass = [3.7000, 8.3930, 2.2750, 1.2190, 1.2190, 0.1879]
+center_of_mass = [ [0, -0.02561, 0.00193], [0.2125, 0, 0.11336], [0.11993, 0.0, 0.0265], [0, -0.0018, 0.01634], [0, 0.0018,0.01634], [0, 0, -0.001159] ]
+-->
   <property name="pi" value="3.14159265" />
 <!-- Inertia parameters -->
@@ -45,23 +45,23 @@
   <property name="forearm_radius" value="0.040" />    <!-- manually measured -->
   <property name="wrist_radius" value="0.045" />      <!-- manually measured -->
-<!-- Collision model -->
-  <property name="base_collision_length" value="0.160" />      <!-- manually measured -->
-  <property name="shoulder_collision_length" value="0.200" />  <!-- manually measured -->
-  <property name="shoulder_collision_offset" value="0.035" />  <!-- manually measured -->
-  <property name="elbow_collision_length" value="0.200" />     <!-- manually measured -->
-  <property name="elbow_collision_offset" value="0.035" />     <!-- manually measured -->
 <xacro:macro name="ur5_robot" params="prefix">
-	<link name="${prefix}base_link" >
-		<visual>
-		  <geometry>
-		    <mesh filename="package://ur_description/meshes/ur5/Base.dae" />
-		  </geometry>
-		  <origin xyz="0.0 0.0 0.003" rpy="0.0 0.0 ${3.0 * pi / 4.0}" />
-		</visual>
-		<inertial>
-		  <mass value="${base_mass}" />
-		  <inertia ixx="1.0" ixy="0.0" ixz="0.0" iyy="1.0" iyz="0.0" izz="1.0"/>
-		</inertial>
-	</link>
+  <link name="${prefix}base_link" >
+    <visual>
+      <geometry>
+		    <mesh filename="package://ur_description/meshes/ur5/visual/Base.dae" />
+      </geometry>
+      <origin xyz="0.0 0.0 0.003" rpy="0.0 0.0 ${3.0 * pi / 4.0}" />
+    </visual>
+	<collision>
+      <geometry>
+        <mesh filename="package://ur_description/meshes/ur5/collision/Base.dae" />
+      </geometry>
+      <!-- <origin rpy="0.0 0.0 0.0" xyz="0.0 0.0 -0.009159"/> -->
+    </collision>
+    <inertial>
+      <mass value="${base_mass}" />
+      <inertia ixx="1.0" ixy="0.0" ixz="0.0" iyy="1.0" iyz="0.0" izz="1.0"/>
+    </inertial>
+  </link>
   <joint name="${prefix}shoulder_pan_joint" type="revolute">
     <parent link="${prefix}base_link" />
@@ -75,12 +75,12 @@
     <visual>
       <geometry>
-        <mesh filename="package://ur_description/meshes/ur5/Shoulder.dae" />
-      </geometry>
-    </visual>
-    <collision>
-      <geometry>
-        <cylinder length="${base_collision_length}" radius="${shoulder_radius}"/>
-      </geometry>
-      <origin xyz="0.0 0.0 ${-shoulder_height + (base_collision_length/2.0)}" rpy="0.0 0.0 0.0" />
+        <mesh filename="package://ur_description/meshes/ur5/visual/Shoulder.dae" />
+      </geometry>
+    </visual>
+    <collision>
+      <geometry>
+        <mesh filename="package://ur_description/meshes/ur5/collision/Shoulder.dae" />
+      </geometry>
+      <!-- <origin rpy="0.0 0.0 0.0" xyz="0.0 0.0 -0.009159"/> -->
     </collision>
     <inertial>
@@ -101,5 +101,5 @@
     <visual>
       <geometry>
-        <mesh filename="package://ur_description/meshes/ur5/UpperArm.dae" />
+        <mesh filename="package://ur_description/meshes/ur5/visual/UpperArm.dae" />
       </geometry>
       <origin xyz="0.0 0.0 0.0" rpy="0.0 0.0 0.0" />
@@ -107,7 +107,7 @@
     <collision>
       <geometry>
-        <cylinder length="${upper_arm_length}" radius="${upper_arm_radius}"/>
-      </geometry>
-      <origin xyz="0.0 0.0 ${upper_arm_length/2.0}" rpy="0.0 0.0 0.0" />
+        <mesh filename="package://ur_description/meshes/ur5/collision/UpperArm.dae" />
+      </geometry>
+<!--       <origin rpy="0.0 0.0 0.0" xyz="0.0 0.0 0.2125"/> -->
     </collision>
     <inertial>
@@ -128,12 +128,12 @@
     <visual>
       <geometry>
-        <mesh filename="package://ur_description/meshes/ur5/Forearm.dae" />
-      </geometry>
-    </visual>
-    <collision>
-      <geometry>
-        <cylinder length="${forearm_length}" radius="${forearm_radius}"/>
-      </geometry>
-      <origin xyz="0.0 0.0 ${forearm_length/2.0}" rpy="0.0 0.0 0.0" />
+        <mesh filename="package://ur_description/meshes/ur5/visual/Forearm.dae" />
+      </geometry>
+    </visual>
+    <collision>
+      <geometry>
+        <mesh filename="package://ur_description/meshes/ur5/collision/Forearm.dae" />
+      </geometry>
+<!--       <origin rpy="0.0 0.0 0.0" xyz="0.0 0.0 0.196125"/> -->
     </collision>
     <inertial>
@@ -148,5 +148,5 @@
     <origin xyz="0.0 0.0 ${forearm_length}" rpy="0.0 ${pi / 2.0} 0.0" />
     <axis xyz="0 1 0" />
-    <limit lower="${-2.0 * pi}" upper="${2.0 * pi}" effort="10.0" velocity="${pi}"/>
+    <limit lower="${-1.0 * pi}" upper="${0.25 * pi}" effort="10.0" velocity="${pi}"/>
     <dynamics damping="10" friction="0.1"/>
   </joint>
@@ -154,5 +154,5 @@
     <visual>
       <geometry>
-        <mesh filename="package://ur_description/meshes/ur5/Wrist1.dae" />
+        <mesh filename="package://ur_description/meshes/ur5/visual/Wrist1.dae" />
       </geometry>
       <origin xyz="0.0 ${wrist_1_length} 0.0" rpy="0.0 ${pi / 2.0} 0.0" />
@@ -160,7 +160,7 @@
     <collision>
       <geometry>
-        <cylinder length="${1.6*wrist_1_length}" radius="${wrist_radius}"/>
-      </geometry>
-      <origin xyz="0.0 ${0.25*wrist_1_length} 0.0" rpy="${-pi/2.0} 0.0 0.0" />
+        <mesh filename="package://ur_description/meshes/ur5/collision/Wrist1.dae" />
+      </geometry>
+      <origin rpy="0.0 1.570796325 0.0" xyz="0.0 0.093 0.0"/>
     </collision>
     <inertial>
@@ -175,5 +175,5 @@
     <origin xyz="0.0 ${wrist_1_length} 0.0" rpy="0.0 0.0 0.0" />
     <axis xyz="0 0 1" />
-    <limit lower="${-2.0 * pi}" upper="${2.0 * pi}" effort="10.0" velocity="${pi}"/>
+    <limit lower="${-1.0 * pi}" upper="${1.0 * pi}" effort="10.0" velocity="${pi}"/>
     <dynamics damping="10" friction="0.1"/>
   </joint>
@@ -181,5 +181,5 @@
     <visual>
       <geometry>
-        <mesh filename="package://ur_description/meshes/ur5/Wrist2.dae" />
+        <mesh filename="package://ur_description/meshes/ur5/visual/Wrist2.dae" />
       </geometry>
       <origin xyz="0.0 0.0 ${wrist_2_length}" rpy="0.0 0.0 0.0" />
@@ -187,7 +187,7 @@
     <collision>
       <geometry>
-        <cylinder length="${1.6*wrist_2_length}" radius="${wrist_radius}"/>
-      </geometry>
-      <origin xyz="0.0 0.0 ${0.25*wrist_2_length}" rpy="0.0 0.0 0.0" />
+        <mesh filename="package://ur_description/meshes/ur5/collision/Wrist2.dae" />
+      </geometry>
+       <origin rpy="0.0 0.0 0.0" xyz="0.0 0.0 0.09465"/>
     </collision>
     <inertial>
@@ -202,5 +202,5 @@
     <origin xyz="0.0 0.0 ${wrist_2_length}" rpy="0.0 0.0 0.0" />
     <axis xyz="0 1 0" />
-    <limit lower="${-2.0 * pi}" upper="${2.0 * pi}" effort="10.0" velocity="${pi}"/>
+    <limit lower="${-1.0 * pi}" upper="${1.0 * pi}" effort="10.0" velocity="${pi}"/>
     <dynamics damping="10" friction="0.1"/>
   </joint>
@@ -208,12 +208,11 @@
     <visual>
       <geometry>
-        <mesh filename="package://ur_description/meshes/ur5/Wrist3.dae" />
-      </geometry>
-    </visual>
-    <collision>
-      <geometry>
-        <cylinder length="${1.65*wrist_3_length}" radius="${wrist_radius}"/>
-      </geometry>
-      <origin xyz="0.0 ${0.15 * wrist_3_length} 0.0" rpy="${-pi/2.0} 0.0 0.0" />
+        <mesh filename="package://ur_description/meshes/ur5/visual/Wrist3.dae" />
+      </geometry>
+    </visual>
+    <collision>
+      <geometry>
+        <mesh filename="package://ur_description/meshes/ur5/collision/Wrist3.dae" />
+      </geometry>
     </collision>
     <inertial>
@@ -256,6 +255,8 @@
   </link>
   -->
-  <xacro:ur5_arm_transmission name="${prefix}" />
-  <xacro:ur5_arm_gazebo name="${prefix}" />
+  <xacro:ur_arm_transmission name="${prefix}" />
+  <gazebo reference="universal_robot">
+    <material>Gazebo/Blue</material>
+  </gazebo>
 </xacro:macro>
 </robot>

File: ur_description/urdf/ur5_robot.urdf.xacro (robot description, xacro)
@@ -10,33 +10,6 @@
   <!-- ur5 -->
   <include filename="$(find ur_description)/urdf/ur5.urdf.xacro" />
-  <!-- foot for arm -->
-	<link name="base_link">
-		<inertial>
-		   <origin xyz="0 0 -10" rpy="0 0 0"/>
-		   <mass value="1000.0"/>
-		   <inertia ixx="100.0"  ixy="0"  ixz="0" iyy="100.0" iyz="0" izz="100.0" />
-		</inertial>
-		<visual>
-		   <origin xyz="0 0 0.25" rpy="0 0 0" />
-		   <geometry>
-			  <cylinder radius="0.1" length="0.5"/>
-		   </geometry>
-		   <material name="Grey" />
-		</visual>
-		<collision>
-		   <origin xyz="0 0 0.25" rpy="0 0 0" />
-		   <geometry>
-			  <cylinder radius="0.1" length="0.5"/>
-		   </geometry>
-		</collision>
-	</link>
-	<!-- joint between base_link and ur_base_link -->
-	<joint name="arm_base_joint" type="fixed" >
-		<origin xyz="0 0 0.5" rpy="0 0 0" />
-		<parent link="base_link" />
-		<child link="arm_base_link" />
-	</joint>
   <!-- arm -->
-  <xacro:ur5_robot prefix="arm_">
+  <xacro:ur5_robot prefix="">
   </xacro:ur5_robot>
 </robot>

Commit message: Update ur5.urdf.xacro
Corrected effort thresholds and friction values for UR5 urdf.

File: ur_description/urdf/ur5.urdf.xacro (robot description, xacro)
@@ -70,6 +70,6 @@
     <origin xyz="0.0 0.0 ${shoulder_height}" rpy="0.0 0.0 0.0" />
     <axis xyz="0 0 1" />
-    <limit lower="${-2.0 * pi}" upper="${2.0 * pi}" effort="10.0" velocity="${pi}"/>
-    <dynamics damping="10" friction="0.1"/>
+    <limit lower="${-2.0 * pi}" upper="${2.0 * pi}" effort="150.0" velocity="${pi}"/>
+    <dynamics damping="0.4" friction="0.0"/>
   </joint>
   <link name="${prefix}shoulder_link">
@@ -96,6 +96,6 @@
     <origin xyz="0.0 ${shoulder_offset} 0.0" rpy="0.0 ${pi / 2.0} 0.0" />
     <axis xyz="0 1 0" />
-    <limit lower="${-2.0 * pi}" upper="${2.0 * pi}" effort="10.0" velocity="${pi}"/>
-    <dynamics damping="10" friction="0.1"/>
+    <limit lower="${-2.0 * pi}" upper="${2.0 * pi}" effort="150.0" velocity="${pi}"/>
+    <dynamics damping="0.4" friction="0.0"/>
   </joint>
   <link name="${prefix}upper_arm_link">
@@ -123,6 +123,6 @@
     <origin xyz="0.0 ${-elbow_offset} ${upper_arm_length}" rpy="0.0 0.0 0.0" />
     <axis xyz="0 1 0" />
-    <limit lower="${-2.0 * pi}" upper="${2.0 * pi}" effort="10.0" velocity="${pi}"/>
-    <dynamics damping="10" friction="0.1"/>
+    <limit lower="${-2.0 * pi}" upper="${2.0 * pi}" effort="150.0" velocity="${pi}"/>
+    <dynamics damping="0.4" friction="0.0"/>
   </joint>
   <link name="${prefix}forearm_link">
@@ -149,6 +149,6 @@
     <origin xyz="0.0 0.0 ${forearm_length}" rpy="0.0 ${pi / 2.0} 0.0" />
     <axis xyz="0 1 0" />
-    <limit lower="${-1.0 * pi}" upper="${0.25 * pi}" effort="10.0" velocity="${pi}"/>
-    <dynamics damping="10" friction="0.1"/>
+    <limit lower="${-1.0 * pi}" upper="${0.25 * pi}" effort="28.0" velocity="${pi}"/>
+    <dynamics damping="0.3" friction="0.0"/>
   </joint>
   <link name="${prefix}wrist_1_link">
@@ -176,6 +176,6 @@
     <origin xyz="0.0 ${wrist_1_length} 0.0" rpy="0.0 0.0 0.0" />
     <axis xyz="0 0 1" />
-    <limit lower="${-1.0 * pi}" upper="${1.0 * pi}" effort="10.0" velocity="${pi}"/>
-    <dynamics damping="10" friction="0.1"/>
+    <limit lower="${-1.0 * pi}" upper="${1.0 * pi}" effort="28.0" velocity="${pi}"/>
+    <dynamics damping="0.3" friction="0.0"/>
   </joint>
   <link name="${prefix}wrist_2_link">
@@ -203,6 +203,6 @@
     <origin xyz="0.0 0.0 ${wrist_2_length}" rpy="0.0 0.0 0.0" />
     <axis xyz="0 1 0" />
-    <limit lower="${-1.0 * pi}" upper="${1.0 * pi}" effort="10.0" velocity="${pi}"/>
-    <dynamics damping="10" friction="0.1"/>
+    <limit lower="${-1.0 * pi}" upper="${1.0 * pi}" effort="28.0" velocity="${pi}"/>
+    <dynamics damping="0.3" friction="0.0"/>
   </joint>
   <link name="${prefix}wrist_3_link">

Commit message: remove ee_link - as in ur10

File: ur_description/urdf/ur5.urdf.xacro (robot description, xacro)
@@ -220,10 +220,4 @@
     </inertial>
   </link>
-  <joint name="${prefix}ee_fixed_joint" type="fixed">
-    <parent link="${prefix}wrist_3_link" />
-    <child link = "${prefix}ee_link" />
-    <origin xyz="0.0 ${wrist_3_length} 0.0" rpy="0.0 0.0 ${pi/2.0}" />
-  </joint>
-  <link name="${prefix}ee_link" />
   <xacro:ur5_arm_transmission prefix="${prefix}" />
   <xacro:ur5_arm_gazebo prefix="${prefix}" />

Commit message: [UR5_wobbling] Fixed wobbling of the UR5 (UR10 untouched).

File: ur_description/urdf/ur5.urdf.xacro (robot description, xacro)
@@ -59,5 +59,5 @@
     <inertial>
       <mass value="${base_mass}" />
-      <inertia ixx="1.0" ixy="0.0" ixz="0.0" iyy="1.0" iyz="0.0" izz="1.0"/>
+      <inertia ixx="0.002" ixy="0.0" ixz="0.0" iyy="0.02" iyz="0.0" izz="0.002"/>
     </inertial>
   </link>
@@ -68,5 +68,5 @@
     <axis xyz="0 0 1" />
     <limit lower="${-2.0 * pi}" upper="${2.0 * pi}" effort="150.0" velocity="${pi}"/>
-    <dynamics damping="0.4" friction="0.0"/>
+    <dynamics damping="0.5" friction="0.0"/>
   </joint>
   <link name="${prefix}shoulder_link">
@@ -84,5 +84,5 @@
     <inertial>
       <mass value="${shoulder_mass}" />
-      <inertia ixx="1.0" ixy="0.0" ixz="0.0" iyy="1.0" iyz="0.0" izz="1.0"/>
+      <inertia ixx="0.002" ixy="0.0" ixz="0.0" iyy="0.02" iyz="0.0" izz="0.002"/>
       <origin xyz="${shoulder_cog}" rpy="0.0 0.0 0.0" />
     </inertial>
@@ -94,5 +94,5 @@
     <axis xyz="0 1 0" />
     <limit lower="${-2.0 * pi}" upper="${2.0 * pi}" effort="150.0" velocity="${pi}"/>
-    <dynamics damping="0.4" friction="0.0"/>
+    <dynamics damping="0.5" friction="0.0"/>
   </joint>
   <link name="${prefix}upper_arm_link">
@@ -111,5 +111,5 @@
     <inertial>
       <mass value="${upper_arm_mass}" />
-      <inertia ixx="1.0" ixy="0.0" ixz="0.0" iyy="1.0" iyz="0.0" izz="1.0"/>
+      <inertia ixx="0.002" ixy="0.0" ixz="0.0" iyy="0.02" iyz="0.0" izz="0.002"/>
       <origin xyz="${upper_arm_cog}" rpy="0.0 0.0 0.0" />
     </inertial>
@@ -121,5 +121,5 @@
     <axis xyz="0 1 0" />
     <limit lower="${-2.0 * pi}" upper="${2.0 * pi}" effort="150.0" velocity="${pi}"/>
-    <dynamics damping="0.4" friction="0.0"/>
+    <dynamics damping="0.5" friction="0.0"/>
   </joint>
   <link name="${prefix}forearm_link">
@@ -138,5 +138,5 @@
       <mass value="${forearm_mass}" />
       <origin xyz="${forearm_cog}" rpy="0.0 0.0 0.0" />
-      <inertia ixx="1.0" ixy="0.0" ixz="0.0" iyy="1.0" iyz="0.0" izz="1.0"/>
+      <inertia ixx="0.002" ixy="0.0" ixz="0.0" iyy="0.02" iyz="0.0" izz="0.002"/>
     </inertial>
   </link>
@@ -147,5 +147,5 @@
     <axis xyz="0 1 0" />
     <limit lower="${-1.0 * pi}" upper="${0.25 * pi}" effort="28.0" velocity="${pi}"/>
-    <dynamics damping="0.3" friction="0.0"/>
+    <dynamics damping="0.5" friction="0.0"/>
   </joint>
   <link name="${prefix}wrist_1_link">
@@ -165,5 +165,5 @@
       <mass value="${wrist_1_mass}" />
       <origin xyz="${wrist_1_cog}" rpy="0.0 0.0 0.0" />
-      <inertia ixx="1.0" ixy="0.0" ixz="0.0" iyy="1.0" iyz="0.0" izz="1.0"/>
+      <inertia ixx="0.002" ixy="0.0" ixz="0.0" iyy="0.02" iyz="0.0" izz="0.002"/>
     </inertial>
   </link>
@@ -174,5 +174,5 @@
     <axis xyz="0 0 1" />
     <limit lower="${-1.0 * pi}" upper="${1.0 * pi}" effort="28.0" velocity="${pi}"/>
-    <dynamics damping="0.3" friction="0.0"/>
+    <dynamics damping="0.5" friction="0.0"/>
   </joint>
   <link name="${prefix}wrist_2_link">
@@ -192,5 +192,5 @@
       <mass value="${wrist_2_mass}" />
       <origin xyz="${wrist_2_cog}" rpy="0.0 0.0 0.0" />
-      <inertia ixx="1.0" ixy="0.0" ixz="0.0" iyy="1.0" iyz="0.0" izz="1.0"/>
+      <inertia ixx="0.002" ixy="0.0" ixz="0.0" iyy="0.02" iyz="0.0" izz="0.002"/>
     </inertial>
   </link>
@@ -201,5 +201,5 @@
     <axis xyz="0 1 0" />
     <limit lower="${-1.0 * pi}" upper="${1.0 * pi}" effort="28.0" velocity="${pi}"/>
-    <dynamics damping="0.3" friction="0.0"/>
+    <dynamics damping="0.5" friction="0.0"/>
   </joint>
   <link name="${prefix}wrist_3_link">
@@ -217,5 +217,5 @@
       <mass value="${wrist_3_mass}" />
       <origin xyz="${wrist_3_cog}" rpy="0.0 0.0 0.0" />
-      <inertia ixx="1.0" ixy="0.0" ixz="0.0" iyy="1.0" iyz="0.0" izz="1.0"/>
+      <inertia ixx="0.002" ixy="0.0" ixz="0.0" iyy="0.02" iyz="0.0" izz="0.002"/>
     </inertial>
   </link>

File: ur_description/urdf/ur5_joint_limited.urdf.xacro (robot description, xacro)
@@ -59,5 +59,5 @@
     <inertial>
       <mass value="${base_mass}" />
-      <inertia ixx="1.0" ixy="0.0" ixz="0.0" iyy="1.0" iyz="0.0" izz="1.0"/>
+      <inertia ixx="0.002" ixy="0.0" ixz="0.0" iyy="0.02" iyz="0.0" izz="0.002"/>
     </inertial>
   </link>
@@ -68,5 +68,5 @@
     <axis xyz="0 0 1" />
     <limit lower="${-pi}" upper="${pi}" effort="150.0" velocity="${pi}"/>
-    <dynamics damping="0.4" friction="0.0"/>
+    <dynamics damping="0.5" friction="0.0"/>
   </joint>
   <link name="${prefix}shoulder_link">
@@ -84,5 +84,5 @@
     <inertial>
       <mass value="${shoulder_mass}" />
-      <inertia ixx="1.0" ixy="0.0" ixz="0.0" iyy="1.0" iyz="0.0" izz="1.0"/>
+      <inertia ixx="0.002" ixy="0.0" ixz="0.0" iyy="0.02" iyz="0.0" izz="0.002"/>
       <origin xyz="${shoulder_cog}" rpy="0.0 0.0 0.0" />
     </inertial>
@@ -94,5 +94,5 @@
     <axis xyz="0 1 0" />
     <limit lower="${-pi}" upper="${pi}" effort="150.0" velocity="${pi}"/>
-    <dynamics damping="0.4" friction="0.0"/>
+    <dynamics damping="0.5" friction="0.0"/>
   </joint>
   <link name="${prefix}upper_arm_link">
@@ -111,5 +111,5 @@
     <inertial>
       <mass value="${upper_arm_mass}" />
-      <inertia ixx="1.0" ixy="0.0" ixz="0.0" iyy="1.0" iyz="0.0" izz="1.0"/>
+      <inertia ixx="0.002" ixy="0.0" ixz="0.0" iyy="0.02" iyz="0.0" izz="0.002"/>
       <origin xyz="${upper_arm_cog}" rpy="0.0 0.0 0.0" />
     </inertial>
@@ -121,5 +121,5 @@
     <axis xyz="0 1 0" />
     <limit lower="${-pi}" upper="${pi}" effort="150.0" velocity="${pi}"/>
-    <dynamics damping="0.4" friction="0.0"/>
+    <dynamics damping="0.5" friction="0.0"/>
   </joint>
   <link name="${prefix}forearm_link">
@@ -138,5 +138,5 @@
       <mass value="${forearm_mass}" />
       <origin xyz="${forearm_cog}" rpy="0.0 0.0 0.0" />
-      <inertia ixx="1.0" ixy="0.0" ixz="0.0" iyy="1.0" iyz="0.0" izz="1.0"/>
+      <inertia ixx="0.002" ixy="0.0" ixz="0.0" iyy="0.02" iyz="0.0" izz="0.002"/>
     </inertial>
   </link>
@@ -147,5 +147,5 @@
     <axis xyz="0 1 0" />
     <limit lower="${-1.0 * pi}" upper="${0.25 * pi}" effort="28.0" velocity="${pi}"/>
-    <dynamics damping="0.3" friction="0.0"/>
+    <dynamics damping="0.5" friction="0.0"/>
   </joint>
   <link name="${prefix}wrist_1_link">
@@ -165,5 +165,5 @@
       <mass value="${wrist_1_mass}" />
       <origin xyz="${wrist_1_cog}" rpy="0.0 0.0 0.0" />
-      <inertia ixx="1.0" ixy="0.0" ixz="0.0" iyy="1.0" iyz="0.0" izz="1.0"/>
+      <inertia ixx="0.002" ixy="0.0" ixz="0.0" iyy="0.02" iyz="0.0" izz="0.002"/>
     </inertial>
   </link>
@@ -174,5 +174,5 @@
     <axis xyz="0 0 1" />
     <limit lower="${-1.0 * pi}" upper="${1.0 * pi}" effort="28.0" velocity="${pi}"/>
-    <dynamics damping="0.3" friction="0.0"/>
+    <dynamics damping="0.5" friction="0.0"/>
   </joint>
   <link name="${prefix}wrist_2_link">
@@ -192,5 +192,5 @@
       <mass value="${wrist_2_mass}" />
       <origin xyz="${wrist_2_cog}" rpy="0.0 0.0 0.0" />
-      <inertia ixx="1.0" ixy="0.0" ixz="0.0" iyy="1.0" iyz="0.0" izz="1.0"/>
+      <inertia ixx="0.002" ixy="0.0" ixz="0.0" iyy="0.02" iyz="0.0" izz="0.002"/>
     </inertial>
   </link>
@@ -201,5 +201,5 @@
     <axis xyz="0 1 0" />
     <limit lower="${-1.0 * pi}" upper="${1.0 * pi}" effort="28.0" velocity="${pi}"/>
-    <dynamics damping="0.3" friction="0.0"/>
+    <dynamics damping="0.5" friction="0.0"/>
   </joint>
   <link name="${prefix}wrist_3_link">
@@ -217,5 +217,5 @@
       <mass value="${wrist_3_mass}" />
       <origin xyz="${wrist_3_cog}" rpy="0.0 0.0 0.0" />
-      <inertia ixx="1.0" ixy="0.0" ixz="0.0" iyy="1.0" iyz="0.0" izz="1.0"/>
+      <inertia ixx="0.002" ixy="0.0" ixz="0.0" iyy="0.02" iyz="0.0" izz="0.002"/>
     </inertial>
   </link>
