Commit message: use correct DH parameter + colored meshes

File: ur_description/urdf/ur3.urdf.xacro (robot description, xacro)
@@ -8,36 +8,32 @@
   <property name="pi" value="3.14159265" />
   <!-- Inertia parameters -->
-  <!-- ToDo: get values for UR3 -->
-  <property name="base_mass" value="4.0" />  <!-- This mass might be incorrect -->
+  <property name="base_mass" value="2.0" />  <!-- This mass might be incorrect -->
   <property name="shoulder_mass" value="2.0" />
-  <property name="upper_arm_mass" value="5.0" />
-  <property name="forearm_mass" value="1.5" />
-  <property name="wrist_1_mass" value="1.0" />
-  <property name="wrist_2_mass" value="1.0" />
-  <property name="wrist_3_mass" value="0.1" />
+  <property name="upper_arm_mass" value="3.42" />
+  <property name="forearm_mass" value="1.26" />
+  <property name="wrist_1_mass" value="0.8" />
+  <property name="wrist_2_mass" value="0.8" />
+  <property name="wrist_3_mass" value="0.35" />
   <!-- These parameters are borrowed from the urcontrol.conf file
        but are not verified for the correct permutation.
        The permutation was guessed by looking at the UR5 parameters.
        Serious use of these parameters needs further inspection. -->
-  <!-- ToDo: get values for UR3 -->
-  <property name="shoulder_cog" value="0.00008 0.00244 -0.037" />
-  <property name="upper_arm_cog" value="0.00001 0.15061 0.38757" />
-  <property name="forearm_cog" value="-0.00012 0.06112 0.1984" />
-  <property name="wrist_1_cog" value="-0.00021 -0.00112 0.02269" />
-  <property name="wrist_2_cog" value="-0.00021 0.00112 0.002269" />
-  <property name="wrist_3_cog" value="0 -0.001156 -0.00149" />
+  <property name="shoulder_cog" value="0.0 -0.02 0.0" />
+  <property name="upper_arm_cog" value="0.13 0.0 0.1157" />
+  <property name="forearm_cog" value="0.05 0.0 0.0238" />
+  <property name="wrist_1_cog" value="0.0 0.0 0.01" />
+  <property name="wrist_2_cog" value="0.0 0.0 0.01" />
+  <property name="wrist_3_cog" value="0.0 0.0 -0.02" />
   <!-- Kinematic model -->
   <!-- Properties from urcontrol.conf -->
-  <!-- ToDo: get values for UR3 -->
-  <property name="ur3_d1" value="0.15" />
-  <property name="ur3_a2" value="-0.244" />
-  <property name="ur3_a3" value="-0.2124" />
-  <property name="ur3_d4" value="0.1146" />
-  <property name="ur3_d5" value="0.0878" />
-  <property name="ur3_d6" value="0.0835" />
+  <property name="ur3_d1" value="0.1519" />
+  <property name="ur3_a2" value="-0.24365" />
+  <property name="ur3_a3" value="-0.21325" />
+  <property name="ur3_d4" value="0.11235" />
+  <property name="ur3_d5" value="0.08535" />
+  <property name="ur3_d6" value="0.0819" />
   <!-- Arbitrary offsets for shoulder/elbow joints -->
-  <!-- ToDo: get values for UR3 -->
-  <property name="shoulder_offset" value="0.121" />  <!-- measured from model -->
-  <property name="elbow_offset" value="-0.0937" /> <!-- measured from model -->
+  <property name="shoulder_offset" value="0.1198" />  <!-- measured from model -->
+  <property name="elbow_offset" value="-0.0925" /> <!-- measured from model -->
   <!-- link lengths used in model -->
   <property name="shoulder_height" value="${ur3_d1}" />
@@ -62,7 +58,4 @@
           <mesh filename="package://ur_description/meshes/ur3/visual/Base.dae"/>
         </geometry>
-        <material name="LightGrey">
-          <color rgba="0.7 0.7 0.7 1.0"/>
-        </material>
       </visual>
       <collision>
@@ -93,7 +86,4 @@
           <mesh filename="package://ur_description/meshes/ur3/visual/Shoulder.dae"/>
         </geometry>
-        <material name="LightGrey">
-          <color rgba="0.7 0.7 0.7 1.0"/>
-        </material>
       </visual>
       <collision>
@@ -124,7 +114,4 @@
           <mesh filename="package://ur_description/meshes/ur3/visual/UpperArm.dae"/>
         </geometry>
-        <material name="LightGrey">
-          <color rgba="0.7 0.7 0.7 1.0"/>
-        </material>
       </visual>
       <collision>
@@ -155,7 +142,4 @@
           <mesh filename="package://ur_description/meshes/ur3/visual/Forearm.dae"/>
         </geometry>
-        <material name="LightGrey">
-          <color rgba="0.7 0.7 0.7 1.0"/>
-        </material>
       </visual>
       <collision>
@@ -186,7 +170,4 @@
           <mesh filename="package://ur_description/meshes/ur3/visual/Wrist1.dae"/>
         </geometry>
-        <material name="LightGrey">
-          <color rgba="0.7 0.7 0.7 1.0"/>
-        </material>
       </visual>
       <collision>
@@ -217,7 +198,4 @@
           <mesh filename="package://ur_description/meshes/ur3/visual/Wrist2.dae"/>
         </geometry>
-        <material name="LightGrey">
-          <color rgba="0.7 0.7 0.7 1.0"/>
-        </material>
       </visual>
       <collision>
@@ -248,7 +226,4 @@
           <mesh filename="package://ur_description/meshes/ur3/visual/Wrist3.dae"/>
         </geometry>
-        <material name="LightGrey">
-          <color rgba="0.7 0.7 0.7 1.0"/>
-        </material>
       </visual>
       <collision>

Commit message: add color to avoid default color 'red' for collision meshes

File: ur_description/urdf/ur3.urdf.xacro (robot description, xacro)
@@ -58,4 +58,7 @@
           <mesh filename="package://ur_description/meshes/ur3/visual/Base.dae"/>
         </geometry>
+        <material name="LightGrey">
+          <color rgba="0.7 0.7 0.7 1.0"/>
+        </material>
       </visual>
       <collision>
@@ -86,4 +89,7 @@
           <mesh filename="package://ur_description/meshes/ur3/visual/Shoulder.dae"/>
         </geometry>
+        <material name="LightGrey">
+          <color rgba="0.7 0.7 0.7 1.0"/>
+        </material>
       </visual>
       <collision>
@@ -114,4 +120,7 @@
           <mesh filename="package://ur_description/meshes/ur3/visual/UpperArm.dae"/>
         </geometry>
+        <material name="LightGrey">
+          <color rgba="0.7 0.7 0.7 1.0"/>
+        </material>
       </visual>
       <collision>
@@ -142,4 +151,7 @@
           <mesh filename="package://ur_description/meshes/ur3/visual/Forearm.dae"/>
         </geometry>
+        <material name="LightGrey">
+          <color rgba="0.7 0.7 0.7 1.0"/>
+        </material>
       </visual>
       <collision>
@@ -170,4 +182,7 @@
           <mesh filename="package://ur_description/meshes/ur3/visual/Wrist1.dae"/>
         </geometry>
+        <material name="LightGrey">
+          <color rgba="0.7 0.7 0.7 1.0"/>
+        </material>
       </visual>
       <collision>
@@ -198,4 +213,7 @@
           <mesh filename="package://ur_description/meshes/ur3/visual/Wrist2.dae"/>
         </geometry>
+        <material name="LightGrey">
+          <color rgba="0.7 0.7 0.7 1.0"/>
+        </material>
       </visual>
       <collision>
@@ -226,4 +244,7 @@
           <mesh filename="package://ur_description/meshes/ur3/visual/Wrist3.dae"/>
         </geometry>
+        <material name="LightGrey">
+          <color rgba="0.7 0.7 0.7 1.0"/>
+        </material>
       </visual>
       <collision>

Commit message: added change to ur3 as well.

File: ur_description/urdf/ur3.urdf.xacro (robot description, xacro)
@@ -139,5 +139,5 @@
       <axis xyz="0 1 0" />
       <xacro:unless value="${joint_limited}">
-        <limit lower="${-2.0 * pi}" upper="${2.0 * pi}" effort="150.0" velocity="3.15"/>
+        <limit lower="${-pi}" upper="${pi}" effort="150.0" velocity="3.15"/>
       </xacro:unless>
       <xacro:if value="${joint_limited}">

Commit message: Fix elbow joint limits (#268)

File: ur_description/urdf/ur3.urdf.xacro (robot description, xacro)
@@ -138,5 +138,5 @@
       <axis xyz="0 1 0" />
       <xacro:unless value="${joint_limited}">
-        <limit lower="${-2.0 * pi}" upper="${2.0 * pi}" effort="150.0" velocity="3.15"/>
+        <limit lower="${-pi}" upper="${pi}" effort="150.0" velocity="3.15"/>
       </xacro:unless>
       <xacro:if value="${joint_limited}">

Commit message: added ur3 and ur5 calibration

File: ur_description/urdf/ur3.urdf.xacro (robot description, xacro)
@@ -22,5 +22,7 @@
     wrist_2_lower_limit:=${-pi}    wrist_2_upper_limit:=${pi}
     wrist_3_lower_limit:=${-pi}    wrist_3_upper_limit:=${pi}
-    transmission_hw_interface:=hardware_interface/PositionJointInterface">
+    transmission_hw_interface:=hardware_interface/PositionJointInterface
+    kinematics_file">
+    <xacro:property name="__kinematics" value="${kinematics_file['kinematics']}"/>
     <!-- Inertia parameters -->
     <xacro:property name="base_mass" value="2.0" />  <!-- This mass might be incorrect -->
@@ -41,24 +43,13 @@
     <xacro:property name="wrist_2_cog" value="0.0 0.0 0.01" />
     <xacro:property name="wrist_3_cog" value="0.0 0.0 -0.02" />
-    <!-- Kinematic model -->
-    <!-- Properties from urcontrol.conf -->
-    <xacro:property name="d1" value="0.1519" />
-    <xacro:property name="a2" value="-0.24365" />
-    <xacro:property name="a3" value="-0.21325" />
-    <xacro:property name="d4" value="0.11235" />
-    <xacro:property name="d5" value="0.08535" />
-    <xacro:property name="d6" value="0.0819" />
     <!-- Arbitrary offsets for shoulder/elbow joints -->
     <xacro:property name="shoulder_offset" value="0.1198" />  <!-- measured from model -->
-    <xacro:property name="elbow_offset" value="-0.0925" /> <!-- measured from model -->
-    <!-- link lengths used in model -->
-    <xacro:property name="shoulder_height" value="${d1}" />
-    <xacro:property name="upper_arm_length" value="${-a2}" />
-    <xacro:property name="forearm_length" value="${-a3}" />
-    <xacro:property name="wrist_1_length" value="${d4 - elbow_offset - shoulder_offset}" />
-    <xacro:property name="wrist_2_length" value="${d5}" />
-    <xacro:property name="wrist_3_length" value="${d6}" />
+    <xacro:property name="elbow_offset" value="0.0275" /> <!-- measured from model -->
+    <xacro:property name="upper_arm_inertia_offset" value="0.12" />  <!-- measured from model -->
+    <!-- This is for compatibility reasons, as transformation between base and base_link was always 180 degree in the ur_description -->
+    <xacro:property name="base_correction" value="${pi}" />
     <link name="${prefix}base_link" >
       <visual>
+        <origin xyz="0 0 0" rpy="0 0 ${base_correction}"/>
         <geometry>
           <mesh filename="package://ur_description/meshes/ur3/visual/base.dae"/>
@@ -69,4 +60,5 @@
       </visual>
       <collision>
+        <origin xyz="0 0 0" rpy="0 0 ${base_correction}"/>
         <geometry>
           <mesh filename="package://ur_description/meshes/ur3/collision/base.stl"/>
@@ -80,5 +72,5 @@
       <parent link="${prefix}base_link" />
       <child link = "${prefix}shoulder_link" />
-      <origin xyz="0.0 0.0 ${shoulder_height}" rpy="0.0 0.0 0.0" />
+      <origin xyz="${__kinematics['shoulder']['x']} ${__kinematics['shoulder']['y']} ${__kinematics['shoulder']['z']}" rpy="${__kinematics['shoulder']['roll']} ${__kinematics['shoulder']['pitch']} ${__kinematics['shoulder']['yaw'] + base_correction}" />
       <axis xyz="0 0 1" />
       <xacro:unless value="${joint_limited}">
@@ -92,4 +84,5 @@
     <link name="${prefix}shoulder_link">
       <visual>
+        <origin xyz="0 0 0" rpy="0 0 ${pi}"/>
         <geometry>
           <mesh filename="package://ur_description/meshes/ur3/visual/shoulder.dae"/>
@@ -100,4 +93,5 @@
       </visual>
       <collision>
+        <origin xyz="0 0 0" rpy="0 0 ${pi}"/>
         <geometry>
           <mesh filename="package://ur_description/meshes/ur3/collision/shoulder.stl"/>
@@ -111,6 +105,6 @@
       <parent link="${prefix}shoulder_link" />
       <child link = "${prefix}upper_arm_link" />
-      <origin xyz="0.0 ${shoulder_offset} 0.0" rpy="0.0 ${pi / 2.0} 0.0" />
-      <axis xyz="0 1 0" />
+      <origin xyz="${__kinematics['upper_arm']['x']} ${__kinematics['upper_arm']['y']} ${__kinematics['upper_arm']['z']}" rpy="${__kinematics['upper_arm']['roll']} ${__kinematics['upper_arm']['pitch']} ${__kinematics['upper_arm']['yaw']}" />
+      <axis xyz="0 0 1" />
       <xacro:unless value="${joint_limited}">
         <limit lower="${-2.0 * pi}" upper="${2.0 * pi}" effort="330.0" velocity="2.16"/>
@@ -123,4 +117,5 @@
     <link name="${prefix}upper_arm_link">
       <visual>
+        <origin xyz="0 0 ${shoulder_offset}" rpy="${pi/2} 0 ${-pi/2}"/>
         <geometry>
           <mesh filename="package://ur_description/meshes/ur3/visual/upperarm.dae"/>
@@ -131,10 +126,11 @@
       </visual>
       <collision>
+        <origin xyz="0 0 ${shoulder_offset}" rpy="${pi/2} 0 ${-pi/2}"/>
         <geometry>
           <mesh filename="package://ur_description/meshes/ur3/collision/upperarm.stl"/>
         </geometry>
       </collision>
-      <xacro:cylinder_inertial radius="0.075" length="${-a2}" mass="${upper_arm_mass}">
-        <origin xyz="0.0 0.0 ${-a2/2.0}" rpy="0 0 0" />
+      <xacro:cylinder_inertial radius="0.075" length="${-1*__kinematics['forearm']['x']}" mass="${upper_arm_mass}">
+        <origin xyz="${0.5*__kinematics['forearm']['x']} 0.0 ${upper_arm_inertia_offset}" rpy="0 ${pi/2} 0" />
       </xacro:cylinder_inertial>
     </link>
@@ -142,6 +138,6 @@
       <parent link="${prefix}upper_arm_link" />
       <child link = "${prefix}forearm_link" />
-      <origin xyz="0.0 ${elbow_offset} ${upper_arm_length}" rpy="0.0 0.0 0.0" />
-      <axis xyz="0 1 0" />
+      <origin xyz="${__kinematics['forearm']['x']} ${__kinematics['forearm']['y']} ${__kinematics['forearm']['z']}" rpy="${__kinematics['forearm']['roll']} ${__kinematics['forearm']['pitch']} ${__kinematics['forearm']['yaw']}" />
+      <axis xyz="0 0 1" />
       <xacro:unless value="${joint_limited}">
         <limit lower="${-pi}" upper="${pi}" effort="150.0" velocity="3.15"/>
@@ -154,4 +150,5 @@
     <link name="${prefix}forearm_link">
       <visual>
+        <origin xyz="0 0 ${elbow_offset}" rpy="${pi/2} 0 ${-pi/2}"/>
          <geometry>
           <mesh filename="package://ur_description/meshes/ur3/visual/forearm.dae"/>
@@ -162,10 +159,11 @@
       </visual>
       <collision>
+        <origin xyz="0 0 ${elbow_offset}" rpy="${pi/2} 0 ${-pi/2}"/>
         <geometry>
           <mesh filename="package://ur_description/meshes/ur3/collision/forearm.stl"/>
         </geometry>
       </collision>
-      <xacro:cylinder_inertial radius="0.075" length="${-a3}" mass="${forearm_mass}">
-        <origin xyz="0.0 0.0 ${-a3/2.0}" rpy="0 0 0" />
+      <xacro:cylinder_inertial radius="0.075" length="${-1*__kinematics['wrist_1']['x']}" mass="${forearm_mass}">
+        <origin xyz="${0.5*__kinematics['forearm']['x']} 0.0 ${elbow_offset}" rpy="0 ${pi/2} 0" />
       </xacro:cylinder_inertial>
     </link>
@@ -173,6 +171,6 @@
       <parent link="${prefix}forearm_link" />
       <child link = "${prefix}wrist_1_link" />
-      <origin xyz="0.0 0.0 ${forearm_length}" rpy="0.0 ${pi / 2.0} 0.0" />
-      <axis xyz="0 1 0" />
+      <origin xyz="${__kinematics['wrist_1']['x']} ${__kinematics['wrist_1']['y']} ${__kinematics['wrist_1']['z']}" rpy="${__kinematics['wrist_1']['roll']} ${__kinematics['wrist_1']['pitch']} ${__kinematics['wrist_1']['yaw']}" />
+      <axis xyz="0 0 1" />
       <xacro:unless value="${joint_limited}">
         <limit lower="${-2.0 * pi}" upper="${2.0 * pi}" effort="54.0" velocity="3.2"/>
@@ -185,4 +183,5 @@
     <link name="${prefix}wrist_1_link">
       <visual>
+        <origin xyz="0 0 -0.085" rpy="${pi/2} 0 0"/>
         <geometry>
           <mesh filename="package://ur_description/meshes/ur3/visual/wrist1.dae"/>
@@ -193,10 +192,11 @@
       </visual>
       <collision>
+        <origin xyz="0 0 -0.085" rpy="${pi/2} 0 0"/>
         <geometry>
           <mesh filename="package://ur_description/meshes/ur3/collision/wrist1.stl"/>
         </geometry>
       </collision>
-      <xacro:cylinder_inertial radius="0.075" length="0.12" mass="${wrist_1_mass}">
-        <origin xyz="0.0 ${wrist_1_length} 0.0" rpy="0 0 0" />
+      <xacro:cylinder_inertial radius="0.075" length="${-1*__kinematics['wrist_2']['y']}" mass="${wrist_1_mass}">
+        <origin xyz="0.0 0.0 0.0" rpy="0 0 0" />
       </xacro:cylinder_inertial>
     </link>
@@ -204,5 +204,5 @@
       <parent link="${prefix}wrist_1_link" />
       <child link = "${prefix}wrist_2_link" />
-      <origin xyz="0.0 ${wrist_1_length} 0.0" rpy="0.0 0.0 0.0" />
+      <origin xyz="${__kinematics['wrist_2']['x']} ${__kinematics['wrist_2']['y']} ${__kinematics['wrist_2']['z']}" rpy="${__kinematics['wrist_2']['roll']} ${__kinematics['wrist_2']['pitch']} ${__kinematics['wrist_2']['yaw']}" />
       <axis xyz="0 0 1" />
       <xacro:unless value="${joint_limited}">
@@ -216,4 +216,5 @@
     <link name="${prefix}wrist_2_link">
       <visual>
+        <origin xyz="0 0 -0.085" rpy="0 0 0"/>
         <geometry>
           <mesh filename="package://ur_description/meshes/ur3/visual/wrist2.dae"/>
@@ -224,10 +225,11 @@
       </visual>
       <collision>
+        <origin xyz="0 0 -0.085" rpy="0 0 0"/>
         <geometry>
           <mesh filename="package://ur_description/meshes/ur3/collision/wrist2.stl"/>
         </geometry>
       </collision>
-      <xacro:cylinder_inertial radius="0.075" length="0.12" mass="${wrist_2_mass}">
-        <origin xyz="0.0 0.0 ${wrist_2_length}" rpy="0 0 0" />
+      <xacro:cylinder_inertial radius="0.075" length="${__kinematics['wrist_3']['y']}" mass="${wrist_2_mass}">
+        <origin xyz="0.0 0.0 0.0" rpy="0 0 0" />
       </xacro:cylinder_inertial>
     </link>
@@ -235,6 +237,6 @@
       <parent link="${prefix}wrist_2_link" />
       <child link = "${prefix}wrist_3_link" />
-      <origin xyz="0.0 0.0 ${wrist_2_length}" rpy="0.0 0.0 0.0" />
-      <axis xyz="0 1 0" />
+      <origin xyz="${__kinematics['wrist_3']['x']} ${__kinematics['wrist_3']['y']} ${__kinematics['wrist_3']['z']}" rpy="${__kinematics['wrist_3']['roll']} ${__kinematics['wrist_3']['pitch']} ${__kinematics['wrist_3']['yaw']}" />
+      <axis xyz="0 0 1" />
       <xacro:unless value="${joint_limited}">
         <limit lower="${-2.0 * pi}" upper="${2.0 * pi}" effort="54.0" velocity="3.2"/>
@@ -247,4 +249,5 @@
     <link name="${prefix}wrist_3_link">
       <visual>
+        <origin xyz="0 0 -0.082" rpy="${pi/2} 0 0"/>
         <geometry>
           <mesh filename="package://ur_description/meshes/ur3/visual/wrist3.dae"/>
@@ -255,10 +258,11 @@
       </visual>
       <collision>
+        <origin xyz="0 0 -0.082" rpy="${pi/2} 0 0"/>
         <geometry>
           <mesh filename="package://ur_description/meshes/ur3/collision/wrist3.stl"/>
         </geometry>
       </collision>
-      <xacro:cylinder_inertial radius="0.032" length="0.04" mass="${wrist_3_mass}">
-        <origin xyz="0.0 ${wrist_3_length - 0.02} 0.0" rpy="${pi/2} 0 0" />
+      <xacro:cylinder_inertial radius="0.045" length="0.0305" mass="${wrist_3_mass}">
+        <origin xyz="0.0 0.0 ${-0.0305/2}" rpy="0 0 0" />
       </xacro:cylinder_inertial>
     </link>
@@ -266,5 +270,5 @@
       <parent link="${prefix}wrist_3_link" />
       <child link = "${prefix}ee_link" />
-      <origin xyz="0.0 ${wrist_3_length} 0.0" rpy="0.0 0.0 ${pi/2.0}" />
+      <origin xyz="0.0 0.0 0.0" rpy="0.0 ${-pi/2.0} ${pi/2.0}" />
     </joint>
     <link name="${prefix}ee_link">
@@ -276,4 +280,9 @@
       </collision>
     </link>
+    <joint name="${prefix}wrist_3_passive_joint" type="fixed">
+      <origin xyz="0 0 0" rpy="0 0 0"/>
+      <parent link="${prefix}wrist_3_link"/>
+      <child link="${prefix}tool0"/>
+    </joint>
     <xacro:ur_arm_transmission prefix="${prefix}" hw_interface="${transmission_hw_interface}" />
     <xacro:ur_arm_gazebo prefix="${prefix}" />
@@ -285,5 +294,5 @@
                  degrees)
       -->
-      <origin xyz="0 0 0" rpy="0 0 ${-pi}"/>
+      <origin xyz="0 0 0" rpy="0 0 ${-base_correction}"/>
       <parent link="${prefix}base_link"/>
       <child link="${prefix}base"/>
@@ -291,9 +300,4 @@
     <!-- Frame coincident with all-zeros TCP on UR controller -->
     <link name="${prefix}tool0"/>
-    <joint name="${prefix}wrist_3_link-tool0_fixed_joint" type="fixed">
-      <origin xyz="0 ${wrist_3_length} 0" rpy="${pi/-2.0} 0 0"/>
-      <parent link="${prefix}wrist_3_link"/>
-      <child link="${prefix}tool0"/>
-    </joint>
   </xacro:macro>
 </robot>
