Commit message: Merged urdf geometry into the same xacro file * same individual base for each robot * no duplicated works

File: ur_description/urdf/ur.geometry.xacro (robot description, xacro)
@@ -1,11 +1,12 @@
 <?xml version="1.0"?>
 <robot xmlns:xacro="http://wiki.ros.org/xacro">
-  <xacro:include filename="$(find ur_description)/urdf/ur.transmission.xacro" />
-  <xacro:include filename="$(find ur_description)/urdf/ur.gazebo.xacro" />
-  <xacro:include filename="$(find ur_description)/urdf/ur.common.xacro" />
-  <xacro:macro name="ur5_robot" params="prefix joints_limits_parameters_file
-                                               physical_parameters_file
-                                               visual_parameters_file
-                                               transmission_hw_interface:=hardware_interface/PositionJointInterface">
+<!--
+  Author: Ludovic Delval
+  Contributor: Felix Messmer, Kelsey Hawkins, Jimmy Da Silva, Ajit Krisshna N L, Muhammad Asif Rana
+-->
+ <xacro:include filename="$(find ur_description)/urdf/ur.transmission.xacro" />
+ <xacro:include filename="$(find ur_description)/urdf/ur.gazebo.xacro" />
+ <xacro:include filename="$(find ur_description)/urdf/ur.common.xacro" />
+ <xacro:macro name="ur_robot" params="prefix joints_limits_parameters_file physical_parameters_file visual_parameters_file transmission_hw_interface:=hardware_interface/PositionJointInterface">
     <xacro:read_file joints_limits_parameters_file="${joints_limits_parameters_file}"
                     physical_parameters_file="${physical_parameters_file}"
@@ -38,5 +39,5 @@
       <axis xyz="0 0 1" />
       <limit lower="${shoulder_pan_lower_limit}" upper="${shoulder_pan_upper_limit}"
-        effort="${shoulder_pan_effort_limit}" velocity="${shoulder_pan_velocity_limit}"/>
+          effort="${shoulder_pan_effort_limit}" velocity="${shoulder_pan_velocity_limit}"/>
       <dynamics damping="0.0" friction="0.0"/>
     </joint>
@@ -82,6 +83,6 @@
         </geometry>
       </collision>
-      <xacro:cylinder_inertial radius="${upperarm_inertia_radius}" length="${upperarm_inertia_length}" mass="${upper_arm_mass}">
-        <origin xyz="0.0 0.0 0.28" rpy="0 0 0" />
+      <xacro:cylinder_inertial radius="${upperarm_inertia_radius}" length="${-a2}" mass="${upper_arm_mass}">
+        <origin xyz="0.0 0.0 ${-a2/2.0}" rpy="0 0 0" />
       </xacro:cylinder_inertial>
     </link>
@@ -109,6 +110,6 @@
         </geometry>
       </collision>
-      <xacro:cylinder_inertial radius="${forearm_inertia_radius}" length="{-a3}"  mass="${forearm_mass}">
-        <origin xyz="0.0 0.0 ${-a3/2}" rpy="0 0 0" />
+      <xacro:cylinder_inertial radius="${forearm_inertia_radius}" length="${-a3}"  mass="${forearm_mass}">
+        <origin xyz="0.0 0.0 ${-a3/2.0}" rpy="0 0 0" />
       </xacro:cylinder_inertial>
     </link>
@@ -137,5 +138,5 @@
       </collision>
       <xacro:cylinder_inertial radius="${wrist_1_inertia_radius}" length="${wrist_1_inertia_length}"  mass="${wrist_1_mass}">
-        <origin xyz="0.0 ${wrist_1_length} 0.0" rpy="0 0 0" />
+        <origin xyz="0.0 0.0 0.0" rpy="0 0 0" />
       </xacro:cylinder_inertial>
     </link>
@@ -146,5 +147,5 @@
       <axis xyz="0 0 1" />
       <limit lower="${wrist_2_lower_limit}" upper="${wrist_2_upper_limit}"
-        effort="${wrist_2_effort_limit}" velocity="${wrist_2_velocity_limit}"/>
+             effort="${wrist_2_effort_limit}" velocity="${wrist_2_velocity_limit}"/>
       <dynamics damping="0.0" friction="0.0"/>
     </joint>
@@ -173,5 +174,5 @@
       <axis xyz="0 1 0" />
       <limit lower="${wrist_3_lower_limit}" upper="${wrist_3_upper_limit}"
-        effort="${wrist_3_effort_limit}" velocity="${wrist_3_velocity_limit}"/>
+             effort="${wrist_3_effort_limit}" velocity="${wrist_3_velocity_limit}"/>
       <dynamics damping="0.0" friction="0.0"/>
     </joint>
@@ -191,5 +192,5 @@
       </collision>
       <xacro:cylinder_inertial radius="${wrist_3_inertia_radius}" length="${wrist_3_inertia_length}"  mass="${wrist_3_mass}">
-        <origin xyz="0.0 ${wrist_3_length - 0.0345/2} 0.0" rpy="0 0 0" />
+        <origin xyz="0.0 ${wrist_3_length - 0.02} 0.0" rpy="0 0 0" />
       </xacro:cylinder_inertial>
     </link>

File: ur_description/urdf/ur10_robot.urdf.xacro (robot description, xacro)
@@ -7,10 +7,9 @@
   <xacro:arg name="visual_params" default="$(find ur_description)/config/ur10/visual_parameters.yaml"/>
   <xacro:arg name="transmission_hw_interface" default="hardware_interface/PositionJointInterface"/>
-  <!-- common stuff -->
-  <xacro:include filename="$(find ur_description)/urdf/common.gazebo.xacro" />
-  <!-- ur10 -->
-  <xacro:include filename="$(find ur_description)/urdf/ur10.urdf.xacro" />
-  <!-- arm -->
-  <xacro:ur10_robot prefix="" joints_limits_parameters_file="${load_yaml('$(arg joints_limits_params)')}"
+   <!-- common stuff -->
+   <xacro:include filename="$(find ur_description)/urdf/common.gazebo.xacro" />
+   <xacro:include filename="$(find ur_description)/urdf/ur.geometry.xacro" />
+   <!-- arm -->
+   <xacro:ur_robot prefix="" joints_limits_parameters_file="${load_yaml('$(arg joints_limits_params)')}"
                              physical_parameters_file="${load_yaml('$(arg physical_params)')}"
                              visual_parameters_file="${load_yaml('$(arg visual_params)')}"

File: ur_description/urdf/ur3_robot.urdf.xacro (robot description, xacro)
@@ -9,8 +9,7 @@
    <!-- common stuff -->
    <xacro:include filename="$(find ur_description)/urdf/common.gazebo.xacro" />
-   <!-- ur3 -->
-   <xacro:include filename="$(find ur_description)/urdf/ur3.urdf.xacro" />
+   <xacro:include filename="$(find ur_description)/urdf/ur.geometry.xacro" />
    <!-- arm -->
-   <xacro:ur3_robot prefix="" joints_limits_parameters_file="${load_yaml('$(arg joints_limits_params)')}"
+   <xacro:ur_robot prefix="" joints_limits_parameters_file="${load_yaml('$(arg joints_limits_params)')}"
                              physical_parameters_file="${load_yaml('$(arg physical_params)')}"
                              visual_parameters_file="${load_yaml('$(arg visual_params)')}"

File: ur_description/urdf/ur5_robot.urdf.xacro (robot description, xacro)
@@ -6,10 +6,9 @@
   <xacro:arg name="visual_params" default="$(find ur_description)/config/ur5/visual_parameters.yaml"/>
   <xacro:arg name="transmission_hw_interface" default="hardware_interface/PositionJointInterface"/>
-  <!-- common stuff -->
-  <xacro:include filename="$(find ur_description)/urdf/common.gazebo.xacro" />
-  <!-- ur5 -->
-  <xacro:include filename="$(find ur_description)/urdf/ur5.urdf.xacro" />
-  <!-- arm -->
-  <xacro:ur5_robot prefix=""  joints_limits_parameters_file="${load_yaml('$(arg joints_limits_params)')}"
+   <!-- common stuff -->
+   <xacro:include filename="$(find ur_description)/urdf/common.gazebo.xacro" />
+   <xacro:include filename="$(find ur_description)/urdf/ur.geometry.xacro" />
+   <!-- arm -->
+   <xacro:ur_robot prefix="" joints_limits_parameters_file="${load_yaml('$(arg joints_limits_params)')}"
                              physical_parameters_file="${load_yaml('$(arg physical_params)')}"
                              visual_parameters_file="${load_yaml('$(arg visual_params)')}"
