Commit message: refactored the yaml into multiple yaml file

File: ur_description/urdf/ur.common.xacro (robot description, xacro)
@@ -1,4 +1,4 @@
 <?xml version="1.0"?>
-<robot xmlns:xacro="http://ros.org/wiki/xacro">
+<robot xmlns:xacro="http://wiki.ros.org/xacro">
 <!--
   Author: Ludovic Delval
@@ -14,10 +14,10 @@
     </inertial>
   </xacro:macro>
-  <xacro:macro name="read_file" params="yaml_file">
-    <xacro:property name="__limits" value="${yaml_file['limits']}"/>
-    <xacro:property name="__dh_parameters" value="${yaml_file['dh_parameters']}"/>
-    <xacro:property name="__offsets" value="${yaml_file['offsets']}"/>
-    <xacro:property name="__inertia_parameters" value="${yaml_file['inertia_parameters']}" />
-    <xacro:property name="__mesh_files" value="${yaml_file['mesh_files']}" />
+  <xacro:macro name="read_file" params="joints_limits_parameters_file physical_parameters_file visual_parameters_file">
+    <xacro:property name="__limits" value="${joints_limits_parameters_file['limits']}"/>
+    <xacro:property name="__dh_parameters" value="${physical_parameters_file['dh_parameters']}"/>
+    <xacro:property name="__offsets" value="${physical_parameters_file['offsets']}"/>
+    <xacro:property name="__inertia_parameters" value="${physical_parameters_file['inertia_parameters']}" />
+    <xacro:property name="__mesh_files" value="${visual_parameters_file['mesh_files']}" />
     <!-- JOINTS LIMIT PARAMETERS -->
     <xacro:property name="shoulder_pan_lower_limit" value="${__limits['shoulder_pan']['lower']}" scope="parent"/>

File: ur_description/urdf/ur10.urdf.xacro (robot description, xacro)
@@ -8,6 +8,11 @@
   <xacro:include filename="$(find ur_description)/urdf/ur.gazebo.xacro" />
   <xacro:include filename="$(find ur_description)/urdf/ur.common.xacro" />
-  <xacro:macro name="ur10_robot" params="prefix yaml_file transmission_hw_interface:=hardware_interface/PositionJointInterface">
-    <xacro:read_file yaml_file="${yaml_file}"/>
+  <xacro:macro name="ur10_robot" params="prefix joints_limits_parameters_file
+                                                physical_parameters_file
+                                                visual_parameters_file
+                                                transmission_hw_interface:=hardware_interface/PositionJointInterface">
+    <xacro:read_file joints_limits_parameters_file="${joints_limits_parameters_file}"
+                    physical_parameters_file="${physical_parameters_file}"
+                    visual_parameters_file="${visual_parameters_file}"/>
     <xacro:compute_lenght d1="${d1}" a2="${a2}" a3="${a3}"
                           d4="${d4}" d5="${d5}" d6="${d6}"

File: ur_description/urdf/ur10_robot.urdf.xacro (robot description, xacro)
@@ -3,5 +3,7 @@
        name="ur10" >
   <!-- common stuff -->
-  <xacro:arg name="yaml_config" default="$(find ur_description)/config/ur10_default.yaml"/>
+  <xacro:arg name="joints_limits_params" default="$(find ur_description)/config/ur10/joints_limits_parameters.yaml"/>
+  <xacro:arg name="physical_params" default="$(find ur_description)/config/ur10/physical_parameters.yaml"/>
+  <xacro:arg name="visual_params" default="$(find ur_description)/config/ur10/visual_parameters.yaml"/>
   <xacro:arg name="transmission_hw_interface" default="hardware_interface/PositionJointInterface"/>
   <!-- common stuff -->
@@ -10,12 +12,7 @@
   <xacro:include filename="$(find ur_description)/urdf/ur10.urdf.xacro" />
   <!-- arm -->
-  <xacro:ur10_robot prefix="" yaml_file="${load_yaml('$(arg yaml_config)')}"
-    transmission_hw_interface="$(arg transmission_hw_interface)"
-  />
-  <link name="world" />
-  <joint name="world_joint" type="fixed">
-    <parent link="world" />
-    <child link = "base_link" />
-    <origin xyz="0.0 0.0 0.0" rpy="0.0 0.0 0.0" />
-  </joint>
+  <xacro:ur10_robot prefix="" joints_limits_parameters_file="${load_yaml('$(arg joints_limits_params)')}"
+                             physical_parameters_file="${load_yaml('$(arg physical_params)')}"
+                             visual_parameters_file="${load_yaml('$(arg visual_params)')}"
+                             transmission_hw_interface="$(arg transmission_hw_interface)"/>
 </robot>

File: ur_description/urdf/ur3.urdf.xacro (robot description, xacro)
@@ -1,4 +1,4 @@
 <?xml version="1.0"?>
-<robot xmlns:xacro="http://ros.org/wiki/xacro">
+<robot xmlns:xacro="http://wiki.ros.org/xacro">
 <!--
   Author: Felix Messmer
@@ -7,10 +7,11 @@
   <xacro:include filename="$(find ur_description)/urdf/ur.gazebo.xacro" />
   <xacro:include filename="$(find ur_description)/urdf/ur.common.xacro" />
-  <xacro:macro name="ur3_robot" params="prefix yaml_file transmission_hw_interface:=hardware_interface/PositionJointInterface">
-    <xacro:read_file yaml_file="${yaml_file}"/>
+  <xacro:macro name="ur3_robot" params="prefix joints_limits_parameters_file physical_parameters_file visual_parameters_file transmission_hw_interface:=hardware_interface/PositionJointInterface">
+    <xacro:read_file joints_limits_parameters_file="${joints_limits_parameters_file}"
+                    physical_parameters_file="${physical_parameters_file}"
+                    visual_parameters_file="${visual_parameters_file}"/>
     <xacro:compute_lenght d1="${d1}" a2="${a2}" a3="${a3}"
                           d4="${d4}" d5="${d5}" d6="${d6}"
-                          shoulder_offset="${shoulder_offset}" elbow_offset="${elbow_offset}"
-/>
+                          shoulder_offset="${shoulder_offset}" elbow_offset="${elbow_offset}"/>
     <link name="${prefix}base_link" >
       <visual>
@@ -63,10 +64,6 @@
       <origin xyz="0.0 ${shoulder_offset} 0.0" rpy="0.0 ${pi / 2.0} 0.0" />
       <axis xyz="0 1 0" />
-      <xacro:unless value="${joint_limited}">
-        <limit lower="${-2.0 * pi}" upper="${2.0 * pi}" effort="330.0" velocity="2.16"/>
-      </xacro:unless>
-      <xacro:if value="${joint_limited}">
-        <limit lower="${shoulder_lift_lower_limit}" upper="${shoulder_lift_upper_limit}" effort="330.0" velocity="2.16"/>
-      </xacro:if>
+      <limit lower="${shoulder_lift_lower_limit}" upper="${shoulder_lift_upper_limit}"
+        effort="${shoulder_lift_effort_limit}" velocity="${shoulder_lift_velocity_limit}"/>
       <dynamics damping="0.0" friction="0.0"/>
     </joint>
@@ -210,5 +207,5 @@
       </collision>
     </link>
-    <xacro:ur_arm_transmission prefix="${prefix}" />
+    <xacro:ur_arm_transmission prefix="${prefix}" hw_interface="${transmission_hw_interface}" />
     <xacro:ur_arm_gazebo prefix="${prefix}" />
     <!-- ROS base_link to UR 'Base' Coordinates transform -->

File: ur_description/urdf/ur3_robot.urdf.xacro (robot description, xacro)
@@ -3,6 +3,8 @@
        name="ur3" >
    <!-- common stuff -->
-   <xacro:arg name="yaml_config" default="$(find ur_description)/config/ur3_default.yaml"/>
-  <xacro:arg name="transmission_hw_interface" default="hardware_interface/PositionJointInterface"/>
+   <xacro:arg name="joints_limits_params" default="$(find ur_description)/config/ur3/joints_limits_parameters.yaml"/>
+   <xacro:arg name="physical_params" default="$(find ur_description)/config/ur3/physical_parameters.yaml"/>
+   <xacro:arg name="visual_params" default="$(find ur_description)/config/ur3/visual_parameters.yaml"/>
+   <xacro:arg name="transmission_hw_interface" default="hardware_interface/PositionJointInterface"/>
    <!-- common stuff -->
    <xacro:include filename="$(find ur_description)/urdf/common.gazebo.xacro" />
@@ -10,5 +12,7 @@
    <xacro:include filename="$(find ur_description)/urdf/ur3.urdf.xacro" />
    <!-- arm -->
-   <xacro:ur3_robot prefix="" yaml_file="${load_yaml('$(arg yaml_config)')}" transmission_hw_interface="$(arg transmission_hw_interface)"
-  />/>
+   <xacro:ur3_robot prefix="" joints_limits_parameters_file="${load_yaml('$(arg joints_limits_params)')}"
+                             physical_parameters_file="${load_yaml('$(arg physical_params)')}"
+                             visual_parameters_file="${load_yaml('$(arg visual_params)')}"
+                             transmission_hw_interface="$(arg transmission_hw_interface)"/>
 </robot>

File: ur_description/urdf/ur5.urdf.xacro (robot description, xacro)
@@ -4,7 +4,11 @@
   <xacro:include filename="$(find ur_description)/urdf/ur.gazebo.xacro" />
   <xacro:include filename="$(find ur_description)/urdf/ur.common.xacro" />
-  <xacro:macro name="ur5_robot" params="prefix yaml_file
-    transmission_hw_interface:=hardware_interface/PositionJointInterface">
-    <xacro:read_file yaml_file="${yaml_file}"/>
+  <xacro:macro name="ur5_robot" params="prefix joints_limits_parameters_file
+                                               physical_parameters_file
+                                               visual_parameters_file
+                                               transmission_hw_interface:=hardware_interface/PositionJointInterface">
+    <xacro:read_file joints_limits_parameters_file="${joints_limits_parameters_file}"
+                    physical_parameters_file="${physical_parameters_file}"
+                    visual_parameters_file="${visual_parameters_file}"/>
     <xacro:compute_lenght d1="${d1}" a2="${a2}" a3="${a3}"
                           d4="${d4}" d5="${d5}" d6="${d6}"

File: ur_description/urdf/ur5_robot.urdf.xacro (robot description, xacro)
@@ -2,6 +2,8 @@
 <robot xmlns:xacro="http://wiki.ros.org/xacro"
        name="ur5" >
+  <xacro:arg name="joints_limits_params" default="$(find ur_description)/config/ur5/joints_limits_parameters.yaml"/>
+  <xacro:arg name="physical_params" default="$(find ur_description)/config/ur5/physical_parameters.yaml"/>
+  <xacro:arg name="visual_params" default="$(find ur_description)/config/ur5/visual_parameters.yaml"/>
   <xacro:arg name="transmission_hw_interface" default="hardware_interface/PositionJointInterface"/>
-  <xacro:arg name="yaml_config" default="$(find ur_description)/config/ur5_default.yaml"/>
   <!-- common stuff -->
   <xacro:include filename="$(find ur_description)/urdf/common.gazebo.xacro" />
@@ -9,6 +11,7 @@
   <xacro:include filename="$(find ur_description)/urdf/ur5.urdf.xacro" />
   <!-- arm -->
-  <xacro:ur5_robot prefix="" yaml_file="${load_yaml('$(arg yaml_config)')}"
-    transmission_hw_interface="$(arg transmission_hw_interface)"
-  />
+  <xacro:ur5_robot prefix=""  joints_limits_parameters_file="${load_yaml('$(arg joints_limits_params)')}"
+                             physical_parameters_file="${load_yaml('$(arg physical_params)')}"
+                             visual_parameters_file="${load_yaml('$(arg visual_params)')}"
+                             transmission_hw_interface="$(arg transmission_hw_interface)"/>
 </robot>

Commit message: fixed length and collision typos

File: ur_description/urdf/ur.common.xacro (robot description, xacro)
@@ -104,37 +104,37 @@
     <xacro:property name="base_visual_material_name" value="${__base_mesh['visual']['material']['name']}" scope="parent"/>
     <xacro:property name="base_visual_material_color" value="${__base_mesh['visual']['material']['color']}" scope="parent"/>
-    <xacro:property name="base_colision_mesh" value="${__base_mesh['collision']['mesh']}" scope="parent"/>
+    <xacro:property name="base_collision_mesh" value="${__base_mesh['collision']['mesh']}" scope="parent"/>
     <xacro:property name="__shoulder_mesh" value="${__mesh_files['shoulder']}"/>
     <xacro:property name="shoulder_visual_mesh" value="${__shoulder_mesh['visual']['mesh']}" scope="parent"/>
     <xacro:property name="shoulder_visual_material_name" value="${__shoulder_mesh['visual']['material']['name']}" scope="parent"/>
     <xacro:property name="shoulder_visual_material_color" value="${__shoulder_mesh['visual']['material']['color']}" scope="parent"/>
-    <xacro:property name="shoulder_colision_mesh" value="${__shoulder_mesh['collision']['mesh']}" scope="parent"/>
+    <xacro:property name="shoulder_collision_mesh" value="${__shoulder_mesh['collision']['mesh']}" scope="parent"/>
     <xacro:property name="__upper_arm_mesh" value="${__mesh_files['upper_arm']}"/>
     <xacro:property name="upper_arm_visual_mesh" value="${__upper_arm_mesh['visual']['mesh']}" scope="parent"/>
     <xacro:property name="upper_arm_visual_material_name" value="${__upper_arm_mesh['visual']['material']['name']}" scope="parent"/>
     <xacro:property name="upper_arm_visual_material_color" value="${__upper_arm_mesh['visual']['material']['color']}" scope="parent"/>
-    <xacro:property name="upper_arm_colision_mesh" value="${__upper_arm_mesh['collision']['mesh']}" scope="parent"/>
+    <xacro:property name="upper_arm_collision_mesh" value="${__upper_arm_mesh['collision']['mesh']}" scope="parent"/>
     <xacro:property name="__forearm_mesh" value="${__mesh_files['forearm']}"/>
     <xacro:property name="forearm_visual_mesh" value="${__forearm_mesh['visual']['mesh']}" scope="parent"/>
     <xacro:property name="forearm_visual_material_name" value="${__forearm_mesh['visual']['material']['name']}" scope="parent"/>
     <xacro:property name="forearm_visual_material_color" value="${__forearm_mesh['visual']['material']['color']}" scope="parent"/>
-    <xacro:property name="forearm_colision_mesh" value="${__forearm_mesh['collision']['mesh']}" scope="parent"/>
+    <xacro:property name="forearm_collision_mesh" value="${__forearm_mesh['collision']['mesh']}" scope="parent"/>
     <xacro:property name="__wrist_1_mesh" value="${__mesh_files['wrist_1']}"/>
     <xacro:property name="wrist_1_visual_mesh" value="${__wrist_1_mesh['visual']['mesh']}" scope="parent"/>
     <xacro:property name="wrist_1_visual_material_name" value="${__wrist_1_mesh['visual']['material']['name']}" scope="parent"/>
     <xacro:property name="wrist_1_visual_material_color" value="${__wrist_1_mesh['visual']['material']['color']}" scope="parent"/>
-    <xacro:property name="wrist_1_colision_mesh" value="${__wrist_1_mesh['collision']['mesh']}" scope="parent"/>
+    <xacro:property name="wrist_1_collision_mesh" value="${__wrist_1_mesh['collision']['mesh']}" scope="parent"/>
     <xacro:property name="__wrist_2_mesh" value="${__mesh_files['wrist_2']}"/>
     <xacro:property name="wrist_2_visual_mesh" value="${__wrist_2_mesh['visual']['mesh']}" scope="parent"/>
     <xacro:property name="wrist_2_visual_material_name" value="${__wrist_2_mesh['visual']['material']['name']}" scope="parent"/>
     <xacro:property name="wrist_2_visual_material_color" value="${__wrist_2_mesh['visual']['material']['color']}" scope="parent"/>
-    <xacro:property name="wrist_2_colision_mesh" value="${__wrist_2_mesh['collision']['mesh']}" scope="parent"/>
+    <xacro:property name="wrist_2_collision_mesh" value="${__wrist_2_mesh['collision']['mesh']}" scope="parent"/>
     <xacro:property name="__wrist_3_mesh" value="${__mesh_files['wrist_3']}"/>
     <xacro:property name="wrist_3_visual_mesh" value="${__wrist_3_mesh['visual']['mesh']}" scope="parent"/>
     <xacro:property name="wrist_3_visual_material_name" value="${__wrist_3_mesh['visual']['material']['name']}" scope="parent"/>
     <xacro:property name="wrist_3_visual_material_color" value="${__wrist_3_mesh['visual']['material']['color']}" scope="parent"/>
-    <xacro:property name="wrist_3_colision_mesh" value="${__wrist_3_mesh['collision']['mesh']}" scope="parent"/>
+    <xacro:property name="wrist_3_collision_mesh" value="${__wrist_3_mesh['collision']['mesh']}" scope="parent"/>
   </xacro:macro>
-  <xacro:macro name="compute_lenght" params="d1 a2 a3 d4 d5 d6 shoulder_offset elbow_offset">
+  <xacro:macro name="compute_length" params="d1 a2 a3 d4 d5 d6 shoulder_offset elbow_offset">
     <xacro:property name="shoulder_height" value="${d1}" scope="parent"/>
     <xacro:property name="upper_arm_length" value="${-a2}" scope="parent"/>

File: ur_description/urdf/ur.geometry.xacro (robot description, xacro)
@@ -12,5 +12,5 @@
                     physical_parameters_file="${physical_parameters_file}"
                     visual_parameters_file="${visual_parameters_file}"/>
-    <xacro:compute_lenght d1="${d1}" a2="${a2}" a3="${a3}"
+    <xacro:compute_length d1="${d1}" a2="${a2}" a3="${a3}"
                           d4="${d4}" d5="${d5}" d6="${d6}"
                           shoulder_offset="${shoulder_offset}" elbow_offset="${elbow_offset}"/>
@@ -26,5 +26,5 @@
       <collision>
         <geometry>
-          <mesh filename="${base_colision_mesh}"/>
+          <mesh filename="${base_collision_mesh}"/>
         </geometry>
       </collision>
@@ -53,5 +53,5 @@
       <collision>
         <geometry>
-          <mesh filename="${shoulder_colision_mesh}"/>
+          <mesh filename="${shoulder_collision_mesh}"/>
         </geometry>
       </collision>
@@ -80,5 +80,5 @@
       <collision>
         <geometry>
-          <mesh filename="${upper_arm_colision_mesh}"/>
+          <mesh filename="${upper_arm_collision_mesh}"/>
         </geometry>
       </collision>
@@ -107,5 +107,5 @@
       <collision>
         <geometry>
-          <mesh filename="${forearm_colision_mesh}"/>
+          <mesh filename="${forearm_collision_mesh}"/>
         </geometry>
       </collision>
@@ -134,5 +134,5 @@
       <collision>
         <geometry>
-          <mesh filename="${wrist_1_colision_mesh}"/>
+          <mesh filename="${wrist_1_collision_mesh}"/>
         </geometry>
       </collision>
@@ -161,5 +161,5 @@
       <collision>
         <geometry>
-          <mesh filename="${wrist_2_colision_mesh}"/>
+          <mesh filename="${wrist_2_collision_mesh}"/>
         </geometry>
       </collision>
@@ -188,5 +188,5 @@
       <collision>
         <geometry>
-          <mesh filename="${wrist_3_colision_mesh}"/>
+          <mesh filename="${wrist_3_collision_mesh}"/>
         </geometry>
       </collision>

Commit message: fixed internia config to match updated parameters

File: ur_description/urdf/ur.common.xacro (robot description, xacro)
@@ -55,4 +55,5 @@
     <xacro:property name="shoulder_offset" value="${__offsets['shoulder_offset']}" scope="parent"/>
     <xacro:property name="elbow_offset" value="${__offsets['elbow_offset']}" scope="parent"/>
+    <xacro:property name="upper_arm_inertia_offset" value="${__offsets['upper_arm_inertia_offset']}" scope="parent"/>
     <!-- INERTIA PARAMETERS -->
     <!-- mass -->
@@ -73,5 +74,4 @@
     <xacro:property name="upperarm_inertia_length" value="${__intertia_links['upperarm']['length']}" scope="parent"/>
     <xacro:property name="forearm_inertia_radius" value="${__intertia_links['forearm']['radius']}" scope="parent"/>
-    <xacro:property name="forearm_inertia_length" value="${__intertia_links['forearm']['length']}" scope="parent"/>
     <xacro:property name="wrist_1_inertia_radius" value="${__intertia_links['wrist_1']['radius']}" scope="parent"/>
     <xacro:property name="wrist_1_inertia_length" value="${__intertia_links['wrist_1']['length']}" scope="parent"/>

File: ur_description/urdf/ur.geometry.xacro (robot description, xacro)
@@ -84,5 +84,5 @@
       </collision>
       <xacro:cylinder_inertial radius="${upperarm_inertia_radius}" length="${-a2}" mass="${upper_arm_mass}">
-        <origin xyz="0.0 0.0 ${-a2/2.0}" rpy="0 0 0" />
+        <origin xyz="0.0 ${-upper_arm_inertia_offset} ${-a2/2.0}" rpy="0 0 0" />
       </xacro:cylinder_inertial>
     </link>
@@ -138,5 +138,5 @@
       </collision>
       <xacro:cylinder_inertial radius="${wrist_1_inertia_radius}" length="${wrist_1_inertia_length}"  mass="${wrist_1_mass}">
-        <origin xyz="0.0 0.0 0.0" rpy="0 0 0" />
+        <origin xyz="0.0 ${wrist_1_length} 0.0" rpy="0 0 0" />
       </xacro:cylinder_inertial>
     </link>
@@ -192,5 +192,5 @@
       </collision>
       <xacro:cylinder_inertial radius="${wrist_3_inertia_radius}" length="${wrist_3_inertia_length}"  mass="${wrist_3_mass}">
-        <origin xyz="0.0 ${wrist_3_length - 0.02} 0.0" rpy="0 0 0" />
+        <origin xyz="0.0 ${wrist_3_length - wrist_3_inertia_length/2} 0.0" rpy="${pi/2} 0 0" />
       </xacro:cylinder_inertial>
     </link>
