Commit message: Use full kinematics parameters in description
the kinematics parameters can be retrieved from a calibration mechanism
to precisely represent the robot's kinematics.

File: ur_description/urdf/ur.common.xacro (robot description, xacro)
@@ -14,5 +14,5 @@
     </inertial>
   </xacro:macro>
-  <xacro:macro name="read_model_data" params="joints_limits_parameters_file physical_parameters_file visual_parameters_file">
+  <xacro:macro name="read_model_data" params="joints_limits_parameters_file kinematics_parameters_file physical_parameters_file visual_parameters_file">
     <xacro:property name="__limits" value="${joints_limits_parameters_file['limits']}"/>
     <xacro:property name="__dh_parameters" value="${physical_parameters_file['dh_parameters']}"/>
@@ -20,4 +20,5 @@
     <xacro:property name="__inertia_parameters" value="${physical_parameters_file['inertia_parameters']}" />
     <xacro:property name="__mesh_files" value="${visual_parameters_file['mesh_files']}" />
+    <xacro:property name="__kinematics" value="${kinematics_parameters_file['kinematics']}" />
     <!-- JOINTS LIMIT PARAMETERS -->
     <xacro:property name="shoulder_pan_lower_limit" value="${__limits['shoulder_pan']['lower']}" scope="parent"/>
@@ -52,8 +53,44 @@
     <xacro:property name="d5" value="${__dh_parameters['d5']}" scope="parent"/>
     <xacro:property name="d6" value="${__dh_parameters['d6']}" scope="parent"/>
+    <!-- kinematics -->
+    <xacro:property name="shoulder_x" value="${__kinematics['shoulder']['x']}" scope="parent"/>
+    <xacro:property name="shoulder_y" value="${__kinematics['shoulder']['y']}" scope="parent"/>
+    <xacro:property name="shoulder_z" value="${__kinematics['shoulder']['z']}" scope="parent"/>
+    <xacro:property name="shoulder_roll" value="${__kinematics['shoulder']['roll']}" scope="parent"/>
+    <xacro:property name="shoulder_pitch" value="${__kinematics['shoulder']['pitch']}" scope="parent"/>
+    <xacro:property name="shoulder_yaw" value="${__kinematics['shoulder']['yaw']}" scope="parent"/>
+    <xacro:property name="upper_arm_x" value="${__kinematics['upper_arm']['x']}" scope="parent"/>
+    <xacro:property name="upper_arm_y" value="${__kinematics['upper_arm']['y']}" scope="parent"/>
+    <xacro:property name="upper_arm_z" value="${__kinematics['upper_arm']['z']}" scope="parent"/>
+    <xacro:property name="upper_arm_roll" value="${__kinematics['upper_arm']['roll']}" scope="parent"/>
+    <xacro:property name="upper_arm_pitch" value="${__kinematics['upper_arm']['pitch']}" scope="parent"/>
+    <xacro:property name="upper_arm_yaw" value="${__kinematics['upper_arm']['yaw']}" scope="parent"/>
+    <xacro:property name="forearm_x" value="${__kinematics['forearm']['x']}" scope="parent"/>
+    <xacro:property name="forearm_y" value="${__kinematics['forearm']['y']}" scope="parent"/>
+    <xacro:property name="forearm_z" value="${__kinematics['forearm']['z']}" scope="parent"/>
+    <xacro:property name="forearm_roll" value="${__kinematics['forearm']['roll']}" scope="parent"/>
+    <xacro:property name="forearm_pitch" value="${__kinematics['forearm']['pitch']}" scope="parent"/>
+    <xacro:property name="forearm_yaw" value="${__kinematics['forearm']['yaw']}" scope="parent"/>
+    <xacro:property name="wrist_1_x" value="${__kinematics['wrist_1']['x']}" scope="parent"/>
+    <xacro:property name="wrist_1_y" value="${__kinematics['wrist_1']['y']}" scope="parent"/>
+    <xacro:property name="wrist_1_z" value="${__kinematics['wrist_1']['z']}" scope="parent"/>
+    <xacro:property name="wrist_1_roll" value="${__kinematics['wrist_1']['roll']}" scope="parent"/>
+    <xacro:property name="wrist_1_pitch" value="${__kinematics['wrist_1']['pitch']}" scope="parent"/>
+    <xacro:property name="wrist_1_yaw" value="${__kinematics['wrist_1']['yaw']}" scope="parent"/>
+    <xacro:property name="wrist_2_x" value="${__kinematics['wrist_2']['x']}" scope="parent"/>
+    <xacro:property name="wrist_2_y" value="${__kinematics['wrist_2']['y']}" scope="parent"/>
+    <xacro:property name="wrist_2_z" value="${__kinematics['wrist_2']['z']}" scope="parent"/>
+    <xacro:property name="wrist_2_roll" value="${__kinematics['wrist_2']['roll']}" scope="parent"/>
+    <xacro:property name="wrist_2_pitch" value="${__kinematics['wrist_2']['pitch']}" scope="parent"/>
+    <xacro:property name="wrist_2_yaw" value="${__kinematics['wrist_2']['yaw']}" scope="parent"/>
+    <xacro:property name="wrist_3_x" value="${__kinematics['wrist_3']['x']}" scope="parent"/>
+    <xacro:property name="wrist_3_y" value="${__kinematics['wrist_3']['y']}" scope="parent"/>
+    <xacro:property name="wrist_3_z" value="${__kinematics['wrist_3']['z']}" scope="parent"/>
+    <xacro:property name="wrist_3_roll" value="${__kinematics['wrist_3']['roll']}" scope="parent"/>
+    <xacro:property name="wrist_3_pitch" value="${__kinematics['wrist_3']['pitch']}" scope="parent"/>
+    <xacro:property name="wrist_3_yaw" value="${__kinematics['wrist_3']['yaw']}" scope="parent"/>
     <!-- OFFSETS -->
     <xacro:property name="shoulder_offset" value="${__offsets['shoulder_offset']}" scope="parent"/>
     <xacro:property name="elbow_offset" value="${__offsets['elbow_offset']}" scope="parent"/>
-    <xacro:property name="upper_arm_inertia_offset" value="${__offsets['upper_arm_inertia_offset']}" scope="parent"/>
     <!-- INERTIA PARAMETERS -->
     <!-- mass -->
@@ -61,4 +98,5 @@
     <xacro:property name="shoulder_mass" value="${__inertia_parameters['shoulder_mass']}" scope="parent"/>
     <xacro:property name="upper_arm_mass" value="${__inertia_parameters['upper_arm_mass']}" scope="parent"/>
+    <xacro:property name="upper_arm_inertia_offset" value="${__inertia_parameters['upper_arm_inertia_offset']}" scope="parent"/>
     <xacro:property name="forearm_mass" value="${__inertia_parameters['forearm_mass']}" scope="parent"/>
     <xacro:property name="wrist_1_mass" value="${__inertia_parameters['wrist_1_mass']}" scope="parent"/>
@@ -74,4 +112,5 @@
     <xacro:property name="upperarm_inertia_length" value="${__intertia_links['upperarm']['length']}" scope="parent"/>
     <xacro:property name="forearm_inertia_radius" value="${__intertia_links['forearm']['radius']}" scope="parent"/>
+    <xacro:property name="forearm_inertia_length" value="${__intertia_links['forearm']['length']}" scope="parent"/>
     <xacro:property name="wrist_1_inertia_radius" value="${__intertia_links['wrist_1']['radius']}" scope="parent"/>
     <xacro:property name="wrist_1_inertia_length" value="${__intertia_links['wrist_1']['length']}" scope="parent"/>
@@ -125,4 +164,5 @@
     <xacro:property name="wrist_1_visual_material_color" value="${__wrist_1_mesh['visual']['material']['color']}" scope="parent"/>
     <xacro:property name="wrist_1_collision_mesh" value="${__wrist_1_mesh['collision']['mesh']}" scope="parent"/>
+    <xacro:property name="wrist_1_visual_offset" value="${__wrist_1_mesh['visual_offset']}" scope="parent"/>
     <xacro:property name="__wrist_2_mesh" value="${__mesh_files['wrist_2']}"/>
     <xacro:property name="wrist_2_visual_mesh" value="${__wrist_2_mesh['visual']['mesh']}" scope="parent"/>
@@ -130,4 +170,5 @@
     <xacro:property name="wrist_2_visual_material_color" value="${__wrist_2_mesh['visual']['material']['color']}" scope="parent"/>
     <xacro:property name="wrist_2_collision_mesh" value="${__wrist_2_mesh['collision']['mesh']}" scope="parent"/>
+    <xacro:property name="wrist_2_visual_offset" value="${__wrist_2_mesh['visual_offset']}" scope="parent"/>
     <xacro:property name="__wrist_3_mesh" value="${__mesh_files['wrist_3']}"/>
     <xacro:property name="wrist_3_visual_mesh" value="${__wrist_3_mesh['visual']['mesh']}" scope="parent"/>
@@ -135,12 +176,5 @@
     <xacro:property name="wrist_3_visual_material_color" value="${__wrist_3_mesh['visual']['material']['color']}" scope="parent"/>
     <xacro:property name="wrist_3_collision_mesh" value="${__wrist_3_mesh['collision']['mesh']}" scope="parent"/>
-  </xacro:macro>
-  <xacro:macro name="compute_length" params="d1 a2 a3 d4 d5 d6 shoulder_offset elbow_offset">
-    <xacro:property name="shoulder_height" value="${d1}" scope="parent"/>
-    <xacro:property name="upper_arm_length" value="${-a2}" scope="parent"/>
-    <xacro:property name="forearm_length" value="${-a3}" scope="parent"/>
-    <xacro:property name="wrist_1_length" value="${d4 - elbow_offset - shoulder_offset}" scope="parent"/>
-    <xacro:property name="wrist_2_length" value="${d5}" scope="parent"/>
-    <xacro:property name="wrist_3_length" value="${d6}" scope="parent"/>
+    <xacro:property name="wrist_3_visual_offset" value="${__wrist_3_mesh['visual_offset']}" scope="parent"/>
   </xacro:macro>
 </robot>

File: ur_description/urdf/ur_robot.macro.xacro (robot description, xacro)
@@ -1,29 +1,31 @@
 <?xml version="1.0"?>
 <robot xmlns:xacro="http://wiki.ros.org/xacro">
-<!--
+  <!--
   Author: Ludovic Delval
   Contributor: Felix Messmer, Kelsey Hawkins, Jimmy Da Silva, Ajit Krisshna N L, Muhammad Asif Rana
--->
+  -->
  <xacro:include filename="$(find ur_description)/urdf/ur.transmission.xacro" />
  <xacro:include filename="$(find ur_description)/urdf/ur.common.xacro" />
- <xacro:macro name="ur_robot" params="prefix joints_limits_parameters_file physical_parameters_file visual_parameters_file
+ <xacro:macro name="ur_robot" params="prefix joints_limits_parameters_file kinematics_parameters_file physical_parameters_file visual_parameters_file
                   transmission_hw_interface:=hardware_interface/PositionJointInterface
                   safety_limits:=false safety_pos_margin:=0.15 safety_k_position:=20">
     <xacro:read_model_data joints_limits_parameters_file="${joints_limits_parameters_file}"
+                    kinematics_parameters_file="${kinematics_parameters_file}"
                     physical_parameters_file="${physical_parameters_file}"
                     visual_parameters_file="${visual_parameters_file}"/>
-    <xacro:compute_length d1="${d1}" a2="${a2}" a3="${a3}"
-                          d4="${d4}" d5="${d5}" d6="${d6}"
-                          shoulder_offset="${shoulder_offset}" elbow_offset="${elbow_offset}"/>
+    <!-- This is for compatibility reasons, as transformation between base and base_link was always 180 degree in the ur_description -->
+    <xacro:property name="base_correction" value="${pi}" />
     <link name="${prefix}base_link" >
       <visual>
+        <origin xyz="0 0 0" rpy="0 0 ${base_correction}"/>
         <geometry>
           <mesh filename="${base_visual_mesh}"/>
         </geometry>
-        <material name="${base_visual_material_name}">
-          <color rgba="${base_visual_material_color}"/>
-        </material>
-      </visual>
-      <collision>
+        <material name="LightGrey">
+          <color rgba="0.7 0.7 0.7 1.0"/>
+        </material>
+      </visual>
+      <collision>
+        <origin xyz="0 0 0" rpy="0 0 ${base_correction}"/>
         <geometry>
           <mesh filename="${base_collision_mesh}"/>
@@ -37,12 +39,13 @@
       <parent link="${prefix}base_link" />
       <child link = "${prefix}shoulder_link" />
-      <origin xyz="0.0 0.0 ${shoulder_height}" rpy="0.0 0.0 0.0" />
+      <origin xyz="${shoulder_x} ${shoulder_y} ${shoulder_z}" rpy="${shoulder_roll} ${shoulder_pitch} ${shoulder_yaw + base_correction}" />
       <axis xyz="0 0 1" />
       <limit lower="${shoulder_pan_lower_limit}" upper="${shoulder_pan_upper_limit}"
-          effort="${shoulder_pan_effort_limit}" velocity="${shoulder_pan_velocity_limit}"/>
+        effort="${shoulder_pan_effort_limit}" velocity="${shoulder_pan_velocity_limit}"/>
       <dynamics damping="0.0" friction="0.0"/>
     </joint>
     <link name="${prefix}shoulder_link">
       <visual>
+        <origin xyz="0 0 0" rpy="0 0 ${pi}"/>
         <geometry>
           <mesh filename="${shoulder_visual_mesh}"/>
@@ -53,4 +56,5 @@
       </visual>
       <collision>
+        <origin xyz="0 0 0" rpy="0 0 ${pi}"/>
         <geometry>
           <mesh filename="${shoulder_collision_mesh}"/>
@@ -64,6 +68,6 @@
       <parent link="${prefix}shoulder_link" />
       <child link = "${prefix}upper_arm_link" />
-      <origin xyz="0.0 ${shoulder_offset} 0.0" rpy="0.0 ${pi / 2.0} 0.0" />
-      <axis xyz="0 1 0" />
+      <origin xyz="${upper_arm_x} ${upper_arm_y} ${upper_arm_z}" rpy="${upper_arm_roll} ${upper_arm_pitch} ${upper_arm_yaw}" />
+      <axis xyz="0 0 1" />
       <limit lower="${shoulder_lift_lower_limit}" upper="${shoulder_lift_upper_limit}"
         effort="${shoulder_lift_effort_limit}" velocity="${shoulder_lift_velocity_limit}"/>
@@ -75,4 +79,5 @@
     <link name="${prefix}upper_arm_link">
       <visual>
+        <origin xyz="0 0 ${shoulder_offset}" rpy="${pi/2} 0 ${-pi/2}"/>
         <geometry>
           <mesh filename="${upper_arm_visual_mesh}"/>
@@ -83,10 +88,11 @@
       </visual>
       <collision>
+        <origin xyz="0 0 ${shoulder_offset}" rpy="${pi/2} 0 ${-pi/2}"/>
         <geometry>
           <mesh filename="${upper_arm_collision_mesh}"/>
         </geometry>
       </collision>
-      <xacro:cylinder_inertial radius="${upperarm_inertia_radius}" length="${upper_arm_length}" mass="${upper_arm_mass}">
-        <origin xyz="0.0 ${-upper_arm_inertia_offset} ${upper_arm_length/2.0}" rpy="0 0 0" />
+      <xacro:cylinder_inertial radius="${upperarm_inertia_radius}" length="${upperarm_inertia_length}" mass="${upper_arm_mass}">
+        <origin xyz="${-0.5 * upperarm_inertia_length} 0.0 ${upper_arm_inertia_offset}" rpy="0 ${pi/2} 0" />
       </xacro:cylinder_inertial>
     </link>
@@ -94,6 +100,6 @@
       <parent link="${prefix}upper_arm_link" />
       <child link = "${prefix}forearm_link" />
-      <origin xyz="0.0 ${elbow_offset} ${upper_arm_length}" rpy="0.0 0.0 0.0" />
-      <axis xyz="0 1 0" />
+      <origin xyz="${forearm_x} ${forearm_y} ${forearm_z}" rpy="${forearm_roll} ${forearm_pitch} ${forearm_yaw}" />
+      <axis xyz="0 0 1" />
       <limit lower="${elbow_joint_lower_limit}" upper="${elbow_joint_upper_limit}"
         effort="${elbow_joint_effort_limit}" velocity="${elbow_joint_velocity_limit}"/>
@@ -105,5 +111,6 @@
     <link name="${prefix}forearm_link">
       <visual>
-         <geometry>
+        <origin xyz="0 0 ${elbow_offset}" rpy="${pi/2} 0 ${-pi/2}"/>
+        <geometry>
           <mesh filename="${forearm_visual_mesh}"/>
         </geometry>
@@ -113,10 +120,11 @@
       </visual>
       <collision>
+        <origin xyz="0 0 ${elbow_offset}" rpy="${pi/2} 0 ${-pi/2}"/>
         <geometry>
           <mesh filename="${forearm_collision_mesh}"/>
         </geometry>
       </collision>
-      <xacro:cylinder_inertial radius="${forearm_inertia_radius}" length="${forearm_length}"  mass="${forearm_mass}">
-        <origin xyz="0.0 0.0 ${forearm_length/2.0}" rpy="0 0 0" />
+      <xacro:cylinder_inertial radius="${forearm_inertia_radius}" length="${forearm_inertia_length}"  mass="${forearm_mass}">
+        <origin xyz="${-0.5 * forearm_inertia_length} 0.0 ${elbow_offset}" rpy="0 ${pi/2} 0" />
       </xacro:cylinder_inertial>
     </link>
@@ -124,6 +132,6 @@
       <parent link="${prefix}forearm_link" />
       <child link = "${prefix}wrist_1_link" />
-      <origin xyz="0.0 0.0 ${forearm_length}" rpy="0.0 ${pi / 2.0} 0.0" />
-      <axis xyz="0 1 0" />
+      <origin xyz="${wrist_1_x} ${wrist_1_y} ${wrist_1_z}" rpy="${wrist_1_roll} ${wrist_1_pitch} ${wrist_1_yaw}" />
+      <axis xyz="0 0 1" />
       <limit lower="${wrist_1_lower_limit}" upper="${wrist_1_upper_limit}"
         effort="${wrist_1_effort_limit}" velocity="${wrist_1_velocity_limit}"/>
@@ -135,4 +143,6 @@
     <link name="${prefix}wrist_1_link">
       <visual>
+        <!-- TODO: Move this to a parameter -->
+        <origin xyz="0 0 ${wrist_1_visual_offset}" rpy="${pi/2} 0 0"/>
         <geometry>
           <mesh filename="${wrist_1_visual_mesh}"/>
@@ -143,4 +153,5 @@
       </visual>
       <collision>
+        <origin xyz="0 0 ${wrist_1_visual_offset}" rpy="${pi/2} 0 0"/>
         <geometry>
           <mesh filename="${wrist_1_collision_mesh}"/>
@@ -148,5 +159,5 @@
       </collision>
       <xacro:cylinder_inertial radius="${wrist_1_inertia_radius}" length="${wrist_1_inertia_length}"  mass="${wrist_1_mass}">
-        <origin xyz="0.0 ${wrist_1_length} 0.0" rpy="0 0 0" />
+        <origin xyz="0.0 0.0 0.0" rpy="0 0 0" />
       </xacro:cylinder_inertial>
     </link>
@@ -154,5 +165,5 @@
       <parent link="${prefix}wrist_1_link" />
       <child link = "${prefix}wrist_2_link" />
-      <origin xyz="0.0 ${wrist_1_length} 0.0" rpy="0.0 0.0 0.0" />
+      <origin xyz="${wrist_2_x} ${wrist_2_y} ${wrist_2_z}" rpy="${wrist_2_roll} ${wrist_2_pitch} ${wrist_2_yaw}" />
       <axis xyz="0 0 1" />
       <limit lower="${wrist_2_lower_limit}" upper="${wrist_2_upper_limit}"
@@ -165,4 +176,5 @@
     <link name="${prefix}wrist_2_link">
       <visual>
+        <origin xyz="0 0 ${wrist_2_visual_offset}" rpy="0 0 0"/>
         <geometry>
           <mesh filename="${wrist_2_visual_mesh}"/>
@@ -173,4 +185,5 @@
       </visual>
       <collision>
+        <origin xyz="0 0 ${wrist_2_visual_offset}" rpy="0 0 0"/>
         <geometry>
           <mesh filename="${wrist_2_collision_mesh}"/>
@@ -178,5 +191,5 @@
       </collision>
       <xacro:cylinder_inertial radius="${wrist_2_inertia_radius}" length="${wrist_2_inertia_length}"  mass="${wrist_2_mass}">
-        <origin xyz="0.0 0.0 ${wrist_2_length}" rpy="0 0 0" />
+        <origin xyz="0.0 0.0 0.0" rpy="0 0 0" />
       </xacro:cylinder_inertial>
     </link>
@@ -184,6 +197,6 @@
       <parent link="${prefix}wrist_2_link" />
       <child link = "${prefix}wrist_3_link" />
-      <origin xyz="0.0 0.0 ${wrist_2_length}" rpy="0.0 0.0 0.0" />
-      <axis xyz="0 1 0" />
+      <origin xyz="${wrist_3_x} ${wrist_3_y} ${wrist_3_z}" rpy="${wrist_3_roll} ${wrist_3_pitch} ${wrist_3_yaw}" />
+      <axis xyz="0 0 1" />
       <limit lower="${wrist_3_lower_limit}" upper="${wrist_3_upper_limit}"
              effort="${wrist_3_effort_limit}" velocity="${wrist_3_velocity_limit}"/>
@@ -195,4 +208,5 @@
     <link name="${prefix}wrist_3_link">
       <visual>
+        <origin xyz="0 0 ${wrist_3_visual_offset}" rpy="${pi/2} 0 0"/>
         <geometry>
           <mesh filename="${wrist_3_visual_mesh}"/>
@@ -203,4 +217,5 @@
       </visual>
       <collision>
+        <origin xyz="0 0 ${wrist_3_visual_offset}" rpy="${pi/2} 0 0"/>
         <geometry>
           <mesh filename="${wrist_3_collision_mesh}"/>
@@ -208,5 +223,5 @@
       </collision>
       <xacro:cylinder_inertial radius="${wrist_3_inertia_radius}" length="${wrist_3_inertia_length}"  mass="${wrist_3_mass}">
-        <origin xyz="0.0 ${wrist_3_length - wrist_3_inertia_length/2} 0.0" rpy="${pi/2} 0 0" />
+        <origin xyz="0.0 0.0 ${-0.5 * wrist_3_inertia_length}" rpy="0 0 0" />
       </xacro:cylinder_inertial>
     </link>
@@ -214,5 +229,5 @@
       <parent link="${prefix}wrist_3_link" />
       <child link = "${prefix}ee_link" />
-      <origin xyz="0.0 ${wrist_3_length} 0.0" rpy="0.0 0.0 ${pi/2.0}" />
+      <origin xyz="0.0 0.0 0.0" rpy="0.0 ${-pi/2.0} ${pi/2.0}" />
     </joint>
     <link name="${prefix}ee_link">
@@ -224,4 +239,9 @@
       </collision>
     </link>
+    <joint name="${prefix}wrist_3_passive_joint" type="fixed">
+      <origin xyz="0 0 0" rpy="0 0 0"/>
+      <parent link="${prefix}wrist_3_link"/>
+      <child link="${prefix}tool0"/>
+    </joint>
     <xacro:ur_arm_transmission prefix="${prefix}" hw_interface="${transmission_hw_interface}" />
     <!-- ROS base_link to UR 'Base' Coordinates transform -->
@@ -229,6 +249,6 @@
     <joint name="${prefix}base_link-base_fixed_joint" type="fixed">
       <!-- NOTE: this rotation is only needed as long as base_link itself is
-                 not corrected wrt the real robot (ie: rotated over 180
-                 degrees)
+      not corrected wrt the real robot (ie: rotated over 180
+      degrees)
       -->
       <origin xyz="0 0 0" rpy="0 0 ${-pi}"/>
@@ -238,9 +258,4 @@
     <!-- Frame coincident with all-zeros TCP on UR controller -->
     <link name="${prefix}tool0"/>
-    <joint name="${prefix}wrist_3_link-tool0_fixed_joint" type="fixed">
-      <origin xyz="0 ${wrist_3_length} 0" rpy="${pi/-2.0} 0 0"/>
-      <parent link="${prefix}wrist_3_link"/>
-      <child link="${prefix}tool0"/>
-    </joint>
   </xacro:macro>
 </robot>

File: ur_description/urdf/ur_robot.urdf.xacro (robot description, xacro)
@@ -4,4 +4,5 @@
    <!-- parameters -->
    <xacro:arg name="joints_limits_params" default=""/>
+   <xacro:arg name="kinematics_params" default=""/>
    <xacro:arg name="physical_params" default=""/>
    <xacro:arg name="visual_params" default=""/>
@@ -14,4 +15,5 @@
    <!-- arm -->
    <xacro:ur_robot prefix="" joints_limits_parameters_file="${load_yaml('$(arg joints_limits_params)')}"
+                             kinematics_parameters_file="${load_yaml('$(arg kinematics_params)')}"
                              physical_parameters_file="${load_yaml('$(arg physical_params)')}"
                              visual_parameters_file="${load_yaml('$(arg visual_params)')}"

File: ur_gazebo/urdf/ur_robot.urdf.xacro (robot description, xacro)
@@ -5,4 +5,5 @@
    <xacro:arg name="joints_limits_params" default="$(find ur_description)/config/ur3/joints_limits_parameters.yaml"/>
    <xacro:arg name="physical_params" default="$(find ur_description)/config/ur3/physical_parameters.yaml"/>
+   <xacro:arg name="kinematics_params" default="$(find ur_description)/config/ur3/default_kinematics.yaml"/>
    <xacro:arg name="visual_params" default="$(find ur_description)/config/ur3/visual_parameters.yaml"/>
    <xacro:arg name="transmission_hw_interface" default="hardware_interface/PositionJointInterface"/>
@@ -15,4 +16,5 @@
    <!-- arm -->
    <xacro:ur_gazebo_robot prefix="" joints_limits_parameters_file="${load_yaml('$(arg joints_limits_params)')}"
+                             kinematics_parameters_file="${load_yaml('$(arg kinematics_params)')}"
                              physical_parameters_file="${load_yaml('$(arg physical_params)')}"
                              visual_parameters_file="${load_yaml('$(arg visual_params)')}"
