Commit message: Updated urdf files use collision/visual models.

File: ur_description/urdf/ur10.urdf.xacro (robot description, xacro)
@@ -42,19 +42,19 @@
   <property name="elbow_collision_length" value="0.200" />
   <property name="elbow_collision_offset" value="0.035" />
-  <xacro:macro name="ur10_robot" params="parent name *origin">
-	<!-- joint between base_link and ur_base_link -->
-	<joint name="${name}_base_joint" type="fixed" >
-		<insert_block name="origin" />
-		<parent link="${parent}" />
-		<child link="${name}_base_link" />
-	</joint>
-	<link name="${name}_base_link" >
-		<visual>
-		  <geometry>
-		    <mesh filename="package://ur_description/meshes/ur10/Base.stl" />
+  <xacro:macro name="ur10_robot" params="prefix">
+	<link name="${prefix}base_link" >
+		<visual>
+		  <geometry>
+		    <mesh filename="package://ur_description/meshes/ur10/visual/Base.stl" />
 		  </geometry>
 		  <origin xyz="0.0 0.0 0.003" rpy="0.0 0.0 ${3.0 * pi / 4.0}" />
 		  <material name="UR/Blue" />
 		</visual>
+		<collision>
+		  <geometry>
+		    <mesh filename="package://ur_description/meshes/ur10/collision/Base.stl" />
+		  </geometry>
+		  <origin xyz="0.0 0.0 0.003" rpy="0.0 0.0 ${3.0 * pi / 4.0}" />
+		</collision>
 		<inertial>
 		  <mass value="${base_mass}" />
@@ -62,7 +62,7 @@
 		</inertial>
 	</link>
-	<joint name="${name}_shoulder_pan_joint" type="revolute">
-		<parent link="${name}_base_link" />
-		<child link = "${name}_shoulder_link" />
+	<joint name="${prefix}shoulder_pan_joint" type="revolute">
+		<parent link="${prefix}base_link" />
+		<child link = "${prefix}shoulder_link" />
 		<origin xyz="0.0 0.0 ${shoulder_height}" rpy="0.0 0.0 0.0" />
 		<axis xyz="0.0 0.0 1.0" />
@@ -70,8 +70,8 @@
 		<dynamics damping="10" friction="0.1"/>
 	</joint>
-	<link name="${name}_shoulder_link">
-		<visual>
-		  <geometry>
-  		    <mesh filename="package://ur_description/meshes/ur10/Shoulder.stl" />
+	<link name="${prefix}shoulder_link">
+		<visual>
+		  <geometry>
+  		    <mesh filename="package://ur_description/meshes/ur10/visual/Shoulder.stl" />
 		  </geometry>
 		  <material name="UR/Grey" />
@@ -79,5 +79,5 @@
 		<collision>
 		  <geometry>
-		    <mesh filename="package://ur_description/meshes/ur10/Shoulder.stl" />
+		    <mesh filename="package://ur_description/meshes/ur10/collision/Shoulder.stl" />
 		  </geometry>
 		</collision>
@@ -88,7 +88,7 @@
 		</inertial>
 	</link>
-	<joint name="${name}_shoulder_lift_joint" type="revolute">
-		<parent link="${name}_shoulder_link" />
-		<child link = "${name}_upper_arm_link" />
+	<joint name="${prefix}shoulder_lift_joint" type="revolute">
+		<parent link="${prefix}shoulder_link" />
+		<child link = "${prefix}upper_arm_link" />
 		<origin xyz="0.0 ${shoulder_offset} 0.0" rpy="0.0 ${pi / 2.0} 0.0" />
 		<axis xyz="0.0 1.0 0.0" />
@@ -96,8 +96,8 @@
 		<dynamics damping="10" friction="0.1"/>
 	</joint>
-	<link name="${name}_upper_arm_link">
-		<visual>
-		  <geometry>
-		    <mesh filename="package://ur_description/meshes/ur10/UpperArm.stl" />
+	<link name="${prefix}upper_arm_link">
+		<visual>
+		  <geometry>
+		    <mesh filename="package://ur_description/meshes/ur10/visual/UpperArm.stl" />
 		  </geometry>
 		  <origin xyz="0.0 0.0 0.0" rpy="0.0 0.0 0.0" />
@@ -106,5 +106,5 @@
 		<collision>
 		  <geometry>
-		    <mesh filename="package://ur_description/meshes/ur10/UpperArm.stl" />
+		    <mesh filename="package://ur_description/meshes/ur10/collision/UpperArm.stl" />
 		  </geometry>
  		  <origin xyz="0.0 0.0 0.0" rpy="0.0 0.0 0.0" />
@@ -116,7 +116,7 @@
 		</inertial>
 	</link>
-	<joint name="${name}_elbow_joint" type="revolute">
-		<parent link="${name}_upper_arm_link" />
-		<child link = "${name}_forearm_link" />
+	<joint name="${prefix}elbow_joint" type="revolute">
+		<parent link="${prefix}upper_arm_link" />
+		<child link = "${prefix}forearm_link" />
 		<origin xyz="0.0 ${-elbow_offset} ${upper_arm_length}" rpy="0.0 0.0 0.0" />
 		<axis xyz="0.0 1.0 0.0" />
@@ -124,8 +124,8 @@
 		<dynamics damping="10" friction="0.1"/>
 	</joint>
-	<link name="${name}_forearm_link">
+	<link name="${prefix}forearm_link">
 		<visual>
  		  <geometry>
-		    <mesh filename="package://ur_description/meshes/ur10/Forearm.stl" />
+		    <mesh filename="package://ur_description/meshes/ur10/visual/Forearm.stl" />
 		  </geometry>
 		  <material name="UR/Grey" />
@@ -133,5 +133,5 @@
 		<collision>
 		  <geometry>
-		    <mesh filename="package://ur_description/meshes/ur10/Forearm.stl" />
+		    <mesh filename="package://ur_description/meshes/ur10/collision/Forearm.stl" />
 		  </geometry>
 		</collision>
@@ -142,7 +142,7 @@
 		</inertial>
 	</link>
-	<joint name="${name}_wrist_1_joint" type="revolute">
- 		<parent link="${name}_forearm_link" />
-		<child link = "${name}_wrist_1_link" />
+	<joint name="${prefix}wrist_1_joint" type="revolute">
+ 		<parent link="${prefix}forearm_link" />
+		<child link = "${prefix}wrist_1_link" />
 		<origin xyz="0.0 0.0 ${forearm_length}" rpy="0.0 ${pi / 2.0} 0.0" />
 		<axis xyz="0.0 1.0 0.0" />
@@ -150,8 +150,8 @@
 		<dynamics damping="10" friction="0.1"/>
 	</joint>
-	<link name="${name}_wrist_1_link">
-		<visual>
-		  <geometry>
-		    <mesh filename="package://ur_description/meshes/ur10/Wrist1.stl" />
+	<link name="${prefix}wrist_1_link">
+		<visual>
+		  <geometry>
+		    <mesh filename="package://ur_description/meshes/ur10/visual/Wrist1.stl" />
 		  </geometry>
 		  <origin xyz="0.0 ${wrist_1_length} 0.0" rpy="0.0 0 0.0" />
@@ -160,5 +160,5 @@
 		<collision>
 		  <geometry>
-		    <mesh filename="package://ur_description/meshes/ur10/Wrist1.stl" />
+		    <mesh filename="package://ur_description/meshes/ur10/collision/Wrist1.stl" />
 		  </geometry>
 		  <origin xyz="0.0 ${wrist_1_length} 0.0" rpy="0.0 0 0.0" />
@@ -170,7 +170,7 @@
 		</inertial>
 	</link>
-	  <joint name="${name}_wrist_2_joint" type="revolute">
-		<parent link="${name}_wrist_1_link" />
-		<child link = "${name}_wrist_2_link" />
+	  <joint name="${prefix}wrist_2_joint" type="revolute">
+		<parent link="${prefix}wrist_1_link" />
+		<child link = "${prefix}wrist_2_link" />
 		<origin xyz="0.0 ${wrist_1_length} 0.0" rpy="0.0 0.0 0.0" />
 		<axis xyz="0.0 0.0 1.0" />
@@ -178,8 +178,8 @@
 		<dynamics damping="10" friction="0.1"/>
 	</joint>
-	<link name="${name}_wrist_2_link">
-		<visual>
-		  <geometry>
-		    <mesh filename="package://ur_description/meshes/ur10/Wrist2.stl" />
+	<link name="${prefix}wrist_2_link">
+		<visual>
+		  <geometry>
+		    <mesh filename="package://ur_description/meshes/ur10/visual/Wrist2.stl" />
 		  </geometry>
 		  <origin xyz="0.0 0.0 ${wrist_2_length}" rpy="0.0 0.0 0.0" />
@@ -188,5 +188,5 @@
 		<collision>
 		  <geometry>
-		    <mesh filename="package://ur_description/meshes/ur10/Wrist2.stl" />
+		    <mesh filename="package://ur_description/meshes/ur10/collision/Wrist2.stl" />
 		  </geometry>
 		  <origin xyz="0.0 0.0 ${wrist_2_length}" rpy="0.0 0.0 0.0" />
@@ -198,7 +198,7 @@
 		</inertial>
 	</link>
-	<joint name="${name}_wrist_3_joint" type="revolute">
-		<parent link="${name}_wrist_2_link" />
-		<child link = "${name}_wrist_3_link" />
+	<joint name="${prefix}wrist_3_joint" type="revolute">
+		<parent link="${prefix}wrist_2_link" />
+		<child link = "${prefix}wrist_3_link" />
 		<origin xyz="0.0 0.0 ${wrist_2_length}" rpy="0.0 0.0 0.0" />
 		<axis xyz="0.0 1.0 0.0" />
@@ -206,8 +206,8 @@
 		<dynamics damping="10" friction="0.1"/>
 	</joint>
-	<link name="${name}_wrist_3_link">
-		<visual>
-		  <geometry>
-		    <mesh filename="package://ur_description/meshes/ur10/Wrist3.stl" />
+	<link name="${prefix}wrist_3_link">
+		<visual>
+		  <geometry>
+		    <mesh filename="package://ur_description/meshes/ur10/visual/Wrist3.stl" />
 		  </geometry>
  		  <origin xyz="0.0 ${wrist_3_length} 0.0" rpy="0.0 0.0 0" />
@@ -216,5 +216,5 @@
 		<collision>
 		  <geometry>
-		    <mesh filename="package://ur_description/meshes/ur10/Wrist3.stl" />
+		    <mesh filename="package://ur_description/meshes/ur10/collision/Wrist3.stl" />
 		  </geometry>
 		  <origin xyz="0.0 ${wrist_3_length} 0.0" rpy="0.0 0.0 0" />
@@ -226,6 +226,6 @@
 		</inertial>
 	</link>
-  <xacro:ur10_arm_transmission name="${name}" />
-  <xacro:ur10_arm_gazebo name="${name}" />
+  <xacro:ur10_arm_transmission name="${prefix}" />
+  <xacro:ur10_arm_gazebo name="${prefix}" />
   </xacro:macro>
 </robot>

File: ur_description/urdf/ur5.urdf.xacro (robot description, xacro)
@@ -4,6 +4,7 @@
        xmlns:interface="http://playerstage.sourceforge.net/gazebo/xmlschema/#interface"
        xmlns:xacro="http://ros.org/wiki/xacro">
-<include filename="$(find ur_description)/urdf/ur5.transmission.xacro" />
+  <include filename="$(find ur_description)/urdf/ur5.transmission.xacro" />
   <include filename="$(find ur_description)/urdf/ur5.gazebo.xacro" />
+  <include filename="$(find ur_description)/urdf/materials.urdf.xacro" />
 <!--
 DH for UR5:
@@ -228,31 +229,4 @@
   </joint>
   <link name="${prefix}ee_link" />
-  <!-- Extra links for collision model -->
-  <!-- Somehow don't work with gazebo TODO: fix this
-  <joint name="${prefix}shoulder_collision_joint" type="fixed">
-    <parent link="${prefix}upper_arm_link" />
-    <child link = "${prefix}shoulder_collision_link" />
-  </joint>
-  <link name="${prefix}shoulder_collision_link">
-    <collision>
-      <geometry>
-        <cylinder length="${shoulder_collision_length}" radius="${shoulder_radius}"/>
-      </geometry>
-      <origin xyz="0.0 ${-shoulder_collision_offset} 0.0" rpy="${-pi / 2.0} 0.0 0.0" />
-    </collision>
-  </link>
-  <joint name="${prefix}elbow_collision_joint" type="fixed">
-    <parent link="${prefix}upper_arm_link" />
-    <child link = "${prefix}elbow_collision_link" />
-  </joint>
-  <link name="${prefix}elbow_collision_link">
-    <collision>
-      <geometry>
-        <cylinder length="${elbow_collision_length}" radius="${elbow_radius}"/>
-      </geometry>
-      <origin xyz="0.0 ${-elbow_collision_offset} ${upper_arm_length}" rpy="${pi / 2.0} 0.0 0.0" />
-    </collision>
-  </link>
-  -->
   <xacro:ur_arm_transmission name="${prefix}" />
   <gazebo reference="universal_robot">

File: ur_description/urdf/ur5_robot.urdf.xacro (robot description, xacro)
@@ -7,5 +7,4 @@
   <!-- common stuff -->
   <include filename="$(find ur_description)/urdf/gazebo.urdf.xacro" />
-  <include filename="$(find ur_description)/urdf/materials.urdf.xacro" />
   <!-- ur5 -->
   <include filename="$(find ur_description)/urdf/ur5.urdf.xacro" />

Commit message: Update ur10.urdf.xacro
Corrected UR10's urdf to faithfully represent joint effort thresholds, velocity limits, and dynamics parameters.

File: ur_description/urdf/ur10.urdf.xacro (robot description, xacro)
@@ -67,6 +67,6 @@
 		<origin xyz="0.0 0.0 ${shoulder_height}" rpy="0.0 0.0 0.0" />
 		<axis xyz="0.0 0.0 1.0" />
-		<limit lower="${-2.0 * pi}" upper="${2.0 * pi}" effort="10.0" velocity="${pi}"/>
-		<dynamics damping="10" friction="0.1"/>
+		<limit lower="${-2.0 * pi}" upper="${2.0 * pi}" effort="330.0" velocity="2.16"/>
+		<dynamics damping="1.2" friction="0.0"/>
 	</joint>
 	<link name="${prefix}shoulder_link">
@@ -94,5 +94,5 @@
 		<axis xyz="0.0 1.0 0.0" />
 		<limit lower="${-2.0 * pi}" upper="${2.0 * pi}" effort="10.0" velocity="${pi}"/>
-		<dynamics damping="10" friction="0.1"/>
+		<dynamics damping="1.2" friction="0.0"/>
 	</joint>
 	<link name="${prefix}upper_arm_link">
@@ -121,6 +121,6 @@
 		<origin xyz="0.0 ${-elbow_offset} ${upper_arm_length}" rpy="0.0 0.0 0.0" />
 		<axis xyz="0.0 1.0 0.0" />
-		<limit lower="${-2.0 * pi}" upper="${2.0 * pi}" effort="10.0" velocity="${pi}"/>
-		<dynamics damping="10" friction="0.1"/>
+		<limit lower="${-2.0 * pi}" upper="${2.0 * pi}" effort="150.0" velocity="${pi}"/>
+		<dynamics damping="0.6" friction="0.0"/>
 	</joint>
 	<link name="${prefix}forearm_link">
@@ -147,6 +147,6 @@
 		<origin xyz="0.0 0.0 ${forearm_length}" rpy="0.0 ${pi / 2.0} 0.0" />
 		<axis xyz="0.0 1.0 0.0" />
-		<limit lower="${-2.0 * pi}" upper="${2.0 * pi}" effort="10.0" velocity="${pi}"/>
-		<dynamics damping="10" friction="0.1"/>
+		<limit lower="${-2.0 * pi}" upper="${2.0 * pi}" effort="54.0" velocity="${pi}"/>
+		<dynamics damping="0.6" friction="0.0"/>
 	</joint>
 	<link name="${prefix}wrist_1_link">
@@ -175,6 +175,6 @@
 		<origin xyz="0.0 ${wrist_1_length} 0.0" rpy="0.0 0.0 0.0" />
 		<axis xyz="0.0 0.0 1.0" />
-		<limit lower="${-2.0 * pi}" upper="${2.0 * pi}" effort="10.0" velocity="${pi}"/>
-		<dynamics damping="10" friction="0.1"/>
+		<limit lower="${-2.0 * pi}" upper="${2.0 * pi}" effort="54.0" velocity="${pi}"/>
+		<dynamics damping="0.6" friction="0.0"/>
 	</joint>
 	<link name="${prefix}wrist_2_link">
@@ -203,6 +203,6 @@
 		<origin xyz="0.0 0.0 ${wrist_2_length}" rpy="0.0 0.0 0.0" />
 		<axis xyz="0.0 1.0 0.0" />
-		<limit lower="${-2.0 * pi}" upper="${2.0 * pi}" effort="10.0" velocity="${pi}"/>
-		<dynamics damping="10" friction="0.1"/>
+		<limit lower="${-2.0 * pi}" upper="${2.0 * pi}" effort="54.0" velocity="${pi}"/>
+		<dynamics damping="0.6" friction="0.0"/>
 	</joint>
 	<link name="${prefix}wrist_3_link">
