Commit message: increase effort limits

File: ur_description/urdf/ur10.urdf.xacro (robot description, xacro)
@@ -64,5 +64,5 @@
     <origin xyz="0.0 0.0 ${shoulder_height}" rpy="0.0 0.0 0.0" />
     <axis xyz="0.0 0.0 1.0" />
-    <limit lower="${-2.0 * pi}" upper="${2.0 * pi}" effort="330.0" velocity="2.16"/>
+    <limit lower="${-2.0 * pi}" upper="${2.0 * pi}" effort="1000.0" velocity="2.16"/>
     <dynamics damping="1.2" friction="0.0"/>
   </joint>
@@ -90,5 +90,5 @@
     <origin xyz="0.0 ${shoulder_offset} 0.0" rpy="0.0 ${pi / 2.0} 0.0" />
     <axis xyz="0.0 1.0 0.0" />
-    <limit lower="${-2.0 * pi}" upper="${2.0 * pi}" effort="10.0" velocity="${pi}"/>
+    <limit lower="${-2.0 * pi}" upper="${2.0 * pi}" effort="1000.0" velocity="${pi}"/>
     <dynamics damping="1.2" friction="0.0"/>
   </joint>
@@ -118,5 +118,5 @@
     <origin xyz="0.0 ${-elbow_offset} ${upper_arm_length}" rpy="0.0 0.0 0.0" />
     <axis xyz="0.0 1.0 0.0" />
-    <limit lower="${-2.0 * pi}" upper="${2.0 * pi}" effort="150.0" velocity="${pi}"/>
+    <limit lower="${-2.0 * pi}" upper="${2.0 * pi}" effort="1000.0" velocity="${pi}"/>
     <dynamics damping="0.6" friction="0.0"/>
   </joint>
@@ -144,5 +144,5 @@
     <origin xyz="0.0 0.0 ${forearm_length}" rpy="0.0 ${pi / 2.0} 0.0" />
     <axis xyz="0.0 1.0 0.0" />
-    <limit lower="${-2.0 * pi}" upper="${2.0 * pi}" effort="54.0" velocity="${pi}"/>
+    <limit lower="${-2.0 * pi}" upper="${2.0 * pi}" effort="1000.0" velocity="${pi}"/>
     <dynamics damping="0.6" friction="0.0"/>
   </joint>
@@ -172,5 +172,5 @@
     <origin xyz="0.0 ${wrist_1_length} 0.0" rpy="0.0 0.0 0.0" />
     <axis xyz="0.0 0.0 1.0" />
-    <limit lower="${-2.0 * pi}" upper="${2.0 * pi}" effort="54.0" velocity="${pi}"/>
+    <limit lower="${-2.0 * pi}" upper="${2.0 * pi}" effort="1000.0" velocity="${pi}"/>
     <dynamics damping="0.6" friction="0.0"/>
   </joint>
@@ -200,5 +200,5 @@
     <origin xyz="0.0 0.0 ${wrist_2_length}" rpy="0.0 0.0 0.0" />
     <axis xyz="0.0 1.0 0.0" />
-    <limit lower="${-2.0 * pi}" upper="${2.0 * pi}" effort="54.0" velocity="${pi}"/>
+    <limit lower="${-2.0 * pi}" upper="${2.0 * pi}" effort="1000.0" velocity="${pi}"/>
     <dynamics damping="0.6" friction="0.0"/>
   </joint>

File: ur_description/urdf/ur10_joint_limited.urdf.xacro (robot description, xacro)
@@ -64,5 +64,5 @@
     <origin xyz="0.0 0.0 ${shoulder_height}" rpy="0.0 0.0 0.0" />
     <axis xyz="0.0 0.0 1.0" />
-    <limit lower="${-pi}" upper="${pi}" effort="330.0" velocity="2.16"/>
+    <limit lower="${-pi}" upper="${pi}" effort="1000.0" velocity="2.16"/>
     <dynamics damping="1.2" friction="0.0"/>
   </joint>
@@ -90,5 +90,5 @@
     <origin xyz="0.0 ${shoulder_offset} 0.0" rpy="0.0 ${pi / 2.0} 0.0" />
     <axis xyz="0.0 1.0 0.0" />
-    <limit lower="${-pi}" upper="${pi}" effort="10.0" velocity="${pi}"/>
+    <limit lower="${-pi}" upper="${pi}" effort="1000.0" velocity="${pi}"/>
     <dynamics damping="1.2" friction="0.0"/>
   </joint>
@@ -118,5 +118,5 @@
     <origin xyz="0.0 ${-elbow_offset} ${upper_arm_length}" rpy="0.0 0.0 0.0" />
     <axis xyz="0.0 1.0 0.0" />
-    <limit lower="${-pi}" upper="${pi}" effort="150.0" velocity="${pi}"/>
+    <limit lower="${-pi}" upper="${pi}" effort="1000.0" velocity="${pi}"/>
     <dynamics damping="0.6" friction="0.0"/>
   </joint>
@@ -144,5 +144,5 @@
     <origin xyz="0.0 0.0 ${forearm_length}" rpy="0.0 ${pi / 2.0} 0.0" />
     <axis xyz="0.0 1.0 0.0" />
-    <limit lower="${-pi}" upper="${pi}" effort="54.0" velocity="${pi}"/>
+    <limit lower="${-pi}" upper="${pi}" effort="1000.0" velocity="${pi}"/>
     <dynamics damping="0.6" friction="0.0"/>
   </joint>
@@ -172,5 +172,5 @@
     <origin xyz="0.0 ${wrist_1_length} 0.0" rpy="0.0 0.0 0.0" />
     <axis xyz="0.0 0.0 1.0" />
-    <limit lower="${-pi}" upper="${pi}" effort="54.0" velocity="${pi}"/>
+    <limit lower="${-pi}" upper="${pi}" effort="1000.0" velocity="${pi}"/>
     <dynamics damping="0.6" friction="0.0"/>
   </joint>
@@ -200,5 +200,5 @@
     <origin xyz="0.0 0.0 ${wrist_2_length}" rpy="0.0 0.0 0.0" />
     <axis xyz="0.0 1.0 0.0" />
-    <limit lower="${-pi}" upper="${pi}" effort="54.0" velocity="${pi}"/>
+    <limit lower="${-pi}" upper="${pi}" effort="1000.0" velocity="${pi}"/>
     <dynamics damping="0.6" friction="0.0"/>
   </joint>

File: ur_description/urdf/ur5.urdf.xacro (robot description, xacro)
@@ -67,5 +67,5 @@
     <origin xyz="0.0 0.0 ${shoulder_height}" rpy="0.0 0.0 0.0" />
     <axis xyz="0 0 1" />
-    <limit lower="${-2.0 * pi}" upper="${2.0 * pi}" effort="150.0" velocity="${pi}"/>
+    <limit lower="${-2.0 * pi}" upper="${2.0 * pi}" effort="1000.0" velocity="${pi}"/>
     <dynamics damping="0.4" friction="0.0"/>
   </joint>
@@ -93,5 +93,5 @@
     <origin xyz="0.0 ${shoulder_offset} 0.0" rpy="0.0 ${pi / 2.0} 0.0" />
     <axis xyz="0 1 0" />
-    <limit lower="${-2.0 * pi}" upper="${2.0 * pi}" effort="150.0" velocity="${pi}"/>
+    <limit lower="${-2.0 * pi}" upper="${2.0 * pi}" effort="1000.0" velocity="${pi}"/>
     <dynamics damping="0.4" friction="0.0"/>
   </joint>
@@ -120,5 +120,5 @@
     <origin xyz="0.0 ${-elbow_offset} ${upper_arm_length}" rpy="0.0 0.0 0.0" />
     <axis xyz="0 1 0" />
-    <limit lower="${-2.0 * pi}" upper="${2.0 * pi}" effort="150.0" velocity="${pi}"/>
+    <limit lower="${-2.0 * pi}" upper="${2.0 * pi}" effort="1000.0" velocity="${pi}"/>
     <dynamics damping="0.4" friction="0.0"/>
   </joint>
@@ -146,5 +146,5 @@
     <origin xyz="0.0 0.0 ${forearm_length}" rpy="0.0 ${pi / 2.0} 0.0" />
     <axis xyz="0 1 0" />
-    <limit lower="${-1.0 * pi}" upper="${0.25 * pi}" effort="28.0" velocity="${pi}"/>
+    <limit lower="${-1.0 * pi}" upper="${0.25 * pi}" effort="1000.0" velocity="${pi}"/>
     <dynamics damping="0.3" friction="0.0"/>
   </joint>
@@ -173,5 +173,5 @@
     <origin xyz="0.0 ${wrist_1_length} 0.0" rpy="0.0 0.0 0.0" />
     <axis xyz="0 0 1" />
-    <limit lower="${-1.0 * pi}" upper="${1.0 * pi}" effort="28.0" velocity="${pi}"/>
+    <limit lower="${-1.0 * pi}" upper="${1.0 * pi}" effort="1000.0" velocity="${pi}"/>
     <dynamics damping="0.3" friction="0.0"/>
   </joint>
@@ -200,5 +200,5 @@
     <origin xyz="0.0 0.0 ${wrist_2_length}" rpy="0.0 0.0 0.0" />
     <axis xyz="0 1 0" />
-    <limit lower="${-1.0 * pi}" upper="${1.0 * pi}" effort="28.0" velocity="${pi}"/>
+    <limit lower="${-1.0 * pi}" upper="${1.0 * pi}" effort="1000.0" velocity="${pi}"/>
     <dynamics damping="0.3" friction="0.0"/>
   </joint>

File: ur_description/urdf/ur5_joint_limited.urdf.xacro (robot description, xacro)
@@ -67,5 +67,5 @@
     <origin xyz="0.0 0.0 ${shoulder_height}" rpy="0.0 0.0 0.0" />
     <axis xyz="0 0 1" />
-    <limit lower="${-pi}" upper="${pi}" effort="150.0" velocity="${pi}"/>
+    <limit lower="${-pi}" upper="${pi}" effort="1000.0" velocity="${pi}"/>
     <dynamics damping="0.4" friction="0.0"/>
   </joint>
@@ -93,5 +93,5 @@
     <origin xyz="0.0 ${shoulder_offset} 0.0" rpy="0.0 ${pi / 2.0} 0.0" />
     <axis xyz="0 1 0" />
-    <limit lower="${-pi}" upper="${pi}" effort="150.0" velocity="${pi}"/>
+    <limit lower="${-pi}" upper="${pi}" effort="1000.0" velocity="${pi}"/>
     <dynamics damping="0.4" friction="0.0"/>
   </joint>
@@ -120,5 +120,5 @@
     <origin xyz="0.0 ${-elbow_offset} ${upper_arm_length}" rpy="0.0 0.0 0.0" />
     <axis xyz="0 1 0" />
-    <limit lower="${-pi}" upper="${pi}" effort="150.0" velocity="${pi}"/>
+    <limit lower="${-pi}" upper="${pi}" effort="1000.0" velocity="${pi}"/>
     <dynamics damping="0.4" friction="0.0"/>
   </joint>
@@ -146,5 +146,5 @@
     <origin xyz="0.0 0.0 ${forearm_length}" rpy="0.0 ${pi / 2.0} 0.0" />
     <axis xyz="0 1 0" />
-    <limit lower="${-1.0 * pi}" upper="${0.25 * pi}" effort="28.0" velocity="${pi}"/>
+    <limit lower="${-1.0 * pi}" upper="${0.25 * pi}" effort="1000.0" velocity="${pi}"/>
     <dynamics damping="0.3" friction="0.0"/>
   </joint>
@@ -173,5 +173,5 @@
     <origin xyz="0.0 ${wrist_1_length} 0.0" rpy="0.0 0.0 0.0" />
     <axis xyz="0 0 1" />
-    <limit lower="${-1.0 * pi}" upper="${1.0 * pi}" effort="28.0" velocity="${pi}"/>
+    <limit lower="${-1.0 * pi}" upper="${1.0 * pi}" effort="1000.0" velocity="${pi}"/>
     <dynamics damping="0.3" friction="0.0"/>
   </joint>
@@ -200,5 +200,5 @@
     <origin xyz="0.0 0.0 ${wrist_2_length}" rpy="0.0 0.0 0.0" />
     <axis xyz="0 1 0" />
-    <limit lower="${-1.0 * pi}" upper="${1.0 * pi}" effort="28.0" velocity="${pi}"/>
+    <limit lower="${-1.0 * pi}" upper="${1.0 * pi}" effort="1000.0" velocity="${pi}"/>
     <dynamics damping="0.3" friction="0.0"/>
   </joint>

Commit message: Changing base_link to ur_base_link in the description and making base_link a dummy link to better support MoveIt.

File: ur_description/urdf/ur10.urdf.xacro (robot description, xacro)
@@ -41,4 +41,11 @@
   <xacro:macro name="ur10_robot" params="prefix">
   <link name="${prefix}base_link" >
+  </link>
+  <joint name="${prefix}base_link_joint" type="fixed">
+    <parent link="${prefix}base_link" />
+    <child link = "${prefix}ur_base_link" />
+    <origin xyz="0.0 0.0 0.0" rpy="0.0 0.0 0.0" />
+  </joint>
+  <link name="${prefix}ur_base_link" >
     <visual>
       <geometry>
@@ -60,5 +67,5 @@
   </link>
   <joint name="${prefix}shoulder_pan_joint" type="revolute">
-    <parent link="${prefix}base_link" />
+    <parent link="${prefix}ur_base_link" />
     <child link = "${prefix}shoulder_link" />
     <origin xyz="0.0 0.0 ${shoulder_height}" rpy="0.0 0.0 0.0" />

File: ur_description/urdf/ur10_joint_limited.urdf.xacro (robot description, xacro)
@@ -41,4 +41,11 @@
   <xacro:macro name="ur10_robot" params="prefix">
   <link name="${prefix}base_link" >
+  </link>
+  <joint name="${prefix}base_link_joint" type="fixed">
+    <parent link="${prefix}base_link" />
+    <child link = "${prefix}ur_base_link" />
+    <origin xyz="0.0 0.0 0.0" rpy="0.0 0.0 0.0" />
+  </joint>
+  <link name="${prefix}ur_base_link" >
     <visual>
       <geometry>
@@ -60,5 +67,5 @@
   </link>
   <joint name="${prefix}shoulder_pan_joint" type="revolute">
-    <parent link="${prefix}base_link" />
+    <parent link="${prefix}ur_base_link" />
     <child link = "${prefix}shoulder_link" />
     <origin xyz="0.0 0.0 ${shoulder_height}" rpy="0.0 0.0 0.0" />

File: ur_description/urdf/ur5.urdf.xacro (robot description, xacro)
@@ -45,4 +45,11 @@
 <xacro:macro name="ur5_robot" params="prefix">
   <link name="${prefix}base_link" >
+  </link>
+  <joint name="${prefix}base_link_joint" type="fixed">
+    <parent link="${prefix}base_link" />
+    <child link = "${prefix}ur_base_link" />
+    <origin xyz="0.0 0.0 0.0" rpy="0.0 0.0 0.0" />
+  </joint>
+  <link name="${prefix}ur_base_link" >
     <visual>
       <geometry>
@@ -63,5 +70,5 @@
   </link>
   <joint name="${prefix}shoulder_pan_joint" type="revolute">
-    <parent link="${prefix}base_link" />
+    <parent link="${prefix}ur_base_link" />
     <child link = "${prefix}shoulder_link" />
     <origin xyz="0.0 0.0 ${shoulder_height}" rpy="0.0 0.0 0.0" />

File: ur_description/urdf/ur5_joint_limited.urdf.xacro (robot description, xacro)
@@ -45,4 +45,11 @@
 <xacro:macro name="ur5_robot" params="prefix">
   <link name="${prefix}base_link" >
+  </link>
+  <joint name="${prefix}base_link_joint" type="fixed">
+    <parent link="${prefix}base_link" />
+    <child link = "${prefix}ur_base_link" />
+    <origin xyz="0.0 0.0 0.0" rpy="0.0 0.0 0.0" />
+  </joint>
+  <link name="${prefix}ur_base_link" >
     <visual>
       <geometry>
@@ -63,5 +70,5 @@
   </link>
   <joint name="${prefix}shoulder_pan_joint" type="revolute">
-    <parent link="${prefix}base_link" />
+    <parent link="${prefix}ur_base_link" />
     <child link = "${prefix}shoulder_link" />
     <origin xyz="0.0 0.0 ${shoulder_height}" rpy="0.0 0.0 0.0" />
