Commit message: use new meshes

File: ur_description/urdf/ur10.urdf.xacro (robot description, xacro)
@@ -7,7 +7,5 @@
   <xacro:include filename="$(find ur_description)/urdf/ur10.transmission.xacro" />
   <xacro:include filename="$(find ur_description)/urdf/ur10.gazebo.xacro" />
-  <xacro:include filename="$(find ur_description)/urdf/materials.urdf.xacro" />
   <property name="pi" value="3.14159265" />
-  <property name="scale" value="0.001 0.001 0.001" />
   <!-- Inertia parameters -->
   <property name="base_mass" value="4.0" />  <!-- This mass might be incorrect -->
@@ -59,14 +57,11 @@
       <visual>
         <geometry>
-          <mesh filename="package://ur_description/meshes/ur10/visual/Base.dae" scale="${scale}"/>
-        </geometry>
-        <origin xyz="0.0 0.0 0.0" rpy="${pi / 2.0} 0.0 0.0" />
-        <material name="UR/Blue" />
-      </visual>
-      <collision>
-        <geometry>
-          <mesh filename="package://ur_description/meshes/ur10/collision/Base.dae" scale="${scale}"/>
-        </geometry>
-        <origin xyz="0.0 0.0 0.0" rpy="${pi / 2.0} 0.0 0.0" />
+          <mesh filename="package://ur_description/meshes/ur10/visual/Base.dae"/>
+        </geometry>
+      </visual>
+      <collision>
+        <geometry>
+          <mesh filename="package://ur_description/meshes/ur10/collision/Base.dae"/>
+        </geometry>
       </collision>
       <xacro:cylinder_inertial radius="0.075" length="0.038" mass="${base_mass}">
@@ -90,14 +85,11 @@
       <visual>
         <geometry>
-          <mesh filename="package://ur_description/meshes/ur10/visual/Shoulder.dae" scale="${scale}"/>
-        </geometry>
-        <origin rpy="${pi / 2.0} 0.0 0.0" xyz="0.0 0.0 -0.127"/>   <!-- -0.127 ????  -->
-        <material name="UR/Grey" />
-      </visual>
-      <collision>
-        <geometry>
-          <mesh filename="package://ur_description/meshes/ur10/collision/Shoulder.dae" scale="${scale}"/>
-        </geometry>
-        <origin rpy="${pi / 2.0} 0.0 0.0" xyz="0.0 0.0 -0.127"/>   <!-- -0.127 ????  -->
+          <mesh filename="package://ur_description/meshes/ur10/visual/Shoulder.dae"/>
+        </geometry>
+      </visual>
+      <collision>
+        <geometry>
+          <mesh filename="package://ur_description/meshes/ur10/collision/Shoulder.dae"/>
+        </geometry>
       </collision>
       <xacro:cylinder_inertial radius="0.075" length="0.178" mass="${shoulder_mass}">
@@ -121,14 +113,11 @@
       <visual>
         <geometry>
-          <mesh filename="package://ur_description/meshes/ur10/visual/UpperArm.dae" scale="${scale}"/>
-        </geometry>
-        <origin xyz="0.0 -0.221 -0.127" rpy="${pi / 2.0} 0.0 0.0" />  <!-- new offset-->
-        <material name="UR/Blue" />
-      </visual>
-      <collision>
-        <geometry>
-          <mesh filename="package://ur_description/meshes/ur10/collision/UpperArm.dae" scale="${scale}"/>
-        </geometry>
-        <origin xyz="0.0 -0.221 -0.127" rpy="${pi / 2.0} 0.0 0.0" />  <!-- new offset-->
+          <mesh filename="package://ur_description/meshes/ur10/visual/UpperArm.dae"/>
+        </geometry>
+      </visual>
+      <collision>
+        <geometry>
+          <mesh filename="package://ur_description/meshes/ur10/collision/UpperArm.dae"/>
+        </geometry>
       </collision>
       <xacro:cylinder_inertial radius="0.075" length="${-ur10_a2}" mass="${upper_arm_mass}">
@@ -152,14 +141,11 @@
       <visual>
          <geometry>
-          <mesh filename="package://ur_description/meshes/ur10/visual/Forearm.dae" scale="${scale}"/>
-        </geometry>
-        <origin xyz="0.0 -0.049 -0.739" rpy="${pi / 2.0} 0.0 0.0" />  <!-- new offset -->
-        <material name="UR/Grey" />
-      </visual>
-      <collision>
-        <geometry>
-          <mesh filename="package://ur_description/meshes/ur10/collision/Forearm.dae" scale="${scale}"/>
-        </geometry>
-        <origin xyz="0.0 -0.049 -0.739" rpy="${pi / 2.0} 0.0 0.0" />  <!-- new offset -->
+          <mesh filename="package://ur_description/meshes/ur10/visual/Forearm.dae"/>
+        </geometry>
+      </visual>
+      <collision>
+        <geometry>
+          <mesh filename="package://ur_description/meshes/ur10/collision/Forearm.dae"/>
+        </geometry>
       </collision>
       <xacro:cylinder_inertial radius="0.075" length="${-ur10_a3}" mass="${forearm_mass}">
@@ -183,14 +169,11 @@
       <visual>
         <geometry>
-          <mesh filename="package://ur_description/meshes/ur10/visual/Wrist1.dae" scale="${scale}"/>
-        </geometry>
-        <origin xyz="0.0 -0.049 -1.312" rpy="${pi / 2.0} 0 0.0" />  <!-- new offset -->
-        <material name="UR/Blue" />
-      </visual>
-      <collision>
-        <geometry>
-          <mesh filename="package://ur_description/meshes/ur10/collision/Wrist1.dae" scale="${scale}"/>
-        </geometry>
-        <origin xyz="0.0 -0.049 -1.312" rpy="${pi / 2.0} 0 0.0" />  <!-- new offset -->
+          <mesh filename="package://ur_description/meshes/ur10/visual/Wrist1.dae"/>
+        </geometry>
+      </visual>
+      <collision>
+        <geometry>
+          <mesh filename="package://ur_description/meshes/ur10/collision/Wrist1.dae"/>
+        </geometry>
       </collision>
       <xacro:cylinder_inertial radius="0.075" length="0.12" mass="${wrist_1_mass}">
@@ -214,14 +197,11 @@
       <visual>
         <geometry>
-          <mesh filename="package://ur_description/meshes/ur10/visual/Wrist2.dae" scale="${scale}"/>
-        </geometry>
-        <origin xyz="0.0 -0.164 -1.312" rpy="${pi / 2.0} 0.0 0.0" />  <!-- new offset -->
-        <material name="UR/Grey" />
-      </visual>
-      <collision>
-        <geometry>
-          <mesh filename="package://ur_description/meshes/ur10/collision/Wrist2.dae" scale="${scale}"/>
-        </geometry>
-        <origin xyz="0.0 -0.164 -1.312" rpy="${pi / 2.0} 0.0 0.0" />  <!-- new offset -->
+          <mesh filename="package://ur_description/meshes/ur10/visual/Wrist2.dae"/>
+        </geometry>
+      </visual>
+      <collision>
+        <geometry>
+          <mesh filename="package://ur_description/meshes/ur10/collision/Wrist2.dae"/>
+        </geometry>
       </collision>
       <xacro:cylinder_inertial radius="0.075" length="0.12" mass="${wrist_2_mass}">
@@ -245,14 +225,11 @@
       <visual>
         <geometry>
-          <mesh filename="package://ur_description/meshes/ur10/visual/Wrist3.dae" scale="${scale}"/>
-        </geometry>
-         <origin xyz="0.0 -0.164 -1.427" rpy="${pi / 2.0} 0.0 0" />   <!-- new offset -->
-        <material name="UR/Blue" />
-      </visual>
-      <collision>
-        <geometry>
-          <mesh filename="package://ur_description/meshes/ur10/collision/Wrist3.dae" scale="${scale}"/>
-        </geometry>
-         <origin xyz="0.0 -0.164 -1.427" rpy="${pi / 2.0} 0.0 0" />   <!-- new offset -->
+          <mesh filename="package://ur_description/meshes/ur10/visual/Wrist3.dae"/>
+        </geometry>
+      </visual>
+      <collision>
+        <geometry>
+          <mesh filename="package://ur_description/meshes/ur10/collision/Wrist3.dae"/>
+        </geometry>
       </collision>
       <xacro:cylinder_inertial radius="0.075" length="0.12" mass="${wrist_3_mass}">

File: ur_description/urdf/ur5.urdf.xacro (robot description, xacro)
@@ -3,7 +3,5 @@
   <xacro:include filename="$(find ur_description)/urdf/ur5.transmission.xacro" />
   <xacro:include filename="$(find ur_description)/urdf/ur5.gazebo.xacro" />
-  <xacro:include filename="$(find ur_description)/urdf/materials.urdf.xacro" />
   <property name="pi" value="3.14159265" />
-  <property name="scale" value="0.001 0.001 0.001" />
   <!-- Inertia parameters -->
   <property name="base_mass" value="4.0" />  <!-- This mass might be incorrect -->
@@ -76,5 +74,4 @@
           <mesh filename="package://ur_description/meshes/ur5/visual/Base.dae" />
         </geometry>
-        <origin xyz="0.0 0.0 0.003" rpy="0.0 0.0 ${3.0 * pi / 4.0}" />
       </visual>
       <collision>
@@ -82,5 +79,4 @@
           <mesh filename="package://ur_description/meshes/ur5/collision/Base.dae" />
         </geometry>
-        <!-- <origin rpy="0.0 0.0 0.0" xyz="0.0 0.0 -0.009159"/> -->
       </collision>
       <xacro:cylinder_inertial radius="0.06" length="0.05" mass="${base_mass}">
@@ -111,5 +107,4 @@
           <mesh filename="package://ur_description/meshes/ur5/collision/Shoulder.dae" />
         </geometry>
-        <!-- <origin rpy="0.0 0.0 0.0" xyz="0.0 0.0 -0.009159"/> -->
       </collision>
       <xacro:cylinder_inertial radius="0.06" length="0.15" mass="${shoulder_mass}">
@@ -135,5 +130,4 @@
           <mesh filename="package://ur_description/meshes/ur5/visual/UpperArm.dae" />
         </geometry>
-        <origin xyz="0.0 0.0 0.0" rpy="0.0 0.0 0.0" />
       </visual>
       <collision>
@@ -141,5 +135,4 @@
           <mesh filename="package://ur_description/meshes/ur5/collision/UpperArm.dae" />
         </geometry>
-        <!-- <origin rpy="0.0 0.0 0.0" xyz="0.0 0.0 0.2125"/> -->
       </collision>
       <xacro:cylinder_inertial radius="0.06" length="0.56" mass="${upper_arm_mass}">
@@ -170,5 +163,4 @@
           <mesh filename="package://ur_description/meshes/ur5/collision/Forearm.dae" />
         </geometry>
-        <!-- <origin rpy="0.0 0.0 0.0" xyz="0.0 0.0 0.196125"/> -->
       </collision>
       <xacro:cylinder_inertial radius="0.06" length="0.5" mass="${forearm_mass}">
@@ -194,5 +186,4 @@
           <mesh filename="package://ur_description/meshes/ur5/visual/Wrist1.dae" />
         </geometry>
-        <origin xyz="0.0 ${wrist_1_length} 0.0" rpy="0.0 ${pi / 2.0} 0.0" />
       </visual>
       <collision>
@@ -200,5 +191,4 @@
           <mesh filename="package://ur_description/meshes/ur5/collision/Wrist1.dae" />
         </geometry>
-        <origin rpy="0.0 1.570796325 0.0" xyz="0.0 0.093 0.0"/>
       </collision>
       <xacro:cylinder_inertial radius="0.6" length="0.12" mass="${wrist_1_mass}">
@@ -224,5 +214,4 @@
           <mesh filename="package://ur_description/meshes/ur5/visual/Wrist2.dae" />
         </geometry>
-        <origin xyz="0.0 0.0 ${wrist_2_length}" rpy="0.0 0.0 0.0" />
       </visual>
       <collision>
@@ -230,5 +219,4 @@
           <mesh filename="package://ur_description/meshes/ur5/collision/Wrist2.dae" />
         </geometry>
-         <origin rpy="0.0 0.0 0.0" xyz="0.0 0.0 0.09465"/>
       </collision>
       <xacro:cylinder_inertial radius="0.6" length="0.12" mass="${wrist_2_mass}">

Commit message: add color to avoid default color 'red' for collision meshes

File: ur_description/urdf/ur10.urdf.xacro (robot description, xacro)
@@ -59,4 +59,7 @@
           <mesh filename="package://ur_description/meshes/ur10/visual/Base.dae"/>
         </geometry>
+        <material name="LightGrey">
+          <color rgba="0.7 0.7 0.7 1.0"/>
+        </material>
       </visual>
       <collision>
@@ -87,4 +90,7 @@
           <mesh filename="package://ur_description/meshes/ur10/visual/Shoulder.dae"/>
         </geometry>
+        <material name="LightGrey">
+          <color rgba="0.7 0.7 0.7 1.0"/>
+        </material>
       </visual>
       <collision>
@@ -115,4 +121,7 @@
           <mesh filename="package://ur_description/meshes/ur10/visual/UpperArm.dae"/>
         </geometry>
+        <material name="LightGrey">
+          <color rgba="0.7 0.7 0.7 1.0"/>
+        </material>
       </visual>
       <collision>
@@ -143,4 +152,7 @@
           <mesh filename="package://ur_description/meshes/ur10/visual/Forearm.dae"/>
         </geometry>
+        <material name="LightGrey">
+          <color rgba="0.7 0.7 0.7 1.0"/>
+        </material>
       </visual>
       <collision>
@@ -171,4 +183,7 @@
           <mesh filename="package://ur_description/meshes/ur10/visual/Wrist1.dae"/>
         </geometry>
+        <material name="LightGrey">
+          <color rgba="0.7 0.7 0.7 1.0"/>
+        </material>
       </visual>
       <collision>
@@ -199,4 +214,7 @@
           <mesh filename="package://ur_description/meshes/ur10/visual/Wrist2.dae"/>
         </geometry>
+        <material name="LightGrey">
+          <color rgba="0.7 0.7 0.7 1.0"/>
+        </material>
       </visual>
       <collision>
@@ -227,4 +245,7 @@
           <mesh filename="package://ur_description/meshes/ur10/visual/Wrist3.dae"/>
         </geometry>
+        <material name="LightGrey">
+          <color rgba="0.7 0.7 0.7 1.0"/>
+        </material>
       </visual>
       <collision>

File: ur_description/urdf/ur5.urdf.xacro (robot description, xacro)
@@ -74,4 +74,7 @@
           <mesh filename="package://ur_description/meshes/ur5/visual/Base.dae" />
         </geometry>
+        <material name="LightGrey">
+          <color rgba="0.7 0.7 0.7 1.0"/>
+        </material>
       </visual>
       <collision>
@@ -102,4 +105,7 @@
           <mesh filename="package://ur_description/meshes/ur5/visual/Shoulder.dae" />
         </geometry>
+        <material name="LightGrey">
+          <color rgba="0.7 0.7 0.7 1.0"/>
+        </material>
       </visual>
       <collision>
@@ -130,4 +136,7 @@
           <mesh filename="package://ur_description/meshes/ur5/visual/UpperArm.dae" />
         </geometry>
+        <material name="LightGrey">
+          <color rgba="0.7 0.7 0.7 1.0"/>
+        </material>
       </visual>
       <collision>
@@ -158,4 +167,7 @@
           <mesh filename="package://ur_description/meshes/ur5/visual/Forearm.dae" />
         </geometry>
+        <material name="LightGrey">
+          <color rgba="0.7 0.7 0.7 1.0"/>
+        </material>
       </visual>
       <collision>
@@ -186,4 +198,7 @@
           <mesh filename="package://ur_description/meshes/ur5/visual/Wrist1.dae" />
         </geometry>
+        <material name="LightGrey">
+          <color rgba="0.7 0.7 0.7 1.0"/>
+        </material>
       </visual>
       <collision>
@@ -214,4 +229,7 @@
           <mesh filename="package://ur_description/meshes/ur5/visual/Wrist2.dae" />
         </geometry>
+        <material name="LightGrey">
+          <color rgba="0.7 0.7 0.7 1.0"/>
+        </material>
       </visual>
       <collision>
@@ -242,4 +260,7 @@
           <mesh filename="package://ur_description/meshes/ur5/visual/Wrist3.dae" />
         </geometry>
+        <material name="LightGrey">
+          <color rgba="0.7 0.7 0.7 1.0"/>
+        </material>
       </visual>
       <collision>

Commit message: description: add ROS-I base and tool0 frames. Fix #49 and #95.
Note that 'base' is essentially 'base_link' but rotated by 180
degrees over the Z-axis. This is necessary as the visual and
collision geometries appear to also have their origins rotated
180 degrees wrt the real robot.

'tool0' is similar to 'ee_link', but with its orientation such
that it coincides with an all-zeros TCP setting on the UR
controller. Users are expected to attach their own TCP frames
to this frame, instead of updating it (see also [1]).

[1] http://wiki.ros.org/Industrial/Tutorials/WorkingWithRosIndustrialRobotSupportPackages#Standardised_links_.2BAC8_frames

File: ur_description/urdf/ur10.urdf.xacro (robot description, xacro)
@@ -273,4 +273,22 @@
     <xacro:ur10_arm_transmission prefix="${prefix}" />
     <xacro:ur10_arm_gazebo prefix="${prefix}" />
+    <!-- ROS base_link to UR 'Base' Coordinates transform -->
+    <link name="${prefix}base"/>
+    <joint name="${prefix}base_link-base" type="fixed">
+      <!-- NOTE: this rotation is only needed as long as base_link itself is
+                 not corrected wrt the real robot (ie: rotated over 180
+                 degrees)
+      -->
+      <origin xyz="0 0 0" rpy="0 0 ${-pi}"/>
+      <parent link="${prefix}base_link"/>
+      <child link="${prefix}base"/>
+    </joint>
+    <!-- Frame coincident with all-zeros TCP on UR controller -->
+    <link name="${prefix}tool0"/>
+    <joint name="${prefix}wrist_3_link-tool0" type="fixed">
+      <origin xyz="0 ${wrist_3_length} 0" rpy="${pi/-2.0} 0 0"/>
+      <parent link="${prefix}wrist_3_link"/>
+      <child link="${prefix}tool0"/>
+    </joint>
   </xacro:macro>
 </robot>

File: ur_description/urdf/ur10_joint_limited_robot.urdf (robot description, URDF)
Before this commit: robot ur10, 9 links, 8 joints
Links:
- added link base
- added link tool0
Joints:
- added joint base_link-base: type fixed, parent base_link, child base, origin xyz=0 0 0 rpy=0 0 -3.14159265
- added joint wrist_3_link-tool0: type fixed, parent wrist_3_link, child tool0, origin xyz=0 0.0922 0 rpy=-1.570796325 0 0

File: ur_description/urdf/ur10_robot.urdf (robot description, URDF)
Before this commit: robot ur10, 9 links, 8 joints
Links:
- added link base
- added link tool0
Joints:
- added joint base_link-base: type fixed, parent base_link, child base, origin xyz=0 0 0 rpy=0 0 -3.14159265
- added joint wrist_3_link-tool0: type fixed, parent wrist_3_link, child tool0, origin xyz=0 0.0922 0 rpy=-1.570796325 0 0

File: ur_description/urdf/ur5.urdf.xacro (robot description, xacro)
@@ -288,4 +288,22 @@
     <xacro:ur5_arm_transmission prefix="${prefix}" />
     <xacro:ur5_arm_gazebo prefix="${prefix}" />
+    <!-- ROS base_link to UR 'Base' Coordinates transform -->
+    <link name="${prefix}base"/>
+    <joint name="${prefix}base_link-base" type="fixed">
+      <!-- NOTE: this rotation is only needed as long as base_link itself is
+                 not corrected wrt the real robot (ie: rotated over 180
+                 degrees)
+      -->
+      <origin xyz="0 0 0" rpy="0 0 ${-pi}"/>
+      <parent link="${prefix}base_link"/>
+      <child link="${prefix}base"/>
+    </joint>
+    <!-- Frame coincident with all-zeros TCP on UR controller -->
+    <link name="${prefix}tool0"/>
+    <joint name="${prefix}wrist_3_link-tool0" type="fixed">
+      <origin xyz="0 ${wrist_3_length} 0" rpy="${pi/-2.0} 0 0"/>
+      <parent link="${prefix}wrist_3_link"/>
+      <child link="${prefix}tool0"/>
+    </joint>
   </xacro:macro>
 </robot>

File: ur_description/urdf/ur5_joint_limited_robot.urdf (robot description, URDF)
Before this commit: robot ur5, 9 links, 8 joints
Links:
- added link base
- added link tool0
Joints:
- added joint base_link-base: type fixed, parent base_link, child base, origin xyz=0 0 0 rpy=0 0 -3.14159265
- added joint wrist_3_link-tool0: type fixed, parent wrist_3_link, child tool0, origin xyz=0 0.0823 0 rpy=-1.570796325 0 0

File: ur_description/urdf/ur5_robot.urdf (robot description, URDF)
Before this commit: robot ur5, 9 links, 8 joints
Links:
- added link base
- added link tool0
Joints:
- added joint base_link-base: type fixed, parent base_link, child base, origin xyz=0 0 0 rpy=0 0 -3.14159265
- added joint wrist_3_link-tool0: type fixed, parent wrist_3_link, child tool0, origin xyz=0 0.0823 0 rpy=-1.570796325 0 0

Commit message: description: add '_joint' suffix to newly introduced joint tags.
This is more in-line with naming of existing joint tags.

File: ur_description/urdf/ur10.urdf.xacro (robot description, xacro)
@@ -275,5 +275,5 @@
     <!-- ROS base_link to UR 'Base' Coordinates transform -->
     <link name="${prefix}base"/>
-    <joint name="${prefix}base_link-base" type="fixed">
+    <joint name="${prefix}base_link-base_fixed_joint" type="fixed">
       <!-- NOTE: this rotation is only needed as long as base_link itself is
                  not corrected wrt the real robot (ie: rotated over 180
@@ -286,5 +286,5 @@
     <!-- Frame coincident with all-zeros TCP on UR controller -->
     <link name="${prefix}tool0"/>
-    <joint name="${prefix}wrist_3_link-tool0" type="fixed">
+    <joint name="${prefix}wrist_3_link-tool0_fixed_joint" type="fixed">
       <origin xyz="0 ${wrist_3_length} 0" rpy="${pi/-2.0} 0 0"/>
       <parent link="${prefix}wrist_3_link"/>

File: ur_description/urdf/ur10_joint_limited_robot.urdf (robot description, URDF)
Before this commit: robot ur10, 11 links, 10 joints
Joints:
- removed joint base_link-base
- removed joint wrist_3_link-tool0
- added joint base_link-base_fixed_joint: type fixed, parent base_link, child base, origin xyz=0 0 0 rpy=0 0 -3.14159265
- added joint wrist_3_link-tool0_fixed_joint: type fixed, parent wrist_3_link, child tool0, origin xyz=0 0.0922 0 rpy=-1.570796325 0 0

File: ur_description/urdf/ur10_robot.urdf (robot description, URDF)
Before this commit: robot ur10, 11 links, 10 joints
Joints:
- removed joint base_link-base
- removed joint wrist_3_link-tool0
- added joint base_link-base_fixed_joint: type fixed, parent base_link, child base, origin xyz=0 0 0 rpy=0 0 -3.14159265
- added joint wrist_3_link-tool0_fixed_joint: type fixed, parent wrist_3_link, child tool0, origin xyz=0 0.0922 0 rpy=-1.570796325 0 0

File: ur_description/urdf/ur5.urdf.xacro (robot description, xacro)
@@ -290,5 +290,5 @@
     <!-- ROS base_link to UR 'Base' Coordinates transform -->
     <link name="${prefix}base"/>
-    <joint name="${prefix}base_link-base" type="fixed">
+    <joint name="${prefix}base_link-base_fixed_joint" type="fixed">
       <!-- NOTE: this rotation is only needed as long as base_link itself is
                  not corrected wrt the real robot (ie: rotated over 180
@@ -301,5 +301,5 @@
     <!-- Frame coincident with all-zeros TCP on UR controller -->
     <link name="${prefix}tool0"/>
-    <joint name="${prefix}wrist_3_link-tool0" type="fixed">
+    <joint name="${prefix}wrist_3_link-tool0_fixed_joint" type="fixed">
       <origin xyz="0 ${wrist_3_length} 0" rpy="${pi/-2.0} 0 0"/>
       <parent link="${prefix}wrist_3_link"/>

File: ur_description/urdf/ur5_joint_limited_robot.urdf (robot description, URDF)
Before this commit: robot ur5, 11 links, 10 joints
Joints:
- removed joint base_link-base
- removed joint wrist_3_link-tool0
- added joint base_link-base_fixed_joint: type fixed, parent base_link, child base, origin xyz=0 0 0 rpy=0 0 -3.14159265
- added joint wrist_3_link-tool0_fixed_joint: type fixed, parent wrist_3_link, child tool0, origin xyz=0 0.0823 0 rpy=-1.570796325 0 0

File: ur_description/urdf/ur5_robot.urdf (robot description, URDF)
Before this commit: robot ur5, 11 links, 10 joints
Joints:
- removed joint base_link-base
- removed joint wrist_3_link-tool0
- added joint base_link-base_fixed_joint: type fixed, parent base_link, child base, origin xyz=0 0 0 rpy=0 0 -3.14159265
- added joint wrist_3_link-tool0_fixed_joint: type fixed, parent wrist_3_link, child tool0, origin xyz=0 0.0823 0 rpy=-1.570796325 0 0
