Commit message: Fix overlapping properties between robot definitions
Uploading a different UR definition used to break the previous definition files by overwriting their link lengths. This commit makes the property names for each robot unique so they are independent of the other robot models.

File: ur_description/urdf/ur5.urdf.xacro (robot description, xacro)
@@ -4,17 +4,17 @@
   <xacro:include filename="$(find ur_description)/urdf/ur.gazebo.xacro" />
   <!-- Inertia parameters -->
-  <xacro:property name="base_mass" value="4.0" />  <!-- This mass might be incorrect -->
-  <xacro:property name="shoulder_mass" value="3.7000" />
-  <xacro:property name="upper_arm_mass" value="8.3930" />
-  <xacro:property name="forearm_mass" value="2.2750" />
-  <xacro:property name="wrist_1_mass" value="1.2190" />
-  <xacro:property name="wrist_2_mass" value="1.2190" />
-  <xacro:property name="wrist_3_mass" value="0.1879" />
-  <xacro:property name="shoulder_cog" value="0.0 0.00193 -0.02561" />
-  <xacro:property name="upper_arm_cog" value="0.0 -0.024201 0.2125" />
-  <xacro:property name="forearm_cog" value="0.0 0.0265 0.11993" />
-  <xacro:property name="wrist_1_cog" value="0.0 0.110949 0.01634" />
-  <xacro:property name="wrist_2_cog" value="0.0 0.0018 0.11099" />
-  <xacro:property name="wrist_3_cog" value="0.0 0.001159 0.0" />
+  <xacro:property name="ur5_base_mass" value="4.0" />  <!-- This mass might be incorrect -->
+  <xacro:property name="ur5_shoulder_mass" value="3.7000" />
+  <xacro:property name="ur5_upper_arm_mass" value="8.3930" />
+  <xacro:property name="ur5_forearm_mass" value="2.2750" />
+  <xacro:property name="ur5_wrist_1_mass" value="1.2190" />
+  <xacro:property name="ur5_wrist_2_mass" value="1.2190" />
+  <xacro:property name="ur5_wrist_3_mass" value="0.1879" />
+  <xacro:property name="ur5_shoulder_cog" value="0.0 0.00193 -0.02561" />
+  <xacro:property name="ur5_upper_arm_cog" value="0.0 -0.024201 0.2125" />
+  <xacro:property name="ur5_forearm_cog" value="0.0 0.0265 0.11993" />
+  <xacro:property name="ur5_wrist_1_cog" value="0.0 0.110949 0.01634" />
+  <xacro:property name="ur5_wrist_2_cog" value="0.0 0.0018 0.11099" />
+  <xacro:property name="ur5_wrist_3_cog" value="0.0 0.001159 0.0" />
   <!-- Kinematic model -->
   <!-- Properties from urcontrol.conf -->
@@ -36,26 +36,26 @@
   <xacro:property name="ur5_d6" value="0.0823" />
   <!-- Arbitrary offsets for shoulder/elbow joints -->
-  <xacro:property name="shoulder_offset" value="0.13585" />  <!-- measured from model -->
-  <xacro:property name="elbow_offset" value="-0.1197" /> <!-- measured from model -->
+  <xacro:property name="ur5_shoulder_offset" value="0.13585" />  <!-- measured from model -->
+  <xacro:property name="ur5_elbow_offset" value="-0.1197" /> <!-- measured from model -->
   <!-- link lengths used in model -->
-  <xacro:property name="shoulder_height" value="${ur5_d1}" />
-  <xacro:property name="upper_arm_length" value="${-ur5_a2}" />
-  <xacro:property name="forearm_length" value="${-ur5_a3}" />
-  <xacro:property name="wrist_1_length" value="${ur5_d4 - elbow_offset - shoulder_offset}" />
-  <xacro:property name="wrist_2_length" value="${ur5_d5}" />
-  <xacro:property name="wrist_3_length" value="${ur5_d6}" />
-  <!--property name="shoulder_height" value="0.089159" /-->
-  <!--property name="shoulder_offset" value="0.13585" /-->  <!-- shoulder_offset - elbow_offset + wrist_1_length = 0.10915 -->
-  <!--property name="upper_arm_length" value="0.42500" /-->
-  <!--property name="elbow_offset" value="0.1197" /-->       <!-- CAD measured -->
-  <!--property name="forearm_length" value="0.39225" /-->
-  <!--property name="wrist_1_length" value="0.093" /-->     <!-- CAD measured -->
-  <!--property name="wrist_2_length" value="0.09465" /-->   <!-- In CAD this distance is 0.930, but in the spec it is 0.09465 -->
-  <!--property name="wrist_3_length" value="0.0823" /-->
-  <xacro:property name="shoulder_radius" value="0.060" />   <!-- manually measured -->
-  <xacro:property name="upper_arm_radius" value="0.054" />  <!-- manually measured -->
-  <xacro:property name="elbow_radius" value="0.060" />      <!-- manually measured -->
-  <xacro:property name="forearm_radius" value="0.040" />    <!-- manually measured -->
-  <xacro:property name="wrist_radius" value="0.045" />      <!-- manually measured -->
+  <xacro:property name="ur5_shoulder_height" value="${ur5_d1}" />
+  <xacro:property name="ur5_upper_arm_length" value="${-ur5_a2}" />
+  <xacro:property name="ur5_forearm_length" value="${-ur5_a3}" />
+  <xacro:property name="ur5_wrist_1_length" value="${ur5_d4 - ur5_elbow_offset - ur5_shoulder_offset}" />
+  <xacro:property name="ur5_wrist_2_length" value="${ur5_d5}" />
+  <xacro:property name="ur5_wrist_3_length" value="${ur5_d6}" />
+  <!--property name="ur5_shoulder_height" value="0.089159" /-->
+  <!--property name="ur5_shoulder_offset" value="0.13585" /-->  <!-- ur5_shoulder_offset - ur5_elbow_offset + ur5_wrist_1_length = 0.10915 -->
+  <!--property name="ur5_upper_arm_length" value="0.42500" /-->
+  <!--property name="ur5_elbow_offset" value="0.1197" /-->       <!-- CAD measured -->
+  <!--property name="ur5_forearm_length" value="0.39225" /-->
+  <!--property name="ur5_wrist_1_length" value="0.093" /-->     <!-- CAD measured -->
+  <!--property name="ur5_wrist_2_length" value="0.09465" /-->   <!-- In CAD this distance is 0.930, but in the spec it is 0.09465 -->
+  <!--property name="ur5_wrist_3_length" value="0.0823" /-->
+  <xacro:property name="ur5_shoulder_radius" value="0.060" />   <!-- manually measured -->
+  <xacro:property name="ur5_upper_arm_radius" value="0.054" />  <!-- manually measured -->
+  <xacro:property name="ur5_elbow_radius" value="0.060" />      <!-- manually measured -->
+  <xacro:property name="ur5_forearm_radius" value="0.040" />    <!-- manually measured -->
+  <xacro:property name="ur5_wrist_radius" value="0.045" />      <!-- manually measured -->
   <xacro:macro name="cylinder_inertial" params="radius length mass *origin">
     <inertial>
@@ -88,5 +88,5 @@
         </geometry>
       </collision>
-      <xacro:cylinder_inertial radius="0.06" length="0.05" mass="${base_mass}">
+      <xacro:cylinder_inertial radius="0.06" length="0.05" mass="${ur5_base_mass}">
         <origin xyz="0.0 0.0 0.0" rpy="0 0 0" />
       </xacro:cylinder_inertial>
@@ -95,5 +95,5 @@
       <parent link="${prefix}base_link" />
       <child link = "${prefix}shoulder_link" />
-      <origin xyz="0.0 0.0 ${shoulder_height}" rpy="0.0 0.0 0.0" />
+      <origin xyz="0.0 0.0 ${ur5_shoulder_height}" rpy="0.0 0.0 0.0" />
       <axis xyz="0 0 1" />
       <xacro:unless value="${joint_limited}">
@@ -119,5 +119,5 @@
         </geometry>
       </collision>
-      <xacro:cylinder_inertial radius="0.06" length="0.15" mass="${shoulder_mass}">
+      <xacro:cylinder_inertial radius="0.06" length="0.15" mass="${ur5_shoulder_mass}">
         <origin xyz="0.0 0.0 0.0" rpy="0 0 0" />
       </xacro:cylinder_inertial>
@@ -126,5 +126,5 @@
       <parent link="${prefix}shoulder_link" />
       <child link = "${prefix}upper_arm_link" />
-      <origin xyz="0.0 ${shoulder_offset} 0.0" rpy="0.0 ${pi / 2.0} 0.0" />
+      <origin xyz="0.0 ${ur5_shoulder_offset} 0.0" rpy="0.0 ${pi / 2.0} 0.0" />
       <axis xyz="0 1 0" />
       <xacro:unless value="${joint_limited}">
@@ -150,5 +150,5 @@
         </geometry>
       </collision>
-      <xacro:cylinder_inertial radius="0.06" length="0.56" mass="${upper_arm_mass}">
+      <xacro:cylinder_inertial radius="0.06" length="0.56" mass="${ur5_upper_arm_mass}">
         <origin xyz="0.0 0.0 0.28" rpy="0 0 0" />
       </xacro:cylinder_inertial>
@@ -157,5 +157,5 @@
       <parent link="${prefix}upper_arm_link" />
       <child link = "${prefix}forearm_link" />
-      <origin xyz="0.0 ${elbow_offset} ${upper_arm_length}" rpy="0.0 0.0 0.0" />
+      <origin xyz="0.0 ${ur5_elbow_offset} ${ur5_upper_arm_length}" rpy="0.0 0.0 0.0" />
       <axis xyz="0 1 0" />
       <xacro:unless value="${joint_limited}">
@@ -181,5 +181,5 @@
         </geometry>
       </collision>
-      <xacro:cylinder_inertial radius="0.06" length="0.5" mass="${forearm_mass}">
+      <xacro:cylinder_inertial radius="0.06" length="0.5" mass="${ur5_forearm_mass}">
         <origin xyz="0.0 0.0 0.25" rpy="0 0 0" />
       </xacro:cylinder_inertial>
@@ -188,5 +188,5 @@
       <parent link="${prefix}forearm_link" />
       <child link = "${prefix}wrist_1_link" />
-      <origin xyz="0.0 0.0 ${forearm_length}" rpy="0.0 ${pi / 2.0} 0.0" />
+      <origin xyz="0.0 0.0 ${ur5_forearm_length}" rpy="0.0 ${pi / 2.0} 0.0" />
       <axis xyz="0 1 0" />
       <xacro:unless value="${joint_limited}">
@@ -212,5 +212,5 @@
         </geometry>
       </collision>
-      <xacro:cylinder_inertial radius="0.6" length="0.12" mass="${wrist_1_mass}">
+      <xacro:cylinder_inertial radius="0.6" length="0.12" mass="${ur5_wrist_1_mass}">
         <origin xyz="0.0 0.0 0.0" rpy="0 0 0" />
       </xacro:cylinder_inertial>
@@ -219,5 +219,5 @@
       <parent link="${prefix}wrist_1_link" />
       <child link = "${prefix}wrist_2_link" />
-      <origin xyz="0.0 ${wrist_1_length} 0.0" rpy="0.0 0.0 0.0" />
+      <origin xyz="0.0 ${ur5_wrist_1_length} 0.0" rpy="0.0 0.0 0.0" />
       <axis xyz="0 0 1" />
       <xacro:unless value="${joint_limited}">
@@ -243,5 +243,5 @@
         </geometry>
       </collision>
-      <xacro:cylinder_inertial radius="0.6" length="0.12" mass="${wrist_2_mass}">
+      <xacro:cylinder_inertial radius="0.6" length="0.12" mass="${ur5_wrist_2_mass}">
         <origin xyz="0.0 0.0 0.0" rpy="0 0 0" />
       </xacro:cylinder_inertial>
@@ -250,5 +250,5 @@
       <parent link="${prefix}wrist_2_link" />
       <child link = "${prefix}wrist_3_link" />
-      <origin xyz="0.0 0.0 ${wrist_2_length}" rpy="0.0 0.0 0.0" />
+      <origin xyz="0.0 0.0 ${ur5_wrist_2_length}" rpy="0.0 0.0 0.0" />
       <axis xyz="0 1 0" />
       <xacro:unless value="${joint_limited}">
@@ -274,5 +274,5 @@
         </geometry>
       </collision>
-      <xacro:cylinder_inertial radius="0.6" length="0.12" mass="${wrist_3_mass}">
+      <xacro:cylinder_inertial radius="0.6" length="0.12" mass="${ur5_wrist_3_mass}">
         <origin xyz="0.0 0.0 0.0" rpy="0 0 0" />
       </xacro:cylinder_inertial>
@@ -281,5 +281,5 @@
       <parent link="${prefix}wrist_3_link" />
       <child link = "${prefix}ee_link" />
-      <origin xyz="0.0 ${wrist_3_length} 0.0" rpy="0.0 0.0 ${pi/2.0}" />
+      <origin xyz="0.0 ${ur5_wrist_3_length} 0.0" rpy="0.0 0.0 ${pi/2.0}" />
     </joint>
     <link name="${prefix}ee_link">
@@ -307,5 +307,5 @@
     <link name="${prefix}tool0"/>
     <joint name="${prefix}wrist_3_link-tool0_fixed_joint" type="fixed">
-      <origin xyz="0 ${wrist_3_length} 0" rpy="${pi/-2.0} 0 0"/>
+      <origin xyz="0 ${ur5_wrist_3_length} 0" rpy="${pi/-2.0} 0 0"/>
       <parent link="${prefix}wrist_3_link"/>
       <child link="${prefix}tool0"/>
