Commit message: Move robot-specific parameters inside macro
This is the cleaner solution for what the previous commit was meant to solve

File: ur_description/urdf/ur10.urdf.xacro (robot description, xacro)
@@ -7,40 +7,4 @@
   <xacro:include filename="$(find ur_description)/urdf/ur.transmission.xacro" />
   <xacro:include filename="$(find ur_description)/urdf/ur.gazebo.xacro" />
-  <!-- Inertia parameters -->
-  <xacro:property name="ur10_base_mass" value="4.0" />  <!-- This mass might be incorrect -->
-  <xacro:property name="ur10_shoulder_mass" value="7.778" />
-  <xacro:property name="ur10_upper_arm_mass" value="12.93" />
-  <xacro:property name="ur10_forearm_mass" value="3.87" />
-  <xacro:property name="ur10_wrist_1_mass" value="1.96" />
-  <xacro:property name="ur10_wrist_2_mass" value="1.96" />
-  <xacro:property name="ur10_wrist_3_mass" value="0.202" />
-  <!-- These parameters are borrowed from the urcontrol.conf file
-       but are not verified for the correct permutation.
-       The permutation was guessed by looking at the UR5 parameters.
-       Serious use of these parameters needs further inspection. -->
-  <xacro:property name="ur10_shoulder_cog" value="0.00008 0.00244 -0.037" />
-  <xacro:property name="ur10_upper_arm_cog" value="0.00001 0.15061 0.38757" />
-  <xacro:property name="ur10_forearm_cog" value="-0.00012 0.06112 0.1984" />
-  <xacro:property name="ur10_wrist_1_cog" value="-0.00021 -0.00112 0.02269" />
-  <xacro:property name="ur10_wrist_2_cog" value="-0.00021 0.00112 0.002269" />
-  <xacro:property name="ur10_wrist_3_cog" value="0 -0.001156 -0.00149" />
-  <!-- Kinematic model -->
-  <!-- Properties from urcontrol.conf -->
-  <xacro:property name="ur10_d1" value="0.1273" />
-  <xacro:property name="ur10_a2" value="-0.612" />
-  <xacro:property name="ur10_a3" value="-0.5723" />
-  <xacro:property name="ur10_d4" value="0.163941" />
-  <xacro:property name="ur10_d5" value="0.1157" />
-  <xacro:property name="ur10_d6" value="0.0922" />
-  <!-- Arbitrary offsets for shoulder/elbow joints -->
-  <xacro:property name="ur10_shoulder_offset" value="0.220941" />  <!-- measured from model -->
-  <xacro:property name="ur10_elbow_offset" value="-0.1719" /> <!-- measured from model -->
-  <!-- link lengths used in model -->
-  <xacro:property name="ur10_shoulder_height" value="${ur10_d1}" />
-  <xacro:property name="ur10_upper_arm_length" value="${-ur10_a2}" />
-  <xacro:property name="ur10_forearm_length" value="${-ur10_a3}" />
-  <xacro:property name="ur10_wrist_1_length" value="${ur10_d4 - ur10_elbow_offset - ur10_shoulder_offset}" />
-  <xacro:property name="ur10_wrist_2_length" value="${ur10_d5}" />
-  <xacro:property name="ur10_wrist_3_length" value="${ur10_d6}" />
   <xacro:macro name="cylinder_inertial" params="radius length mass *origin">
     <inertial>
@@ -59,4 +23,40 @@
 		 wrist_2_lower_limit:=${-pi}    wrist_2_upper_limit:=${pi}
 		 wrist_3_lower_limit:=${-pi}    wrist_3_upper_limit:=${pi}">
+    <!-- Inertia parameters -->
+    <xacro:property name="base_mass" value="4.0" />  <!-- This mass might be incorrect -->
+    <xacro:property name="shoulder_mass" value="7.778" />
+    <xacro:property name="upper_arm_mass" value="12.93" />
+    <xacro:property name="forearm_mass" value="3.87" />
+    <xacro:property name="wrist_1_mass" value="1.96" />
+    <xacro:property name="wrist_2_mass" value="1.96" />
+    <xacro:property name="wrist_3_mass" value="0.202" />
+    <!-- These parameters are borrowed from the urcontrol.conf file
+        but are not verified for the correct permutation.
+        The permutation was guessed by looking at the UR5 parameters.
+        Serious use of these parameters needs further inspection. -->
+    <xacro:property name="shoulder_cog" value="0.00008 0.00244 -0.037" />
+    <xacro:property name="upper_arm_cog" value="0.00001 0.15061 0.38757" />
+    <xacro:property name="forearm_cog" value="-0.00012 0.06112 0.1984" />
+    <xacro:property name="wrist_1_cog" value="-0.00021 -0.00112 0.02269" />
+    <xacro:property name="wrist_2_cog" value="-0.00021 0.00112 0.002269" />
+    <xacro:property name="wrist_3_cog" value="0 -0.001156 -0.00149" />
+    <!-- Kinematic model -->
+    <!-- Properties from urcontrol.conf -->
+    <xacro:property name="d1" value="0.1273" />
+    <xacro:property name="a2" value="-0.612" />
+    <xacro:property name="a3" value="-0.5723" />
+    <xacro:property name="d4" value="0.163941" />
+    <xacro:property name="d5" value="0.1157" />
+    <xacro:property name="d6" value="0.0922" />
+    <!-- Arbitrary offsets for shoulder/elbow joints -->
+    <xacro:property name="shoulder_offset" value="0.220941" />  <!-- measured from model -->
+    <xacro:property name="elbow_offset" value="-0.1719" /> <!-- measured from model -->
+    <!-- link lengths used in model -->
+    <xacro:property name="shoulder_height" value="${d1}" />
+    <xacro:property name="upper_arm_length" value="${-a2}" />
+    <xacro:property name="forearm_length" value="${-a3}" />
+    <xacro:property name="wrist_1_length" value="${d4 - elbow_offset - shoulder_offset}" />
+    <xacro:property name="wrist_2_length" value="${d5}" />
+    <xacro:property name="wrist_3_length" value="${d6}" />
     <link name="${prefix}base_link" >
       <visual>
@@ -73,5 +73,5 @@
         </geometry>
       </collision>
-      <xacro:cylinder_inertial radius="0.075" length="0.038" mass="${ur10_base_mass}">
+      <xacro:cylinder_inertial radius="0.075" length="0.038" mass="${base_mass}">
         <origin xyz="0.0 0.0 0.0" rpy="0 0 0" />
       </xacro:cylinder_inertial>
@@ -80,5 +80,5 @@
       <parent link="${prefix}base_link" />
       <child link = "${prefix}shoulder_link" />
-      <origin xyz="0.0 0.0 ${ur10_shoulder_height}" rpy="0.0 0.0 0.0" />
+      <origin xyz="0.0 0.0 ${shoulder_height}" rpy="0.0 0.0 0.0" />
       <axis xyz="0 0 1" />
       <xacro:unless value="${joint_limited}">
@@ -104,5 +104,5 @@
         </geometry>
       </collision>
-      <xacro:cylinder_inertial radius="0.075" length="0.178" mass="${ur10_shoulder_mass}">
+      <xacro:cylinder_inertial radius="0.075" length="0.178" mass="${shoulder_mass}">
         <origin xyz="0.0 0.0 0.0" rpy="0 0 0" />
       </xacro:cylinder_inertial>
@@ -111,5 +111,5 @@
       <parent link="${prefix}shoulder_link" />
       <child link = "${prefix}upper_arm_link" />
-      <origin xyz="0.0 ${ur10_shoulder_offset} 0.0" rpy="0.0 ${pi / 2.0} 0.0" />
+      <origin xyz="0.0 ${shoulder_offset} 0.0" rpy="0.0 ${pi / 2.0} 0.0" />
       <axis xyz="0 1 0" />
       <xacro:unless value="${joint_limited}">
@@ -135,6 +135,6 @@
         </geometry>
       </collision>
-      <xacro:cylinder_inertial radius="0.075" length="${-ur10_a2}" mass="${ur10_upper_arm_mass}">
-        <origin xyz="0.0 0.0 ${-ur10_a2/2.0}" rpy="0 0 0" />
+      <xacro:cylinder_inertial radius="0.075" length="${-a2}" mass="${upper_arm_mass}">
+        <origin xyz="0.0 0.0 ${-a2/2.0}" rpy="0 0 0" />
       </xacro:cylinder_inertial>
     </link>
@@ -142,5 +142,5 @@
       <parent link="${prefix}upper_arm_link" />
       <child link = "${prefix}forearm_link" />
-      <origin xyz="0.0 ${ur10_elbow_offset} ${ur10_upper_arm_length}" rpy="0.0 0.0 0.0" />
+      <origin xyz="0.0 ${elbow_offset} ${upper_arm_length}" rpy="0.0 0.0 0.0" />
       <axis xyz="0 1 0" />
       <xacro:unless value="${joint_limited}">
@@ -166,6 +166,6 @@
         </geometry>
       </collision>
-      <xacro:cylinder_inertial radius="0.075" length="${-ur10_a3}" mass="${ur10_forearm_mass}">
-        <origin xyz="0.0 0.0 ${-ur10_a3/2.0}" rpy="0 0 0" />
+      <xacro:cylinder_inertial radius="0.075" length="${-a3}" mass="${forearm_mass}">
+        <origin xyz="0.0 0.0 ${-a3/2.0}" rpy="0 0 0" />
       </xacro:cylinder_inertial>
     </link>
@@ -173,5 +173,5 @@
       <parent link="${prefix}forearm_link" />
       <child link = "${prefix}wrist_1_link" />
-      <origin xyz="0.0 0.0 ${ur10_forearm_length}" rpy="0.0 ${pi / 2.0} 0.0" />
+      <origin xyz="0.0 0.0 ${forearm_length}" rpy="0.0 ${pi / 2.0} 0.0" />
       <axis xyz="0 1 0" />
       <xacro:unless value="${joint_limited}">
@@ -197,5 +197,5 @@
         </geometry>
       </collision>
-      <xacro:cylinder_inertial radius="0.075" length="0.12" mass="${ur10_wrist_1_mass}">
+      <xacro:cylinder_inertial radius="0.075" length="0.12" mass="${wrist_1_mass}">
         <origin xyz="0.0 0.0 0.0" rpy="0 0 0" />
       </xacro:cylinder_inertial>
@@ -204,5 +204,5 @@
       <parent link="${prefix}wrist_1_link" />
       <child link = "${prefix}wrist_2_link" />
-      <origin xyz="0.0 ${ur10_wrist_1_length} 0.0" rpy="0.0 0.0 0.0" />
+      <origin xyz="0.0 ${wrist_1_length} 0.0" rpy="0.0 0.0 0.0" />
       <axis xyz="0 0 1" />
       <xacro:unless value="${joint_limited}">
@@ -228,5 +228,5 @@
         </geometry>
       </collision>
-      <xacro:cylinder_inertial radius="0.075" length="0.12" mass="${ur10_wrist_2_mass}">
+      <xacro:cylinder_inertial radius="0.075" length="0.12" mass="${wrist_2_mass}">
         <origin xyz="0.0 0.0 0.0" rpy="0 0 0" />
       </xacro:cylinder_inertial>
@@ -235,5 +235,5 @@
       <parent link="${prefix}wrist_2_link" />
       <child link = "${prefix}wrist_3_link" />
-      <origin xyz="0.0 0.0 ${ur10_wrist_2_length}" rpy="0.0 0.0 0.0" />
+      <origin xyz="0.0 0.0 ${wrist_2_length}" rpy="0.0 0.0 0.0" />
       <axis xyz="0 1 0" />
       <xacro:unless value="${joint_limited}">
@@ -259,5 +259,5 @@
         </geometry>
       </collision>
-      <xacro:cylinder_inertial radius="0.075" length="0.12" mass="${ur10_wrist_3_mass}">
+      <xacro:cylinder_inertial radius="0.075" length="0.12" mass="${wrist_3_mass}">
         <origin xyz="0.0 0.0 0.0" rpy="0 0 0" />
       </xacro:cylinder_inertial>
@@ -266,5 +266,5 @@
       <parent link="${prefix}wrist_3_link" />
       <child link = "${prefix}ee_link" />
-      <origin xyz="0.0 ${ur10_wrist_3_length} 0.0" rpy="0.0 0.0 ${pi/2.0}" />
+      <origin xyz="0.0 ${wrist_3_length} 0.0" rpy="0.0 0.0 ${pi/2.0}" />
     </joint>
     <link name="${prefix}ee_link">
@@ -292,5 +292,5 @@
     <link name="${prefix}tool0"/>
     <joint name="${prefix}wrist_3_link-tool0_fixed_joint" type="fixed">
-      <origin xyz="0 ${ur10_wrist_3_length} 0" rpy="${pi/-2.0} 0 0"/>
+      <origin xyz="0 ${wrist_3_length} 0" rpy="${pi/-2.0} 0 0"/>
       <parent link="${prefix}wrist_3_link"/>
       <child link="${prefix}tool0"/>

File: ur_description/urdf/ur3.urdf.xacro (robot description, xacro)
@@ -6,41 +6,5 @@
   <xacro:include filename="$(find ur_description)/urdf/ur.transmission.xacro" />
   <xacro:include filename="$(find ur_description)/urdf/ur.gazebo.xacro" />
-  <!-- Inertia parameters -->
-  <xacro:property name="ur3_base_mass" value="2.0" />  <!-- This mass might be incorrect -->
-  <xacro:property name="ur3_shoulder_mass" value="2.0" />
-  <xacro:property name="ur3_upper_arm_mass" value="3.42" />
-  <xacro:property name="ur3_forearm_mass" value="1.26" />
-  <xacro:property name="ur3_wrist_1_mass" value="0.8" />
-  <xacro:property name="ur3_wrist_2_mass" value="0.8" />
-  <xacro:property name="ur3_wrist_3_mass" value="0.35" />
-  <!-- These parameters are borrowed from the urcontrol.conf file
-       but are not verified for the correct permutation.
-       The permutation was guessed by looking at the UR5 parameters.
-       Serious use of these parameters needs further inspection. -->
-  <xacro:property name="ur3_shoulder_cog" value="0.0 -0.02 0.0" />
-  <xacro:property name="ur3_upper_arm_cog" value="0.13 0.0 0.1157" />
-  <xacro:property name="ur3_forearm_cog" value="0.05 0.0 0.0238" />
-  <xacro:property name="ur3_wrist_1_cog" value="0.0 0.0 0.01" />
-  <xacro:property name="ur3_wrist_2_cog" value="0.0 0.0 0.01" />
-  <xacro:property name="ur3_wrist_3_cog" value="0.0 0.0 -0.02" />
-  <!-- Kinematic model -->
-  <!-- Properties from urcontrol.conf -->
-  <xacro:property name="ur3_d1" value="0.1519" />
-  <xacro:property name="ur3_a2" value="-0.24365" />
-  <xacro:property name="ur3_a3" value="-0.21325" />
-  <xacro:property name="ur3_d4" value="0.11235" />
-  <xacro:property name="ur3_d5" value="0.08535" />
-  <xacro:property name="ur3_d6" value="0.0819" />
-  <!-- Arbitrary offsets for shoulder/elbow joints -->
-  <xacro:property name="ur3_shoulder_offset" value="0.1198" />  <!-- measured from model -->
-  <xacro:property name="ur3_elbow_offset" value="-0.0925" /> <!-- measured from model -->
-  <!-- link lengths used in model -->
-  <xacro:property name="ur3_shoulder_height" value="${ur3_d1}" />
-  <xacro:property name="ur3_upper_arm_length" value="${-ur3_a2}" />
-  <xacro:property name="ur3_forearm_length" value="${-ur3_a3}" />
-  <xacro:property name="ur3_wrist_1_length" value="${ur3_d4 - ur3_elbow_offset - ur3_shoulder_offset}" />
-  <xacro:property name="ur3_wrist_2_length" value="${ur3_d5}" />
-  <xacro:property name="ur3_wrist_3_length" value="${ur3_d6}" />
-  <xacro:macro name="cylinder_inertial" params="radius length mass *origin">
+   <xacro:macro name="cylinder_inertial" params="radius length mass *origin">
     <inertial>
       <mass value="${mass}" />
@@ -58,4 +22,40 @@
      wrist_2_lower_limit:=${-pi}    wrist_2_upper_limit:=${pi}
      wrist_3_lower_limit:=${-pi}    wrist_3_upper_limit:=${pi}">
+    <!-- Inertia parameters -->
+    <xacro:property name="base_mass" value="2.0" />  <!-- This mass might be incorrect -->
+    <xacro:property name="shoulder_mass" value="2.0" />
+    <xacro:property name="upper_arm_mass" value="3.42" />
+    <xacro:property name="forearm_mass" value="1.26" />
+    <xacro:property name="wrist_1_mass" value="0.8" />
+    <xacro:property name="wrist_2_mass" value="0.8" />
+    <xacro:property name="wrist_3_mass" value="0.35" />
+    <!-- These parameters are borrowed from the urcontrol.conf file
+        but are not verified for the correct permutation.
+        The permutation was guessed by looking at the UR5 parameters.
+        Serious use of these parameters needs further inspection. -->
+    <xacro:property name="shoulder_cog" value="0.0 -0.02 0.0" />
+    <xacro:property name="upper_arm_cog" value="0.13 0.0 0.1157" />
+    <xacro:property name="forearm_cog" value="0.05 0.0 0.0238" />
+    <xacro:property name="wrist_1_cog" value="0.0 0.0 0.01" />
+    <xacro:property name="wrist_2_cog" value="0.0 0.0 0.01" />
+    <xacro:property name="wrist_3_cog" value="0.0 0.0 -0.02" />
+    <!-- Kinematic model -->
+    <!-- Properties from urcontrol.conf -->
+    <xacro:property name="d1" value="0.1519" />
+    <xacro:property name="a2" value="-0.24365" />
+    <xacro:property name="a3" value="-0.21325" />
+    <xacro:property name="d4" value="0.11235" />
+    <xacro:property name="d5" value="0.08535" />
+    <xacro:property name="d6" value="0.0819" />
+    <!-- Arbitrary offsets for shoulder/elbow joints -->
+    <xacro:property name="shoulder_offset" value="0.1198" />  <!-- measured from model -->
+    <xacro:property name="elbow_offset" value="-0.0925" /> <!-- measured from model -->
+    <!-- link lengths used in model -->
+    <xacro:property name="shoulder_height" value="${d1}" />
+    <xacro:property name="upper_arm_length" value="${-a2}" />
+    <xacro:property name="forearm_length" value="${-a3}" />
+    <xacro:property name="wrist_1_length" value="${d4 - elbow_offset - shoulder_offset}" />
+    <xacro:property name="wrist_2_length" value="${d5}" />
+    <xacro:property name="wrist_3_length" value="${d6}" />
     <link name="${prefix}base_link" >
       <visual>
@@ -72,5 +72,5 @@
         </geometry>
       </collision>
-      <xacro:cylinder_inertial radius="0.075" length="0.038" mass="${ur3_base_mass}">
+      <xacro:cylinder_inertial radius="0.075" length="0.038" mass="${base_mass}">
         <origin xyz="0.0 0.0 0.0" rpy="0 0 0" />
       </xacro:cylinder_inertial>
@@ -79,5 +79,5 @@
       <parent link="${prefix}base_link" />
       <child link = "${prefix}shoulder_link" />
-      <origin xyz="0.0 0.0 ${ur3_shoulder_height}" rpy="0.0 0.0 0.0" />
+      <origin xyz="0.0 0.0 ${shoulder_height}" rpy="0.0 0.0 0.0" />
       <axis xyz="0 0 1" />
       <xacro:unless value="${joint_limited}">
@@ -103,5 +103,5 @@
         </geometry>
       </collision>
-      <xacro:cylinder_inertial radius="0.075" length="0.178" mass="${ur3_shoulder_mass}">
+      <xacro:cylinder_inertial radius="0.075" length="0.178" mass="${shoulder_mass}">
         <origin xyz="0.0 0.0 0.0" rpy="0 0 0" />
       </xacro:cylinder_inertial>
@@ -110,5 +110,5 @@
       <parent link="${prefix}shoulder_link" />
       <child link = "${prefix}upper_arm_link" />
-      <origin xyz="0.0 ${ur3_shoulder_offset} 0.0" rpy="0.0 ${pi / 2.0} 0.0" />
+      <origin xyz="0.0 ${shoulder_offset} 0.0" rpy="0.0 ${pi / 2.0} 0.0" />
       <axis xyz="0 1 0" />
       <xacro:unless value="${joint_limited}">
@@ -134,6 +134,6 @@
         </geometry>
       </collision>
-      <xacro:cylinder_inertial radius="0.075" length="${-ur3_a2}" mass="${ur3_upper_arm_mass}">
-        <origin xyz="0.0 0.0 ${-ur3_a2/2.0}" rpy="0 0 0" />
+      <xacro:cylinder_inertial radius="0.075" length="${-a2}" mass="${upper_arm_mass}">
+        <origin xyz="0.0 0.0 ${-a2/2.0}" rpy="0 0 0" />
       </xacro:cylinder_inertial>
     </link>
@@ -141,5 +141,5 @@
       <parent link="${prefix}upper_arm_link" />
       <child link = "${prefix}forearm_link" />
-      <origin xyz="0.0 ${ur3_elbow_offset} ${ur3_upper_arm_length}" rpy="0.0 0.0 0.0" />
+      <origin xyz="0.0 ${elbow_offset} ${upper_arm_length}" rpy="0.0 0.0 0.0" />
       <axis xyz="0 1 0" />
       <xacro:unless value="${joint_limited}">
@@ -165,6 +165,6 @@
         </geometry>
       </collision>
-      <xacro:cylinder_inertial radius="0.075" length="${-ur3_a3}" mass="${ur3_forearm_mass}">
-        <origin xyz="0.0 0.0 ${-ur3_a3/2.0}" rpy="0 0 0" />
+      <xacro:cylinder_inertial radius="0.075" length="${-a3}" mass="${forearm_mass}">
+        <origin xyz="0.0 0.0 ${-a3/2.0}" rpy="0 0 0" />
       </xacro:cylinder_inertial>
     </link>
@@ -172,5 +172,5 @@
       <parent link="${prefix}forearm_link" />
       <child link = "${prefix}wrist_1_link" />
-      <origin xyz="0.0 0.0 ${ur3_forearm_length}" rpy="0.0 ${pi / 2.0} 0.0" />
+      <origin xyz="0.0 0.0 ${forearm_length}" rpy="0.0 ${pi / 2.0} 0.0" />
       <axis xyz="0 1 0" />
       <xacro:unless value="${joint_limited}">
@@ -196,5 +196,5 @@
         </geometry>
       </collision>
-      <xacro:cylinder_inertial radius="0.075" length="0.12" mass="${ur3_wrist_1_mass}">
+      <xacro:cylinder_inertial radius="0.075" length="0.12" mass="${wrist_1_mass}">
         <origin xyz="0.0 0.0 0.0" rpy="0 0 0" />
       </xacro:cylinder_inertial>
@@ -203,5 +203,5 @@
       <parent link="${prefix}wrist_1_link" />
       <child link = "${prefix}wrist_2_link" />
-      <origin xyz="0.0 ${ur3_wrist_1_length} 0.0" rpy="0.0 0.0 0.0" />
+      <origin xyz="0.0 ${wrist_1_length} 0.0" rpy="0.0 0.0 0.0" />
       <axis xyz="0 0 1" />
       <xacro:unless value="${joint_limited}">
@@ -227,5 +227,5 @@
         </geometry>
       </collision>
-      <xacro:cylinder_inertial radius="0.075" length="0.12" mass="${ur3_wrist_2_mass}">
+      <xacro:cylinder_inertial radius="0.075" length="0.12" mass="${wrist_2_mass}">
         <origin xyz="0.0 0.0 0.0" rpy="0 0 0" />
       </xacro:cylinder_inertial>
@@ -234,5 +234,5 @@
       <parent link="${prefix}wrist_2_link" />
       <child link = "${prefix}wrist_3_link" />
-      <origin xyz="0.0 0.0 ${ur3_wrist_2_length}" rpy="0.0 0.0 0.0" />
+      <origin xyz="0.0 0.0 ${wrist_2_length}" rpy="0.0 0.0 0.0" />
       <axis xyz="0 1 0" />
       <xacro:unless value="${joint_limited}">
@@ -258,5 +258,5 @@
         </geometry>
       </collision>
-      <xacro:cylinder_inertial radius="0.075" length="0.12" mass="${ur3_wrist_3_mass}">
+      <xacro:cylinder_inertial radius="0.075" length="0.12" mass="${wrist_3_mass}">
         <origin xyz="0.0 0.0 0.0" rpy="0 0 0" />
       </xacro:cylinder_inertial>
@@ -265,5 +265,5 @@
       <parent link="${prefix}wrist_3_link" />
       <child link = "${prefix}ee_link" />
-      <origin xyz="0.0 ${ur3_wrist_3_length} 0.0" rpy="0.0 0.0 ${pi/2.0}" />
+      <origin xyz="0.0 ${wrist_3_length} 0.0" rpy="0.0 0.0 ${pi/2.0}" />
     </joint>
     <link name="${prefix}ee_link">
@@ -291,5 +291,5 @@
     <link name="${prefix}tool0"/>
     <joint name="${prefix}wrist_3_link-tool0_fixed_joint" type="fixed">
-      <origin xyz="0 ${ur3_wrist_3_length} 0" rpy="${pi/-2.0} 0 0"/>
+      <origin xyz="0 ${wrist_3_length} 0" rpy="${pi/-2.0} 0 0"/>
       <parent link="${prefix}wrist_3_link"/>
       <child link="${prefix}tool0"/>
