Commit message: Updated cog for ur16 how I understand the documentation
used documentation:
https://www.universal-robots.com/how-tos-and-faqs/faq/ur-faq/parameters-for-calculations-of-kinematics-and-dynamics-45257/

Note: This changes inertia for all robots as the main xacro file is changed.

File: ur_description/urdf/ur_macro.xacro (robot description, xacro)
@@ -102,5 +102,5 @@
       </collision>
       <xacro:cylinder_inertial radius="${shoulder_inertia_radius}" length="${shoulder_inertia_length}" mass="${shoulder_mass}">
-        <origin xyz="0 0 0" rpy="0 0 0" />
+        <origin xyz="${shoulder_cog}" rpy="0 0 0" />
       </xacro:cylinder_inertial>
     </link>
@@ -122,5 +122,5 @@
       </collision>
       <xacro:cylinder_inertial radius="${upperarm_inertia_radius}" length="${upperarm_inertia_length}" mass="${upper_arm_mass}">
-        <origin xyz="${-0.5 * upperarm_inertia_length} 0.0 ${upper_arm_inertia_offset}" rpy="0 ${pi/2} 0" />
+        <origin xyz="${upper_arm_cog}" rpy="0 ${pi/2} 0" />
       </xacro:cylinder_inertial>
     </link>
@@ -142,5 +142,5 @@
       </collision>
       <xacro:cylinder_inertial radius="${forearm_inertia_radius}" length="${forearm_inertia_length}"  mass="${forearm_mass}">
-        <origin xyz="${-0.5 * forearm_inertia_length} 0.0 ${elbow_offset}" rpy="0 ${pi/2} 0" />
+        <origin xyz="${forearm_cog}" rpy="0 ${pi/2} 0" />
       </xacro:cylinder_inertial>
     </link>
@@ -163,5 +163,5 @@
       </collision>
       <xacro:cylinder_inertial radius="${wrist_1_inertia_radius}" length="${wrist_1_inertia_length}"  mass="${wrist_1_mass}">
-        <origin xyz="0 0 0" rpy="0 0 0" />
+        <origin xyz="${wrist_1_cog}" rpy="0 0 0" />
       </xacro:cylinder_inertial>
     </link>
@@ -183,5 +183,5 @@
       </collision>
       <xacro:cylinder_inertial radius="${wrist_2_inertia_radius}" length="${wrist_2_inertia_length}"  mass="${wrist_2_mass}">
-        <origin xyz="0 0 0" rpy="0 0 0" />
+        <origin xyz="${wrist_2_cog}" rpy="0 0 0" />
       </xacro:cylinder_inertial>
     </link>
@@ -203,5 +203,5 @@
       </collision>
       <xacro:cylinder_inertial radius="${wrist_3_inertia_radius}" length="${wrist_3_inertia_length}"  mass="${wrist_3_mass}">
-        <origin xyz="0.0 0.0 ${-0.5 * wrist_3_inertia_length}" rpy="0 0 0" />
+        <origin xyz="${wrist_3_cog}" rpy="0 0 0" />
       </xacro:cylinder_inertial>
     </link>

Commit message: description: remove ee_link link.
Also remove the tiny collision object, as it's no longer needed now that MoveIt has been fixed.

File: ur_description/urdf/ur_macro.xacro (robot description, xacro)
@@ -211,16 +211,4 @@
       </xacro:cylinder_inertial>
     </link>
-    <link name="${prefix}ee_link">
-      <!-- TODO: remove this. This was only added to work-around a MoveIt issue
-           where links without geometry were ignored while collision checking.
-           NOTE: this will be removed in a future revision of this file.
-      -->
-      <collision>
-        <geometry>
-          <box size="0.01 0.01 0.01"/>
-        </geometry>
-        <origin rpy="0 0 0" xyz="-0.01 0 0"/>
-      </collision>
-    </link>
     <!-- joints: main serial chain -->
     <joint name="${prefix}shoulder_pan_joint" type="revolute">
@@ -292,9 +280,4 @@
       </xacro:if>
       <dynamics damping="0" friction="0"/>
-    </joint>
-    <joint name="${prefix}ee_fixed_joint" type="fixed">
-      <parent link="${prefix}wrist_3_link" />
-      <child link="${prefix}ee_link" />
-      <origin xyz="0 0 0" rpy="0.0 ${-pi/2.0} ${pi/2.0}" />
     </joint>
     <!-- ROS base_link to UR 'Base' Coordinates transform -->

Commit message: description: introduce flange frame.
This is the correct EEF attachment point: REP-103 aligned and no unwanted rotations (as tool0).

File: ur_description/urdf/ur_macro.xacro (robot description, xacro)
@@ -292,9 +292,16 @@
       <child link="${prefix}base"/>
     </joint>
+    <!-- ROS-Industrial 'flange' frame: attachment point for EEF models -->
+    <link name="${prefix}flange" />
+    <joint name="${prefix}wrist_3-flange" type="fixed">
+      <parent link="${prefix}wrist_3_link" />
+      <child link="${prefix}flange" />
+      <origin xyz="0 0 0" rpy="0 ${-pi/2.0} ${-pi/2.0}" />
+    </joint>
     <!-- Frame coincident with all-zeros TCP on UR controller -->
     <link name="${prefix}tool0"/>
-    <joint name="${prefix}wrist_3_passive_joint" type="fixed">
+    <joint name="${prefix}flange-tool0" type="fixed">
       <origin xyz="0 0 0" rpy="0 0 0"/>
-      <parent link="${prefix}wrist_3_link"/>
+      <parent link="${prefix}flange"/>
       <child link="${prefix}tool0"/>
     </joint>

Commit message: description: fix orientation of tool0.
Now that flange is its parent.

File: ur_description/urdf/ur_macro.xacro (robot description, xacro)
@@ -302,5 +302,6 @@
     <link name="${prefix}tool0"/>
     <joint name="${prefix}flange-tool0" type="fixed">
-      <origin xyz="0 0 0" rpy="0 0 0"/>
+      <!-- default toolframe: X+ left, Y+ up, Z+ front -->
+      <origin xyz="0 0 0" rpy="${pi/2.0} 0 ${pi/2.0}"/>
       <parent link="${prefix}flange"/>
       <child link="${prefix}tool0"/>

Commit message: description: remove the 'base_correction' property.
There is an offset between 'base_link' and 'base', but it's a fixed one, known and does not need to be a property.

Rectify the problem with the 'base_link' mesh in a follow-up commit.

File: ur_description/urdf/ur_macro.xacro (robot description, xacro)
@@ -63,14 +63,8 @@
     <!-- Add URDF transmission elements (for ros_control) -->
     <xacro:ur_arm_transmission prefix="${prefix}" hw_interface="${transmission_hw_interface}" />
-    <!-- This is for compatibility reasons, as the rotiation between base and
-         base_link has always been 180 degrees in ur_description. The reason
-         for this is unknown, but for now this kept as a form of bw-compatibility.
-         NOTE: this WILL be removed in a future revision of this file
-     -->
-    <xacro:property name="base_correction" value="${pi}" />
     <!-- links: main serial chain -->
     <link name="${prefix}base_link" >
       <visual>
-        <origin xyz="0 0 0" rpy="0 0 ${base_correction}"/>
+        <origin xyz="0 0 0" rpy="0 0 0"/>
         <geometry>
           <mesh filename="${base_visual_mesh}"/>
@@ -81,5 +75,5 @@
       </visual>
       <collision>
-        <origin xyz="0 0 0" rpy="0 0 ${base_correction}"/>
+        <origin xyz="0 0 0" rpy="0 0 0"/>
         <geometry>
           <mesh filename="${base_collision_mesh}"/>
@@ -215,5 +209,5 @@
       <parent link="${prefix}base_link" />
       <child link="${prefix}shoulder_link" />
-      <origin xyz="${shoulder_x} ${shoulder_y} ${shoulder_z}" rpy="${shoulder_roll} ${shoulder_pitch} ${shoulder_yaw + base_correction}" />
+      <origin xyz="${shoulder_x} ${shoulder_y} ${shoulder_z}" rpy="${shoulder_roll} ${shoulder_pitch} ${shoulder_yaw}" />
       <axis xyz="0 0 1" />
       <limit lower="${shoulder_pan_lower_limit}" upper="${shoulder_pan_upper_limit}"
@@ -284,9 +278,5 @@
     <link name="${prefix}base"/>
     <joint name="${prefix}base_link-base_fixed_joint" type="fixed">
-      <!-- NOTE: this rotation is only needed as long as base_link itself is
-      not corrected wrt the real robot (ie: rotated over 180
-      degrees)
-      -->
-      <origin xyz="0 0 0" rpy="0 0 ${-pi}"/>
+      <origin xyz="0 0 0" rpy="0 0 0"/>
       <parent link="${prefix}base_link"/>
       <child link="${prefix}base"/>

Commit message: description: introduce base_link_inertia link.
To work around the root-link-with-inertia limitation in KDL.

File: ur_description/urdf/ur_macro.xacro (robot description, xacro)
@@ -64,5 +64,6 @@
     <xacro:ur_arm_transmission prefix="${prefix}" hw_interface="${transmission_hw_interface}" />
     <!-- links: main serial chain -->
-    <link name="${prefix}base_link" >
+    <link name="${prefix}base_link"/>
+    <link name="${prefix}base_link_inertia">
       <visual>
         <origin xyz="0 0 0" rpy="0 0 0"/>
@@ -206,6 +207,11 @@
     </link>
     <!-- joints: main serial chain -->
+    <joint name="${prefix}base_link-base_link_inertia" type="fixed">
+      <parent link="${prefix}base_link" />
+      <child link="${prefix}base_link_inertia" />
+      <origin xyz="0 0 0" rpy="0 0 0" />
+    </joint>
     <joint name="${prefix}shoulder_pan_joint" type="revolute">
-      <parent link="${prefix}base_link" />
+      <parent link="${prefix}base_link_inertia" />
       <child link="${prefix}shoulder_link" />
       <origin xyz="${shoulder_x} ${shoulder_y} ${shoulder_z}" rpy="${shoulder_roll} ${shoulder_pitch} ${shoulder_yaw}" />

Commit message: description: rotate for UR internal frames.

File: ur_description/urdf/ur_macro.xacro (robot description, xacro)
@@ -210,5 +210,10 @@
       <parent link="${prefix}base_link" />
       <child link="${prefix}base_link_inertia" />
-      <origin xyz="0 0 0" rpy="0 0 0" />
+      <!-- 'base_link' is REP-103 aligned (so X+ forward), while the internal
+           frames of the robot/controller have X+ pointing backwards.
+           Use the joint between 'base_link' and 'base_link_inertia' (a dummy
+           link/frame) to introduce the necessary rotation over Z (of pi rad).
+      -->
+      <origin xyz="0 0 0" rpy="0 0 ${pi}" />
     </joint>
     <joint name="${prefix}shoulder_pan_joint" type="revolute">

Commit message: description: fix orientation of 'base' frame.
So it's coincident with the robot's/controller's 'Base' frame. It's actually 180 degrees rotated over Z wrt 'base_link'.

File: ur_description/urdf/ur_macro.xacro (robot description, xacro)
@@ -289,5 +289,10 @@
     <link name="${prefix}base"/>
     <joint name="${prefix}base_link-base_fixed_joint" type="fixed">
-      <origin xyz="0 0 0" rpy="0 0 0"/>
+      <!-- Note the rotation over Z of pi radians: as base_link is REP-103
+           aligned (ie: has X+ forward, Y+ left and Z+ up), this is needed
+           to correctly align 'base' with the 'Base' coordinate system of
+           the UR controller.
+      -->
+      <origin xyz="0 0 0" rpy="0 0 ${pi}"/>
       <parent link="${prefix}base_link"/>
       <child link="${prefix}base"/>

Commit message: description: correct orientation of Base mesh.
Connector should be aligned with Y+ of 'base' frame.

File: ur_description/urdf/ur_macro.xacro (robot description, xacro)
@@ -67,5 +67,5 @@
     <link name="${prefix}base_link_inertia">
       <visual>
-        <origin xyz="0 0 0" rpy="0 0 0"/>
+        <origin xyz="0 0 0" rpy="0 0 ${pi}"/>
         <geometry>
           <mesh filename="${base_visual_mesh}"/>
@@ -76,5 +76,5 @@
       </visual>
       <collision>
-        <origin xyz="0 0 0" rpy="0 0 0"/>
+        <origin xyz="0 0 0" rpy="0 0 ${pi}"/>
         <geometry>
           <mesh filename="${base_collision_mesh}"/>

Commit message: description: use mat def from yaml for base_link.

File: ur_description/urdf/ur_macro.xacro (robot description, xacro)
@@ -76,6 +76,6 @@
           <mesh filename="${base_visual_mesh}"/>
         </geometry>
-        <material name="LightGrey">
-          <color rgba="0.7 0.7 0.7 1.0"/>
+        <material name="${base_visual_material_name}">
+          <color rgba="${base_visual_material_color}"/>
         </material>
       </visual>
