Commit message: Simplification of generic xacro and launch files
Model specific xacro and launch files replaced by generic ones.
Default arguments and parameters only defined once in lowest level files by replacing empty strings.
Omit properties same as default.
Still all properties can be overridden in upper level files.
Less redefining of arguments and parameters by pass_all_args in launch and using upper level parameters in xacro files.
Paths, file names, names, comments and format adjusted.

File: ur_description/urdf/macro.xacro (robot description, xacro)
@@ -6,6 +6,6 @@
     expecting a flattened '.urdf' file. See the top-level '.xacro' for that
     (but note: that .xacro must still be processed by the xacro command).
-    For use in '.launch' files: use one of the 'load_urX.launch' convenience
-    launch files.
+    For use in '.launch' files: use the 'load.launch' convenience
+    launch file.
     This file models the base kinematic chain of a UR robot, which then gets
     parameterised by various configuration files to convert it into a UR3(e),
@@ -42,18 +42,43 @@
      - Muhammad Asif Rana
   -->
-  <xacro:include filename="$(find ur_description)/urdf/inc/ur_transmissions.xacro" />
-  <xacro:include filename="$(find ur_description)/urdf/inc/ur_common.xacro" />
-  <xacro:macro name="ur_robot" params="
-    prefix
-    joint_limits_parameters_file
-    kinematics_parameters_file
-    physical_parameters_file
-    visual_parameters_file
+  <xacro:include filename="$(find ur_description)/urdf/transmissions.xacro" />
+  <xacro:macro name="ur" params="
+    model:=^|''
+    prefix:=^|''
+    joint_limits_parameters_file:=^|''
+    kinematics_parameters_file:=^|''
+    physical_parameters_file:=^|''
+    visual_parameters_file:=^|''
     transmission_hw_interface:=hardware_interface/PositionJointInterface
-    safety_limits:=false
-    safety_pos_margin:=0.15
-    safety_k_position:=20"
-  >
+    safety_limits:=^|''
+    safety_pos_margin:=^|''
+    safety_k_position:=^|''
+  ">
+    <!-- Override empty parameters with default values -->
+    <xacro:if value="${not joint_limits_parameters_file}">
+      <xacro:property name="joint_limits_parameters_file" value="$(find ur_description)/config/${model}/joint_limits.yaml"/>
+    </xacro:if>
+    <xacro:if value="${not kinematics_parameters_file}">
+      <xacro:property name="kinematics_parameters_file" value="$(find ur_description)/config/${model}/default_kinematics.yaml"/>
+    </xacro:if>
+    <xacro:if value="${not physical_parameters_file}">
+      <xacro:property name="physical_parameters_file" value="$(find ur_description)/config/${model}/physical_parameters.yaml"/>
+    </xacro:if>
+    <xacro:if value="${not visual_parameters_file}">
+      <xacro:property name="visual_parameters_file" value="$(find ur_description)/config/${model}/visual_parameters.yaml"/>
+    </xacro:if>
+    <xacro:if value="${not safety_limits}">
+      <xacro:property name="safety_limits" value="false"/>
+    </xacro:if>
+    <xacro:if value="${not safety_pos_margin}">
+      <xacro:property name="safety_pos_margin" value="0.15"/>
+    </xacro:if>
+    <xacro:if value="${not safety_k_position}">
+      <xacro:property name="safety_k_position" value="20"/>
+    </xacro:if>
+    <!-- Non empty prefix ends with "_" -->
+    <xacro:property name="prefix" value="${prefix + '_' if prefix and not prefix.endswith('_') else ''}" lazy_eval="false"/>
     <!-- Load configuration data from the provided .yaml files -->
+    <xacro:include filename="$(find ur_description)/urdf/common.xacro" />
     <xacro:read_model_data
       joint_limits_parameters_file="${joint_limits_parameters_file}"

File: ur_description/urdf/ur.xacro (robot description, xacro)
@@ -1,30 +1,34 @@
 <?xml version="1.0"?>
-<robot xmlns:xacro="http://wiki.ros.org/xacro" name="$(arg robot_model)_robot">
-   <!-- import main macro -->
-   <xacro:include filename="$(find ur_description)/urdf/inc/ur_macro.xacro"/>
-   <!-- parameters -->
-   <xacro:arg name="joint_limit_params" default=""/>
-   <xacro:arg name="kinematics_params" default=""/>
-   <xacro:arg name="physical_params" default=""/>
-   <xacro:arg name="visual_params" default=""/>
-   <!-- legal values:
+<robot xmlns:xacro="http://wiki.ros.org/xacro" name="$(arg model)_robot">
+  <!-- Parameters -->
+  <xacro:arg name="model" default=""/> <!-- ur3, ur3e, ur5, ur5e, ur10, ur10e or ur16e -->
+  <xacro:arg name="prefix" default=""/>
+  <xacro:arg name="joint_limit_params" default=""/>
+  <xacro:arg name="kinematics_params" default=""/>
+  <xacro:arg name="physical_params" default=""/>
+  <xacro:arg name="visual_params" default=""/>
+  <!-- legal values:
          - hardware_interface/PositionJointInterface
          - hardware_interface/VelocityJointInterface
          - hardware_interface/EffortJointInterface
-   -->
-   <xacro:arg name="transmission_hw_interface" default="hardware_interface/PositionJointInterface"/>
-   <xacro:arg name="safety_limits" default="false"/>
-   <xacro:arg name="safety_pos_margin" default="0.15"/>
-   <xacro:arg name="safety_k_position" default="20"/>
-   <!-- arm -->
-   <xacro:ur_robot
-     prefix=""
-     joint_limits_parameters_file="$(arg joint_limit_params)"
-     kinematics_parameters_file="$(arg kinematics_params)"
-     physical_parameters_file="$(arg physical_params)"
-     visual_parameters_file="$(arg visual_params)"
-     transmission_hw_interface="$(arg transmission_hw_interface)"
-     safety_limits="$(arg safety_limits)"
-     safety_pos_margin="$(arg safety_pos_margin)"
-     safety_k_position="$(arg safety_k_position)"/>
+  -->
+  <xacro:arg name="transmission_hw_interface" default="hardware_interface/PositionJointInterface"/>
+  <xacro:arg name="safety_limits" default=""/>
+  <xacro:arg name="safety_pos_margin" default=""/>
+  <xacro:arg name="safety_k_position" default=""/>
+  <!-- Import macro -->
+  <xacro:include filename="$(find ur_description)/urdf/macro.xacro"/>
+  <!-- Call macro -->
+  <xacro:ur
+    model="$(arg model)"
+    prefix="$(arg prefix)"
+    joint_limits_parameters_file="$(arg joint_limit_params)"
+    kinematics_parameters_file="$(arg kinematics_params)"
+    physical_parameters_file="$(arg physical_params)"
+    visual_parameters_file="$(arg visual_params)"
+    transmission_hw_interface="$(arg transmission_hw_interface)"
+    safety_limits="$(arg safety_limits)"
+    safety_pos_margin="$(arg safety_pos_margin)"
+    safety_k_position="$(arg safety_k_position)"
+  />
 </robot>

File: ur_gazebo/urdf/macro.xacro (robot description, xacro)
@@ -9,10 +9,10 @@
     expecting a flattened '.urdf' file. See the top-level '.xacro' for that
     (but note: that .xacro must still be processed by the xacro command).
-    For use in '.launch' files: use one of the 'load_urX.launch' convenience
+    For use in '.launch' files: use the 'load.launch' convenience
     launch files.
     NOTE: this Gazebo model makes use of the same set of parameter files as the
     main xacro macro (in ur_description). It is therefor possible to use the
     kinematic calibration exported from a REAL UR robot. Please refer to the
-    ur_macro.xacro in ur_description for more information about this.
+    macro.xacro in ur_description for more information about this.
     Main author of the migration to yaml configs: Ludovic Delval.
     Contributors to previous versions (in no particular order):
@@ -31,32 +31,25 @@
   -->
   <!-- Definition of the main macro -->
-  <xacro:macro name="ur_robot_gazebo" params="
-   prefix
-   joint_limits_parameters_file
-   kinematics_parameters_file
-   physical_parameters_file
-   visual_parameters_file
-   transmission_hw_interface:=hardware_interface/EffortJointInterface
-   safety_limits:=false safety_pos_margin:=0.15 safety_k_position:=20"
-  >
+  <xacro:macro name="ur_gazebo" params="
+    model:=^|''
+    prefix:=^|''
+    joint_limits_parameters_file:=^|''
+    kinematics_parameters_file:=^|''
+    physical_parameters_file:=^|''
+    visual_parameters_file:=^|''
+    transmission_hw_interface:=hardware_interface/EffortJointInterface
+    safety_limits:=^|''
+    safety_pos_margin:=^|''
+    safety_k_position:=^|''
+  ">
     <!--
       Import the xacro macro for the REAL robot (which we'll augment with Gazebo
       specific elements in the wrapper macro below).
-      NOTE: this imports the '_macro.xacro' from ur_description, as that contains
+      NOTE: this imports the 'macro.xacro' from ur_description, as that contains
       the definitions for the real robot.
     -->
-  <xacro:include filename="$(find ur_description)/urdf/inc/ur_macro.xacro"/>
+    <xacro:include filename="$(find ur_description)/urdf/macro.xacro"/>
     <!-- Instantiate model for the REAL robot. -->
-    <xacro:ur_robot
-      prefix="${prefix}"
-      joint_limits_parameters_file="${joint_limits_parameters_file}"
-      kinematics_parameters_file="${kinematics_parameters_file}"
-      physical_parameters_file="${physical_parameters_file}"
-      visual_parameters_file="${visual_parameters_file}"
-      transmission_hw_interface="${transmission_hw_interface}"
-      safety_limits="${safety_limits}"
-      safety_pos_margin="${safety_pos_margin}"
-      safety_k_position="${safety_k_position}"
-    />
+    <xacro:ur/>
     <!-- Configure self collision properties per link -->
     <gazebo reference="${prefix}shoulder_link">

File: ur_gazebo/urdf/ur.xacro (robot description, xacro)
@@ -1,7 +1,7 @@
 <?xml version="1.0"?>
-<robot xmlns:xacro="http://wiki.ros.org/xacro" name="$(arg robot_model)_robot">
+<robot xmlns:xacro="http://wiki.ros.org/xacro" name="$(arg model)_robot">
   <!--
     This is a top-level xacro instantiating the Gazebo-specific version of the
-    'ur_robot' macro (ie: 'ur_robot_gazebo') and passing it values for all its
+    'ur_robot' macro (ie: 'ur_gazebo') and passing it values for all its
     required arguments.
     This file should be considered the Gazebo-specific variant of the file
@@ -24,6 +24,7 @@
           xacro macro (which is hosted by ur_description).
   -->
-  <xacro:include filename="$(find ur_gazebo)/urdf/ur_macro.xacro"/>
+  <xacro:include filename="$(find ur_gazebo)/urdf/macro.xacro"/>
   <!--Declare arguments -->
+  <xacro:arg name="prefix" default=""/>
   <xacro:arg name="joint_limit_params" default=""/>
   <xacro:arg name="physical_params" default=""/>
@@ -39,10 +40,11 @@
   -->
   <xacro:arg name="transmission_hw_interface" default="hardware_interface/EffortJointInterface"/>
-  <xacro:arg name="safety_limits" default="false"/>
-  <xacro:arg name="safety_pos_margin" default="0.15"/>
-  <xacro:arg name="safety_k_position" default="20"/>
+  <xacro:arg name="safety_limits" default=""/>
+  <xacro:arg name="safety_pos_margin" default=""/>
+  <xacro:arg name="safety_k_position" default=""/>
   <!-- Instantiate the Gazebo robot and pass it all the required arguments. -->
-  <xacro:ur_robot_gazebo
-    prefix=""
+  <xacro:ur_gazebo
+    model="$(arg model)"
+    prefix="$(arg prefix)"
     joint_limits_parameters_file="$(arg joint_limit_params)"
     kinematics_parameters_file="$(arg kinematics_params)"

Commit message: Revolute joint macro using configuration data

File: ur_description/urdf/macro.xacro (robot description, xacro)
@@ -42,5 +42,4 @@
      - Muhammad Asif Rana
   -->
-  <xacro:include filename="$(find ur_description)/urdf/transmissions.xacro" />
   <xacro:macro name="ur" params="
     model:=^|''
@@ -97,6 +96,4 @@
       visual_parameters_file="${visual_parameters_file}"/>
     <!-- Links: main serial chain -->
-    <xacro:ur_arm_transmission prefix="${prefix}" hw_interface="${transmission_hw_interface}" />
-    <!-- links: main serial chain -->
     <link name="${prefix}base_link"/>
     <!-- ROS-Industrial 'base' frame: base_link to UR 'Base' Coordinates transform -->
@@ -169,95 +166,51 @@
          link/frame) to introduce the necessary rotation over Z (of pi rad). -->
     <xacro:joint_fixed parent="base_link" child="base_inertia_link" rpy="0 0 ${pi}"/>
-    <joint name="${prefix}shoulder_pan_joint" type="revolute">
-      <parent link="${prefix}base_link_inertia" />
-      <child link="${prefix}shoulder_link" />
-      <origin xyz="${shoulder_x} ${shoulder_y} ${shoulder_z}" rpy="${shoulder_roll} ${shoulder_pitch} ${shoulder_yaw}" />
-      <axis xyz="0 0 1" />
-      <limit lower="${shoulder_pan_lower_limit}" upper="${shoulder_pan_upper_limit}"
-        effort="${shoulder_pan_effort_limit}" velocity="${shoulder_pan_velocity_limit}"/>
-      <xacro:if value="${safety_limits}">
-         <safety_controller soft_lower_limit="${shoulder_pan_lower_limit + safety_pos_margin}" soft_upper_limit="${shoulder_pan_upper_limit - safety_pos_margin}" k_position="${safety_k_position}" k_velocity="0.0"/>
-      </xacro:if>
-      <dynamics damping="0" friction="0"/>
-    </joint>
-    <joint name="${prefix}shoulder_lift_joint" type="revolute">
-      <parent link="${prefix}shoulder_link" />
-      <child link="${prefix}upper_arm_link" />
-      <origin xyz="${upper_arm_x} ${upper_arm_y} ${upper_arm_z}" rpy="${upper_arm_roll} ${upper_arm_pitch} ${upper_arm_yaw}" />
-      <axis xyz="0 0 1" />
-      <limit lower="${shoulder_lift_lower_limit}" upper="${shoulder_lift_upper_limit}"
-        effort="${shoulder_lift_effort_limit}" velocity="${shoulder_lift_velocity_limit}"/>
-      <xacro:if value="${safety_limits}">
-         <safety_controller soft_lower_limit="${shoulder_lift_lower_limit + safety_pos_margin}" soft_upper_limit="${shoulder_lift_upper_limit - safety_pos_margin}" k_position="${safety_k_position}" k_velocity="0.0"/>
-      </xacro:if>
-      <dynamics damping="0" friction="0"/>
-    </joint>
-    <joint name="${prefix}elbow_joint" type="revolute">
-      <parent link="${prefix}upper_arm_link" />
-      <child link="${prefix}forearm_link" />
-      <origin xyz="${forearm_x} ${forearm_y} ${forearm_z}" rpy="${forearm_roll} ${forearm_pitch} ${forearm_yaw}" />
-      <axis xyz="0 0 1" />
-      <limit lower="${elbow_joint_lower_limit}" upper="${elbow_joint_upper_limit}"
-        effort="${elbow_joint_effort_limit}" velocity="${elbow_joint_velocity_limit}"/>
-      <xacro:if value="${safety_limits}">
-         <safety_controller soft_lower_limit="${elbow_joint_lower_limit + safety_pos_margin}" soft_upper_limit="${elbow_joint_upper_limit - safety_pos_margin}" k_position="${safety_k_position}" k_velocity="0.0"/>
-      </xacro:if>
-      <dynamics damping="0" friction="0"/>
-    </joint>
-    <joint name="${prefix}wrist_1_joint" type="revolute">
-      <parent link="${prefix}forearm_link" />
-      <child link="${prefix}wrist_1_link" />
-      <origin xyz="${wrist_1_x} ${wrist_1_y} ${wrist_1_z}" rpy="${wrist_1_roll} ${wrist_1_pitch} ${wrist_1_yaw}" />
-      <axis xyz="0 0 1" />
-      <limit lower="${wrist_1_lower_limit}" upper="${wrist_1_upper_limit}"
-        effort="${wrist_1_effort_limit}" velocity="${wrist_1_velocity_limit}"/>
-      <xacro:if value="${safety_limits}">
-         <safety_controller soft_lower_limit="${wrist_1_lower_limit + safety_pos_margin}" soft_upper_limit="${wrist_1_upper_limit - safety_pos_margin}" k_position="${safety_k_position}" k_velocity="0.0"/>
-      </xacro:if>
-      <dynamics damping="0" friction="0"/>
-    </joint>
-    <joint name="${prefix}wrist_2_joint" type="revolute">
-      <parent link="${prefix}wrist_1_link" />
-      <child link="${prefix}wrist_2_link" />
-      <origin xyz="${wrist_2_x} ${wrist_2_y} ${wrist_2_z}" rpy="${wrist_2_roll} ${wrist_2_pitch} ${wrist_2_yaw}" />
-      <axis xyz="0 0 1" />
-      <limit lower="${wrist_2_lower_limit}" upper="${wrist_2_upper_limit}"
-             effort="${wrist_2_effort_limit}" velocity="${wrist_2_velocity_limit}"/>
-      <xacro:if value="${safety_limits}">
-         <safety_controller soft_lower_limit="${wrist_2_lower_limit + safety_pos_margin}" soft_upper_limit="${wrist_2_upper_limit - safety_pos_margin}" k_position="${safety_k_position}" k_velocity="0.0"/>
-      </xacro:if>
-      <dynamics damping="0" friction="0"/>
-    </joint>
-    <joint name="${prefix}wrist_3_joint" type="revolute">
-      <parent link="${prefix}wrist_2_link" />
-      <child link="${prefix}wrist_3_link" />
-      <origin xyz="${wrist_3_x} ${wrist_3_y} ${wrist_3_z}" rpy="${wrist_3_roll} ${wrist_3_pitch} ${wrist_3_yaw}" />
-      <axis xyz="0 0 1" />
-      <limit lower="${wrist_3_lower_limit}" upper="${wrist_3_upper_limit}"
-             effort="${wrist_3_effort_limit}" velocity="${wrist_3_velocity_limit}"/>
-      <xacro:if value="${safety_limits}">
-         <safety_controller soft_lower_limit="${wrist_3_lower_limit + safety_pos_margin}" soft_upper_limit="${wrist_3_upper_limit - safety_pos_margin}" k_position="${safety_k_position}" k_velocity="0.0"/>
-      </xacro:if>
-      <dynamics damping="0" friction="0"/>
-    </joint>
-    <!-- ROS-Industrial 'base' frame: base_link to UR 'Base' Coordinates transform -->
-    <link name="${prefix}base"/>
-    <joint name="${prefix}base_link-base_fixed_joint" type="fixed">
-      <!-- Note the rotation over Z of pi radians: as base_link is REP-103
-           aligned (ie: has X+ forward, Y+ left and Z+ up), this is needed
-           to correctly align 'base' with the 'Base' coordinate system of
-           the UR controller.
+    <!-- Note the rotation over Z of pi radians: as base_link is REP-103
+         aligned (ie: has X+ forward, Y+ left and Z+ up), this is needed
+         to correctly align 'base' with the 'Base' coordinate system of
+         the UR controller. -->
     <xacro:joint_fixed parent="base_link" child="base" rpy="0 0 ${pi}"/>
-      <origin xyz="0 0 0" rpy="0 0 ${pi}"/>
-      <parent link="${prefix}base_link"/>
-      <child link="${prefix}base"/>
-    </joint>
-    <!-- ROS-Industrial 'flange' frame: attachment point for EEF models -->
-    <link name="${prefix}flange" />
-    <joint name="${prefix}wrist_3-flange" type="fixed">
-      <parent link="${prefix}wrist_3_link" />
-      <child link="${prefix}flange" />
-      <origin xyz="0 0 0" rpy="0 ${-pi/2.0} ${-pi/2.0}" />
-    </joint>
+    <!-- Controlled revolute joint macro using configuration data -->
+    <xacro:macro name="joint" params="name parent child">
+       <!-- Kinematics -->
+      <xacro:property name="kinematic" value="${kinematics[child]}"/>
+      <xacro:property name="x" value="${kinematic['x']}"/>
+      <xacro:property name="y" value="${kinematic['y']}"/>
+      <xacro:property name="z" value="${kinematic['z']}"/>
+      <xacro:property name="roll" value="${kinematic['roll']}"/>
+      <xacro:property name="pitch" value="${kinematic['pitch']}"/>
+      <xacro:property name="yaw" value="${kinematic['yaw']}"/>
+      <!-- Joint limits -->
+      <xacro:property name="limit" value="${limits[name]}"/>
+      <xacro:property name="lower_limit" value="${limit['min_position']}"/>
+      <xacro:property name="upper_limit" value="${limit['max_position']}"/>
+      <xacro:property name="velocity_limit" value="${limit['max_velocity']}"/>
+      <xacro:property name="effort_limit" value="${limit['max_effort']}"/>
+      <joint name="${prefix}${name}_joint" type="revolute">
+        <parent link="${prefix}${parent}_link"/>
+        <child link="${prefix}${child}_link"/>
+        <origin xyz="${x} ${y} ${z}" rpy="${roll} ${pitch} ${yaw}"/>
+        <axis xyz="0 0 1"/>
+        <limit lower="${lower_limit}" upper="${upper_limit}" effort="${effort_limit}" velocity="${velocity_limit}"/>
+        <xacro:if value="${safety_limits}">
+           <safety_controller soft_lower_limit="${lower_limit + safety_pos_margin}" soft_upper_limit="${upper_limit - safety_pos_margin}" k_position="${safety_k_position}" k_velocity="0"/>
+        </xacro:if>
+      </joint>
+      <!-- Transmission for ros_control -->
+      <transmission name="${prefix}${name}_trans">
+        <type>transmission_interface/SimpleTransmission</type>
+        <joint name="${prefix}${name}_joint">
+          <hardwareInterface>${transmission_hw_interface}</hardwareInterface>
+        </joint>
+        <actuator name="${prefix}${name}_motor"/>
+      </transmission>
+    </xacro:macro>
+    <!-- Controlled revolute joins -->
+    <xacro:joint name="shoulder_pan" parent="base_inertia" child="shoulder"/>
+    <xacro:joint name="shoulder_lift" parent="shoulder" child="upper_arm"/>
+    <xacro:joint name="elbow" parent="upper_arm" child="forearm"/>
+    <xacro:joint name="wrist_1" parent="forearm" child="wrist_1"/>
+    <xacro:joint name="wrist_2" parent="wrist_1" child="wrist_2"/>
+    <xacro:joint name="wrist_3" parent="wrist_2" child="wrist_3"/>
     <xacro:joint_fixed parent="wrist_3_link" child="flange" rpy="0 ${-pi/2} ${-pi/2}"/>
     <!-- Default toolframe: X+ left, Y+ up, Z+ front -->
