Commit message: gazebo: use new arg names for joint limits.
Renamed in ur_description, so use the new names here as well and pass the right values.

File: ur_gazebo/urdf/ur_robot.urdf.xacro (robot description, xacro)
@@ -3,5 +3,5 @@
        name="ur" >
    <!-- common stuff -->
-   <xacro:arg name="joints_limits_params" default="$(find ur_description)/config/ur3/joint_limits.yaml"/>
+   <xacro:arg name="joint_limit_params" default="$(find ur_description)/config/ur3/joint_limits.yaml"/>
    <xacro:arg name="physical_params" default="$(find ur_description)/config/ur3/physical_parameters.yaml"/>
    <xacro:arg name="kinematics_params" default="$(find ur_description)/config/ur3/default_kinematics.yaml"/>
@@ -15,5 +15,5 @@
    <xacro:include filename="$(find ur_gazebo)/urdf/common.gazebo.xacro"/>
    <!-- arm -->
-   <xacro:ur_gazebo_robot prefix="" joints_limits_parameters_file="${load_yaml('$(arg joints_limits_params)')}"
+   <xacro:ur_gazebo_robot prefix="" joint_limits_parameters_file="${load_yaml('$(arg joint_limit_params)')}"
                              kinematics_parameters_file="${load_yaml('$(arg kinematics_params)')}"
                              physical_parameters_file="${load_yaml('$(arg physical_params)')}"

File: ur_gazebo/urdf/ur_robot_gazebo.macro.xacro (robot description, xacro)
@@ -5,8 +5,8 @@
 -->
  <xacro:include filename="$(find ur_description)/urdf/ur_macro.xacro"/>
- <xacro:macro name="ur_gazebo_robot" params="prefix joints_limits_parameters_file kinematics_parameters_file physical_parameters_file visual_parameters_file
+ <xacro:macro name="ur_gazebo_robot" params="prefix joint_limits_parameters_file kinematics_parameters_file physical_parameters_file visual_parameters_file
                   transmission_hw_interface:=hardware_interface/PositionJointInterface
                   safety_limits:=false safety_pos_margin:=0.15 safety_k_position:=20">
-    <xacro:ur_robot prefix="${prefix}" joints_limits_parameters_file="${joints_limits_parameters_file}"
+    <xacro:ur_robot prefix="${prefix}" joint_limits_parameters_file="${joint_limits_parameters_file}"
                     kinematics_parameters_file="${kinematics_parameters_file}"
                     physical_parameters_file="${physical_parameters_file}"
