Commit message: gazebo: use new robot and macro name.
Align with filenames and other ROS-Industrial Gazebo support packages.

File: ur_gazebo/urdf/ur.xacro (robot description, xacro)
@@ -1,5 +1,4 @@
 <?xml version="1.0"?>
-<robot xmlns:xacro="http://wiki.ros.org/xacro"
-       name="ur" >
+<robot xmlns:xacro="http://wiki.ros.org/xacro" name="ur_robot_gazebo">
    <!-- common stuff -->
    <xacro:arg name="joint_limit_params" default="$(find ur_description)/config/ur3/joint_limits.yaml"/>
@@ -14,5 +13,5 @@
    <xacro:include filename="$(find ur_gazebo)/urdf/ur_macro.xacro"/>
    <!-- arm -->
-   <xacro:ur_gazebo_robot prefix="" joint_limits_parameters_file="$(arg joint_limit_params)"
+   <xacro:ur_robot_gazebo prefix="" joint_limits_parameters_file="$(arg joint_limit_params)"
                              kinematics_parameters_file="$(arg kinematics_params)"
                              physical_parameters_file="$(arg physical_params)"

File: ur_gazebo/urdf/ur_macro.xacro (robot description, xacro)
@@ -5,5 +5,5 @@
 -->
  <xacro:include filename="$(find ur_description)/urdf/ur_macro.xacro"/>
- <xacro:macro name="ur_gazebo_robot" params="prefix joint_limits_parameters_file kinematics_parameters_file physical_parameters_file visual_parameters_file
+ <xacro:macro name="ur_robot_gazebo" params="prefix joint_limits_parameters_file kinematics_parameters_file physical_parameters_file visual_parameters_file
                   transmission_hw_interface:=hardware_interface/PositionJointInterface
                   safety_limits:=false safety_pos_margin:=0.15 safety_k_position:=20">

Commit message: gazebo: formatting and comments of xacros.

File: ur_gazebo/urdf/ur.xacro (robot description, xacro)
@@ -1,29 +1,58 @@
 <?xml version="1.0"?>
 <robot xmlns:xacro="http://wiki.ros.org/xacro" name="ur_robot_gazebo">
-   <!-- common stuff -->
+   <!--
+     This is a top-level xacro instantiating the Gazebo-specific version of the
+     'ur_robot' macro (ie: 'ur_robot_gazebo') and passing it values for all its
+     required arguments.
+     This file should be considered the Gazebo-specific variant of the file
+     with the same name in the ur_description package. It accepts the same
+     arguments, but instead of configuring everything for a real robot, will
+     generate a Gazebo-compatible URDF with a ros_control hardware_interface
+     attached to it.
+     Only use this top-level xacro if you plan on spawning the robot in Gazebo
+     'by itself', without any gripper or any other geometry attached.
+     If you need to attach an end-effector, camera or need to integrate the
+     robot into a larger workcell and want to spawn that as a single entity in
+     Gazebo, DO NOT EDIT THIS FILE.
+     Instead: create a new top-level xacro, give it a proper name, include the
+     required '.xacro' files, instantiate the models (ie: call the macros) and
+     connect everything by adding the appropriate joints.
+   -->
+   <!-- Import main macro.
+        Note: this imports the Gazebo-wrapper main macro, NOT the regular
+        xacro macro (which is hosted by ur_description).
+   -->
+   <xacro:include filename="$(find ur_gazebo)/urdf/ur_macro.xacro"/>
+   <!-- parameters -->
    <xacro:arg name="joint_limit_params" default="$(find ur_description)/config/ur3/joint_limits.yaml"/>
    <xacro:arg name="physical_params" default="$(find ur_description)/config/ur3/physical_parameters.yaml"/>
    <xacro:arg name="kinematics_params" default="$(find ur_description)/config/ur3/default_kinematics.yaml"/>
    <xacro:arg name="visual_params" default="$(find ur_description)/config/ur3/visual_parameters.yaml"/>
+   <!-- legal values:
+         - hardware_interface/PositionJointInterface
+         - hardware_interface/VelocityJointInterface
+         - hardware_interface/EffortJointInterface
+   -->
    <xacro:arg name="transmission_hw_interface" default="hardware_interface/PositionJointInterface"/>
    <xacro:arg name="safety_limits" default="false"/>
    <xacro:arg name="safety_pos_margin" default="0.15"/>
    <xacro:arg name="safety_k_position" default="20"/>
-   <!-- common stuff -->
-   <xacro:include filename="$(find ur_gazebo)/urdf/ur_macro.xacro"/>
-   <!-- arm -->
-   <xacro:ur_robot_gazebo prefix="" joint_limits_parameters_file="$(arg joint_limit_params)"
-                             kinematics_parameters_file="$(arg kinematics_params)"
-                             physical_parameters_file="$(arg physical_params)"
-                             visual_parameters_file="$(arg visual_params)"
-                             transmission_hw_interface="$(arg transmission_hw_interface)"
-                             safety_limits="$(arg safety_limits)"
-                             safety_pos_margin="$(arg safety_pos_margin)"
-                             safety_k_position="$(arg safety_k_position)"/>
-   <link name="world" />
+   <!-- Instantiate the Gazebo robot and pass it all the required arguments. -->
+   <xacro:ur_robot_gazebo
+     prefix=""
+     joint_limits_parameters_file="$(arg joint_limit_params)"
+     kinematics_parameters_file="$(arg kinematics_params)"
+     physical_parameters_file="$(arg physical_params)"
+     visual_parameters_file="$(arg visual_params)"
+     transmission_hw_interface="$(arg transmission_hw_interface)"
+     safety_limits="$(arg safety_limits)"
+     safety_pos_margin="$(arg safety_pos_margin)"
+     safety_k_position="$(arg safety_k_position)"/>
+   <!-- Attach the Gazebo model to Gazebo's world frame -->
+   <link name="world"/>
    <joint name="world_joint" type="fixed">
-      <parent link="world" />
-      <child link = "base_link" />
-      <origin xyz="0.0 0.0 0.0" rpy="0.0 0.0 0.0" />
+      <parent link="world"/>
+      <child link="base_link"/>
+      <origin xyz="0 0 0" rpy="0 0 0"/>
    </joint>
 </robot>

File: ur_gazebo/urdf/ur_macro.xacro (robot description, xacro)
@@ -1,2 +1,3 @@
+<?xml version="1.0"?>
 <robot xmlns:xacro="http://wiki.ros.org/xacro">
 <!--
@@ -4,16 +5,32 @@
   Contributor: Felix Messmer, Kelsey Hawkins, Jimmy Da Silva, Ajit Krisshna N L, Muhammad Asif Rana
 -->
+ <!-- Import the xacro macro for the REAL robot (which we'll augment with
+      Gazebo-specific elements in the wrapper macro below).
+      Note: this imports the '_macro.xacro' from ur_description, as that
+      contains the definitions for the real robot.
+ -->
  <xacro:include filename="$(find ur_description)/urdf/ur_macro.xacro"/>
- <xacro:macro name="ur_robot_gazebo" params="prefix joint_limits_parameters_file kinematics_parameters_file physical_parameters_file visual_parameters_file
-                  transmission_hw_interface:=hardware_interface/PositionJointInterface
-                  safety_limits:=false safety_pos_margin:=0.15 safety_k_position:=20">
-    <xacro:ur_robot prefix="${prefix}" joint_limits_parameters_file="${joint_limits_parameters_file}"
-                    kinematics_parameters_file="${kinematics_parameters_file}"
-                    physical_parameters_file="${physical_parameters_file}"
-                    visual_parameters_file="${visual_parameters_file}"
-                    transmission_hw_interface="${transmission_hw_interface}"
-                    safety_limits="${safety_limits}"
-                    safety_pos_margin="${safety_pos_margin}"
-                    safety_k_position="${safety_k_position}"/>
+ <xacro:macro name="ur_robot_gazebo" params="
+  prefix
+  joint_limits_parameters_file
+  kinematics_parameters_file
+  physical_parameters_file
+  visual_parameters_file
+  transmission_hw_interface:=hardware_interface/PositionJointInterface
+  safety_limits:=false safety_pos_margin:=0.15 safety_k_position:=20"
+ >
+    <!-- Instantiate model for the REAL robot.
+         Add additional elements needed by Gazebo as well.
+    -->
+    <xacro:ur_robot
+      prefix="${prefix}"
+      joint_limits_parameters_file="${joint_limits_parameters_file}"
+      kinematics_parameters_file="${kinematics_parameters_file}"
+      physical_parameters_file="${physical_parameters_file}"
+      visual_parameters_file="${visual_parameters_file}"
+      transmission_hw_interface="${transmission_hw_interface}"
+      safety_limits="${safety_limits}"
+      safety_pos_margin="${safety_pos_margin}"
+      safety_k_position="${safety_k_position}"/>
     <gazebo reference="${prefix}shoulder_link">
       <selfCollide>true</selfCollide>

Commit message: gazebo: 2-spaces per indent level.

File: ur_gazebo/urdf/ur.xacro (robot description, xacro)
@@ -1,58 +1,58 @@
 <?xml version="1.0"?>
 <robot xmlns:xacro="http://wiki.ros.org/xacro" name="ur_robot_gazebo">
-   <!--
-     This is a top-level xacro instantiating the Gazebo-specific version of the
-     'ur_robot' macro (ie: 'ur_robot_gazebo') and passing it values for all its
-     required arguments.
-     This file should be considered the Gazebo-specific variant of the file
-     with the same name in the ur_description package. It accepts the same
-     arguments, but instead of configuring everything for a real robot, will
-     generate a Gazebo-compatible URDF with a ros_control hardware_interface
-     attached to it.
-     Only use this top-level xacro if you plan on spawning the robot in Gazebo
-     'by itself', without any gripper or any other geometry attached.
-     If you need to attach an end-effector, camera or need to integrate the
-     robot into a larger workcell and want to spawn that as a single entity in
-     Gazebo, DO NOT EDIT THIS FILE.
-     Instead: create a new top-level xacro, give it a proper name, include the
-     required '.xacro' files, instantiate the models (ie: call the macros) and
-     connect everything by adding the appropriate joints.
-   -->
-   <!-- Import main macro.
-        Note: this imports the Gazebo-wrapper main macro, NOT the regular
-        xacro macro (which is hosted by ur_description).
-   -->
-   <xacro:include filename="$(find ur_gazebo)/urdf/ur_macro.xacro"/>
-   <!-- parameters -->
-   <xacro:arg name="joint_limit_params" default="$(find ur_description)/config/ur3/joint_limits.yaml"/>
-   <xacro:arg name="physical_params" default="$(find ur_description)/config/ur3/physical_parameters.yaml"/>
-   <xacro:arg name="kinematics_params" default="$(find ur_description)/config/ur3/default_kinematics.yaml"/>
-   <xacro:arg name="visual_params" default="$(find ur_description)/config/ur3/visual_parameters.yaml"/>
-   <!-- legal values:
-         - hardware_interface/PositionJointInterface
-         - hardware_interface/VelocityJointInterface
-         - hardware_interface/EffortJointInterface
-   -->
-   <xacro:arg name="transmission_hw_interface" default="hardware_interface/PositionJointInterface"/>
-   <xacro:arg name="safety_limits" default="false"/>
-   <xacro:arg name="safety_pos_margin" default="0.15"/>
-   <xacro:arg name="safety_k_position" default="20"/>
-   <!-- Instantiate the Gazebo robot and pass it all the required arguments. -->
-   <xacro:ur_robot_gazebo
-     prefix=""
-     joint_limits_parameters_file="$(arg joint_limit_params)"
-     kinematics_parameters_file="$(arg kinematics_params)"
-     physical_parameters_file="$(arg physical_params)"
-     visual_parameters_file="$(arg visual_params)"
-     transmission_hw_interface="$(arg transmission_hw_interface)"
-     safety_limits="$(arg safety_limits)"
-     safety_pos_margin="$(arg safety_pos_margin)"
-     safety_k_position="$(arg safety_k_position)"/>
-   <!-- Attach the Gazebo model to Gazebo's world frame -->
-   <link name="world"/>
-   <joint name="world_joint" type="fixed">
-      <parent link="world"/>
-      <child link="base_link"/>
-      <origin xyz="0 0 0" rpy="0 0 0"/>
-   </joint>
+  <!--
+    This is a top-level xacro instantiating the Gazebo-specific version of the
+    'ur_robot' macro (ie: 'ur_robot_gazebo') and passing it values for all its
+    required arguments.
+    This file should be considered the Gazebo-specific variant of the file
+    with the same name in the ur_description package. It accepts the same
+    arguments, but instead of configuring everything for a real robot, will
+    generate a Gazebo-compatible URDF with a ros_control hardware_interface
+    attached to it.
+    Only use this top-level xacro if you plan on spawning the robot in Gazebo
+    'by itself', without any gripper or any other geometry attached.
+    If you need to attach an end-effector, camera or need to integrate the
+    robot into a larger workcell and want to spawn that as a single entity in
+    Gazebo, DO NOT EDIT THIS FILE.
+    Instead: create a new top-level xacro, give it a proper name, include the
+    required '.xacro' files, instantiate the models (ie: call the macros) and
+    connect everything by adding the appropriate joints.
+  -->
+  <!-- Import main macro.
+       Note: this imports the Gazebo-wrapper main macro, NOT the regular
+       xacro macro (which is hosted by ur_description).
+  -->
+  <xacro:include filename="$(find ur_gazebo)/urdf/ur_macro.xacro"/>
+  <!--Declare arguments -->
+  <xacro:arg name="joint_limit_params" default="$(find ur_description)/config/ur3/joint_limits.yaml"/>
+  <xacro:arg name="physical_params" default="$(find ur_description)/config/ur3/physical_parameters.yaml"/>
+  <xacro:arg name="kinematics_params" default="$(find ur_description)/config/ur3/default_kinematics.yaml"/>
+  <xacro:arg name="visual_params" default="$(find ur_description)/config/ur3/visual_parameters.yaml"/>
+  <!-- legal values:
+      - hardware_interface/PositionJointInterface
+      - hardware_interface/VelocityJointInterface
+      - hardware_interface/EffortJointInterface
+  -->
+  <xacro:arg name="transmission_hw_interface" default="hardware_interface/PositionJointInterface"/>
+  <xacro:arg name="safety_limits" default="false"/>
+  <xacro:arg name="safety_pos_margin" default="0.15"/>
+  <xacro:arg name="safety_k_position" default="20"/>
+  <!-- Instantiate the Gazebo robot and pass it all the required arguments. -->
+  <xacro:ur_robot_gazebo
+    prefix=""
+    joint_limits_parameters_file="$(arg joint_limit_params)"
+    kinematics_parameters_file="$(arg kinematics_params)"
+    physical_parameters_file="$(arg physical_params)"
+    visual_parameters_file="$(arg visual_params)"
+    transmission_hw_interface="$(arg transmission_hw_interface)"
+    safety_limits="$(arg safety_limits)"
+    safety_pos_margin="$(arg safety_pos_margin)"
+    safety_k_position="$(arg safety_k_position)"/>
+  <!-- Attach the Gazebo model to Gazebo's world frame -->
+  <link name="world"/>
+  <joint name="world_joint" type="fixed">
+    <parent link="world"/>
+    <child link="base_link"/>
+    <origin xyz="0 0 0" rpy="0 0 0"/>
+  </joint>
 </robot>

File: ur_gazebo/urdf/ur_macro.xacro (robot description, xacro)
@@ -1,23 +1,23 @@
 <?xml version="1.0"?>
 <robot xmlns:xacro="http://wiki.ros.org/xacro">
-<!--
-  Author: Ludovic Delval
-  Contributor: Felix Messmer, Kelsey Hawkins, Jimmy Da Silva, Ajit Krisshna N L, Muhammad Asif Rana
--->
- <!-- Import the xacro macro for the REAL robot (which we'll augment with
-      Gazebo-specific elements in the wrapper macro below).
-      Note: this imports the '_macro.xacro' from ur_description, as that
-      contains the definitions for the real robot.
- -->
- <xacro:include filename="$(find ur_description)/urdf/ur_macro.xacro"/>
- <xacro:macro name="ur_robot_gazebo" params="
-  prefix
-  joint_limits_parameters_file
-  kinematics_parameters_file
-  physical_parameters_file
-  visual_parameters_file
-  transmission_hw_interface:=hardware_interface/PositionJointInterface
-  safety_limits:=false safety_pos_margin:=0.15 safety_k_position:=20"
- >
+  <!--
+    Author: Ludovic Delval
+    Contributor: Felix Messmer, Kelsey Hawkins, Jimmy Da Silva, Ajit Krisshna N L, Muhammad Asif Rana
+  -->
+  <!-- Import the xacro macro for the REAL robot (which we'll augment with
+       Gazebo-specific elements in the wrapper macro below).
+       Note: this imports the '_macro.xacro' from ur_description, as that
+       contains the definitions for the real robot.
+  -->
+  <xacro:include filename="$(find ur_description)/urdf/ur_macro.xacro"/>
+  <xacro:macro name="ur_robot_gazebo" params="
+   prefix
+   joint_limits_parameters_file
+   kinematics_parameters_file
+   physical_parameters_file
+   visual_parameters_file
+   transmission_hw_interface:=hardware_interface/PositionJointInterface
+   safety_limits:=false safety_pos_margin:=0.15 safety_k_position:=20"
+  >
     <!-- Instantiate model for the REAL robot.
          Add additional elements needed by Gazebo as well.

Commit message: Add tool0_controller frame for gazebo simulation
In order to make the simulation more consistent to the ur_robot_driver
(and ur_modern_driver) this adds a tool0_controller frame.
For the driver this corresponds to the tool transformation published by
the robot controller directly. As this doesn't exist for the simulated
robot, this adds the frame using an identity transform from tool0.

File: ur_gazebo/urdf/ur.xacro (robot description, xacro)
@@ -67,3 +67,9 @@
     <origin xyz="0 0 0" rpy="0 0 0"/>
   </joint>
+  <link name="tool0_controller"/>
+  <joint name="tool_controller_fake_joint" type="fixed">
+    <parent link="tool0"/>
+    <child link="tool0_controller"/>
+    <origin xyz="0 0 0" rpy="0 0 0"/>
+  </joint>
 </robot>
