Commit message: description: they're joint limits.
Not joints limits.

File: ur_description/urdf/inc/ur_common.xacro (robot description, xacro)
@@ -24,6 +24,6 @@
           and as such should be considered to be for internal use only.
   -->
-  <xacro:macro name="read_model_data" params="joints_limits_parameters_file kinematics_parameters_file physical_parameters_file visual_parameters_file">
-    <xacro:property name="__limits" value="${joints_limits_parameters_file['limits']}"/>
+  <xacro:macro name="read_model_data" params="joint_limits_parameters_file kinematics_parameters_file physical_parameters_file visual_parameters_file">
+    <xacro:property name="__limits" value="${joint_limits_parameters_file['limits']}"/>
     <xacro:property name="__dh_parameters" value="${physical_parameters_file['dh_parameters']}"/>
     <xacro:property name="__offsets" value="${physical_parameters_file['offsets']}"/>

File: ur_description/urdf/ur.xacro (robot description, xacro)
@@ -4,5 +4,5 @@
    <xacro:include filename="$(find ur_description)/urdf/ur_macro.xacro"/>
    <!-- parameters -->
-   <xacro:arg name="joints_limits_params" default=""/>
+   <xacro:arg name="joint_limit_params" default=""/>
    <xacro:arg name="kinematics_params" default=""/>
    <xacro:arg name="physical_params" default=""/>
@@ -20,5 +20,5 @@
    <xacro:ur_robot
      prefix=""
-     joints_limits_parameters_file="${load_yaml('$(arg joints_limits_params)')}"
+     joint_limits_parameters_file="${load_yaml('$(arg joint_limit_params)')}"
      kinematics_parameters_file="${load_yaml('$(arg kinematics_params)')}"
      physical_parameters_file="${load_yaml('$(arg physical_params)')}"

File: ur_description/urdf/ur_macro.xacro (robot description, xacro)
@@ -46,5 +46,5 @@
   <xacro:macro name="ur_robot" params="
     prefix
-    joints_limits_parameters_file
+    joint_limits_parameters_file
     kinematics_parameters_file
     physical_parameters_file
@@ -57,5 +57,5 @@
     <!-- Load configuration data from the provided .yaml files -->
     <xacro:read_model_data
-      joints_limits_parameters_file="${joints_limits_parameters_file}"
+      joint_limits_parameters_file="${joint_limits_parameters_file}"
       kinematics_parameters_file="${kinematics_parameters_file}"
       physical_parameters_file="${physical_parameters_file}"

Commit message: description: load values from new params.
'ros_control format' uses different names, so use them.

File: ur_description/urdf/inc/ur_common.xacro (robot description, xacro)
@@ -25,5 +25,5 @@
   -->
   <xacro:macro name="read_model_data" params="joint_limits_parameters_file kinematics_parameters_file physical_parameters_file visual_parameters_file">
-    <xacro:property name="__limits" value="${joint_limits_parameters_file['limits']}"/>
+    <xacro:property name="__limits" value="${joint_limits_parameters_file['joint_limits']}"/>
     <xacro:property name="__dh_parameters" value="${physical_parameters_file['dh_parameters']}"/>
     <xacro:property name="__offsets" value="${physical_parameters_file['offsets']}"/>
@@ -32,28 +32,28 @@
     <xacro:property name="__kinematics" value="${kinematics_parameters_file['kinematics']}" />
     <!-- JOINTS LIMIT PARAMETERS -->
-    <xacro:property name="shoulder_pan_lower_limit" value="${__limits['shoulder_pan']['lower']}" scope="parent"/>
-    <xacro:property name="shoulder_pan_upper_limit" value="${__limits['shoulder_pan']['upper']}" scope="parent"/>
-    <xacro:property name="shoulder_pan_velocity_limit" value="${__limits['shoulder_pan']['velocity']}" scope="parent"/>
-    <xacro:property name="shoulder_pan_effort_limit" value="${__limits['shoulder_pan']['effort']}" scope="parent"/>
-    <xacro:property name="shoulder_lift_lower_limit" value="${__limits['shoulder_lift']['lower']}" scope="parent"/>
-    <xacro:property name="shoulder_lift_upper_limit" value="${__limits['shoulder_lift']['upper']}" scope="parent"/>
-    <xacro:property name="shoulder_lift_velocity_limit" value="${__limits['shoulder_lift']['velocity']}" scope="parent"/>
-    <xacro:property name="shoulder_lift_effort_limit" value="${__limits['shoulder_lift']['effort']}" scope="parent"/>
-    <xacro:property name="elbow_joint_lower_limit" value="${__limits['elbow_joint']['lower']}" scope="parent"/>
-    <xacro:property name="elbow_joint_upper_limit" value="${__limits['elbow_joint']['upper']}" scope="parent"/>
-    <xacro:property name="elbow_joint_velocity_limit" value="${__limits['elbow_joint']['velocity']}" scope="parent"/>
-    <xacro:property name="elbow_joint_effort_limit" value="${__limits['elbow_joint']['effort']}" scope="parent"/>
-    <xacro:property name="wrist_1_lower_limit" value="${__limits['wrist_1']['lower']}" scope="parent"/>
-    <xacro:property name="wrist_1_upper_limit" value="${__limits['wrist_1']['upper']}" scope="parent"/>
-    <xacro:property name="wrist_1_velocity_limit" value="${__limits['wrist_1']['velocity']}" scope="parent"/>
-    <xacro:property name="wrist_1_effort_limit" value="${__limits['wrist_1']['effort']}" scope="parent"/>
-    <xacro:property name="wrist_2_lower_limit" value="${__limits['wrist_2']['lower']}" scope="parent"/>
-    <xacro:property name="wrist_2_upper_limit" value="${__limits['wrist_2']['upper']}" scope="parent"/>
-    <xacro:property name="wrist_2_velocity_limit" value="${__limits['wrist_2']['velocity']}" scope="parent"/>
-    <xacro:property name="wrist_2_effort_limit" value="${__limits['wrist_2']['effort']}" scope="parent"/>
-    <xacro:property name="wrist_3_lower_limit" value="${__limits['wrist_3']['lower']}" scope="parent"/>
-    <xacro:property name="wrist_3_upper_limit" value="${__limits['wrist_3']['upper']}" scope="parent"/>
-    <xacro:property name="wrist_3_velocity_limit" value="${__limits['wrist_3']['velocity']}" scope="parent"/>
-    <xacro:property name="wrist_3_effort_limit" value="${__limits['wrist_3']['effort']}" scope="parent"/>
+    <xacro:property name="shoulder_pan_lower_limit" value="${__limits['shoulder_pan']['min_position']}" scope="parent"/>
+    <xacro:property name="shoulder_pan_upper_limit" value="${__limits['shoulder_pan']['max_position']}" scope="parent"/>
+    <xacro:property name="shoulder_pan_velocity_limit" value="${__limits['shoulder_pan']['max_velocity']}" scope="parent"/>
+    <xacro:property name="shoulder_pan_effort_limit" value="${__limits['shoulder_pan']['max_effort']}" scope="parent"/>
+    <xacro:property name="shoulder_lift_lower_limit" value="${__limits['shoulder_lift']['min_position']}" scope="parent"/>
+    <xacro:property name="shoulder_lift_upper_limit" value="${__limits['shoulder_lift']['max_position']}" scope="parent"/>
+    <xacro:property name="shoulder_lift_velocity_limit" value="${__limits['shoulder_lift']['max_velocity']}" scope="parent"/>
+    <xacro:property name="shoulder_lift_effort_limit" value="${__limits['shoulder_lift']['max_effort']}" scope="parent"/>
+    <xacro:property name="elbow_joint_lower_limit" value="${__limits['elbow_joint']['min_position']}" scope="parent"/>
+    <xacro:property name="elbow_joint_upper_limit" value="${__limits['elbow_joint']['max_position']}" scope="parent"/>
+    <xacro:property name="elbow_joint_velocity_limit" value="${__limits['elbow_joint']['max_velocity']}" scope="parent"/>
+    <xacro:property name="elbow_joint_effort_limit" value="${__limits['elbow_joint']['max_effort']}" scope="parent"/>
+    <xacro:property name="wrist_1_lower_limit" value="${__limits['wrist_1']['min_position']}" scope="parent"/>
+    <xacro:property name="wrist_1_upper_limit" value="${__limits['wrist_1']['max_position']}" scope="parent"/>
+    <xacro:property name="wrist_1_velocity_limit" value="${__limits['wrist_1']['max_velocity']}" scope="parent"/>
+    <xacro:property name="wrist_1_effort_limit" value="${__limits['wrist_1']['max_effort']}" scope="parent"/>
+    <xacro:property name="wrist_2_lower_limit" value="${__limits['wrist_2']['min_position']}" scope="parent"/>
+    <xacro:property name="wrist_2_upper_limit" value="${__limits['wrist_2']['max_position']}" scope="parent"/>
+    <xacro:property name="wrist_2_velocity_limit" value="${__limits['wrist_2']['max_velocity']}" scope="parent"/>
+    <xacro:property name="wrist_2_effort_limit" value="${__limits['wrist_2']['max_effort']}" scope="parent"/>
+    <xacro:property name="wrist_3_lower_limit" value="${__limits['wrist_3']['min_position']}" scope="parent"/>
+    <xacro:property name="wrist_3_upper_limit" value="${__limits['wrist_3']['max_position']}" scope="parent"/>
+    <xacro:property name="wrist_3_velocity_limit" value="${__limits['wrist_3']['max_velocity']}" scope="parent"/>
+    <xacro:property name="wrist_3_effort_limit" value="${__limits['wrist_3']['max_effort']}" scope="parent"/>
     <!-- DH PARAMETERS -->
     <xacro:property name="d1" value="${__dh_parameters['d1']}" scope="parent"/>

Commit message: description: delegate loading yaml files to read_model_data(..).
This avoids having to 'remember' to load_yaml(..) the contents of those files in every user of the 'ur_robot' macro, and seems to conform to the idea behind the '*_parameters_file' naming of the parameters (they're paths to files, not yaml strings).

File: ur_description/urdf/inc/ur_common.xacro (robot description, xacro)
@@ -25,10 +25,16 @@
   -->
   <xacro:macro name="read_model_data" params="joint_limits_parameters_file kinematics_parameters_file physical_parameters_file visual_parameters_file">
-    <xacro:property name="__limits" value="${joint_limits_parameters_file['joint_limits']}"/>
-    <xacro:property name="__dh_parameters" value="${physical_parameters_file['dh_parameters']}"/>
-    <xacro:property name="__offsets" value="${physical_parameters_file['offsets']}"/>
-    <xacro:property name="__inertia_parameters" value="${physical_parameters_file['inertia_parameters']}" />
-    <xacro:property name="__mesh_files" value="${visual_parameters_file['mesh_files']}" />
-    <xacro:property name="__kinematics" value="${kinematics_parameters_file['kinematics']}" />
+    <!-- Read .yaml files from disk, load content into properties -->
+    <xacro:property name="__joint_limit_parameters" value="${load_yaml(joint_limits_parameters_file)}"/>
+    <xacro:property name="__kinematics_parameters" value="${load_yaml(kinematics_parameters_file)}"/>
+    <xacro:property name="__physical_parameters" value="${load_yaml(physical_parameters_file)}"/>
+    <xacro:property name="__visual_parameters" value="${load_yaml(visual_parameters_file)}"/>
+    <!-- Extract subsections from yaml dictionaries -->
+    <xacro:property name="__limits" value="${__joint_limit_parameters['joint_limits']}"/>
+    <xacro:property name="__dh_parameters" value="${__physical_parameters['dh_parameters']}"/>
+    <xacro:property name="__offsets" value="${__physical_parameters['offsets']}"/>
+    <xacro:property name="__inertia_parameters" value="${__physical_parameters['inertia_parameters']}" />
+    <xacro:property name="__mesh_files" value="${__visual_parameters['mesh_files']}" />
+    <xacro:property name="__kinematics" value="${__kinematics_parameters['kinematics']}" />
     <!-- JOINTS LIMIT PARAMETERS -->
     <xacro:property name="shoulder_pan_lower_limit" value="${__limits['shoulder_pan']['min_position']}" scope="parent"/>

File: ur_description/urdf/ur.xacro (robot description, xacro)
@@ -20,8 +20,8 @@
    <xacro:ur_robot
      prefix=""
-     joint_limits_parameters_file="${load_yaml('$(arg joint_limit_params)')}"
-     kinematics_parameters_file="${load_yaml('$(arg kinematics_params)')}"
-     physical_parameters_file="${load_yaml('$(arg physical_params)')}"
-     visual_parameters_file="${load_yaml('$(arg visual_params)')}"
+     joint_limits_parameters_file="$(arg joint_limit_params)"
+     kinematics_parameters_file="$(arg kinematics_params)"
+     physical_parameters_file="$(arg physical_params)"
+     visual_parameters_file="$(arg visual_params)"
      transmission_hw_interface="$(arg transmission_hw_interface)"
      safety_limits="$(arg safety_limits)"

Commit message: Fix UR3 mesh positing.

File: ur_description/urdf/inc/ur_common.xacro (robot description, xacro)
@@ -193,4 +193,10 @@
     <xacro:property name="wrist_3_collision_mesh" value="${wrist_3_mesh['collision']['mesh']}" scope="parent"/>
     <xacro:property name="wrist_3_visual_offset" value="${wrist_3_mesh['visual_offset']}" scope="parent"/>
+    <xacro:if value="${'visual_offset_xyz' in wrist_3_mesh}">
+      <xacro:property name="wrist_3_visual_offset_xyz" value="${wrist_3_mesh['visual_offset_xyz']}" scope="parent"/>
+    </xacro:if>
+    <xacro:unless value="${'visual_offset_xyz' in wrist_3_mesh}">
+      <xacro:property name="wrist_3_visual_offset_xyz" value='' scope="parent"/>
+    </xacro:unless>
   </xacro:macro>
 </robot>

File: ur_description/urdf/inc/ur_macro.xacro (robot description, xacro)
@@ -187,6 +187,10 @@
     </link>
     <link name="${prefix}wrist_3_link">
-      <visual>
-        <origin xyz="0 0 ${wrist_3_visual_offset}" rpy="${pi/2} 0 0"/>
+      <xacro:property name="mesh_offset" value="${wrist_3_visual_offset_xyz}" scope="parent"/>
+      <xacro:if value="${wrist_3_visual_offset_xyz == ''}">
+        <xacro:property name="mesh_offset" value="0 0 ${wrist_3_visual_offset}" scope="parent"/>
+      </xacro:if>
+      <visual>
+        <origin xyz="${mesh_offset}" rpy="${pi/2} 0 0"/>
         <geometry>
           <mesh filename="${wrist_3_visual_mesh}"/>
@@ -197,5 +201,5 @@
       </visual>
       <collision>
-        <origin xyz="0 0 ${wrist_3_visual_offset}" rpy="${pi/2} 0 0"/>
+        <origin xyz="${mesh_offset}" rpy="${pi/2} 0 0"/>
         <geometry>
           <mesh filename="${wrist_3_collision_mesh}"/>
