Commit message: Replace symlinks with copies of files
For two reasons:
 - windows compatibility
 - corrrect naming of models

File: ur_description/urdf/inc/ur12e_macro.xacro (robot description, xacro)
@@ -1 +1,43 @@
-ur10e_macro.xacro
+<?xml version="1.0"?>
+<robot xmlns:xacro="http://wiki.ros.org/xacro">
+  <!--
+    Convenience wrapper for the 'ur_robot' macro which provides default values
+    for the various "parameters files" parameters for a ur12e.
+    This file can be used when composing a more complex scene with one or more
+    ur12e robots.
+    While the generic 'ur_robot' macro could also be used, it would require
+    the user to provide values for all parameters, as that macro does not set
+    any model-specific defaults (not even for the generic parameters, such as
+    the visual and physical parameters and joint limits).
+    Refer to the main 'ur_macro.xacro' in this package for information about
+    use, contributors and limitations.
+    NOTE: users will most likely want to override *at least* the
+          'kinematics_parameters_file' parameter. Otherwise, a default kinematic
+          model will be used, which will almost certainly not correspond to any
+          real robot.
+  -->
+  <xacro:macro name="ur12e_robot" params="
+   prefix
+   joint_limits_parameters_file:='$(find ur_description)/config/ur12e/joint_limits.yaml'
+   kinematics_parameters_file:='$(find ur_description)/config/ur12e/default_kinematics.yaml'
+   physical_parameters_file:='$(find ur_description)/config/ur12e/physical_parameters.yaml'
+   visual_parameters_file:='$(find ur_description)/config/ur12e/visual_parameters.yaml'
+   transmission_hw_interface:=hardware_interface/PositionJointInterface
+   safety_limits:=false
+   safety_pos_margin:=0.15
+   safety_k_position:=20"
+  >
+    <xacro:include filename="$(find ur_description)/urdf/inc/ur_macro.xacro"/>
+    <xacro:ur_robot
+      prefix="${prefix}"
+      joint_limits_parameters_file="${joint_limits_parameters_file}"
+      kinematics_parameters_file="${kinematics_parameters_file}"
+      physical_parameters_file="${physical_parameters_file}"
+      visual_parameters_file="${visual_parameters_file}"
+      transmission_hw_interface="${transmission_hw_interface}"
+      safety_limits="${safety_limits}"
+      safety_pos_margin="${safety_pos_margin}"
+      safety_k_position="${safety_k_position}"
+    />
+  </xacro:macro>
+</robot>

File: ur_description/urdf/inc/ur7e_macro.xacro (robot description, xacro)
@@ -1 +1,43 @@
-ur5e_macro.xacro
+<?xml version="1.0"?>
+<robot xmlns:xacro="http://wiki.ros.org/xacro">
+  <!--
+    Convenience wrapper for the 'ur_robot' macro which provides default values
+    for the various "parameters files" parameters for a ur7e.
+    This file can be used when composing a more complex scene with one or more
+    ur7e robots.
+    While the generic 'ur_robot' macro could also be used, it would require
+    the user to provide values for all parameters, as that macro does not set
+    any model-specific defaults (not even for the generic parameters, such as
+    the visual and physical parameters and joint limits).
+    Refer to the main 'ur_macro.xacro' in this package for information about
+    use, contributors and limitations.
+    NOTE: users will most likely want to override *at least* the
+          'kinematics_parameters_file' parameter. Otherwise, a default kinematic
+          model will be used, which will almost certainly not correspond to any
+          real robot.
+  -->
+  <xacro:macro name="ur7e_robot" params="
+   prefix
+   joint_limits_parameters_file:='$(find ur_description)/config/ur7e/joint_limits.yaml'
+   kinematics_parameters_file:='$(find ur_description)/config/ur7e/default_kinematics.yaml'
+   physical_parameters_file:='$(find ur_description)/config/ur7e/physical_parameters.yaml'
+   visual_parameters_file:='$(find ur_description)/config/ur7e/visual_parameters.yaml'
+   transmission_hw_interface:=hardware_interface/PositionJointInterface
+   safety_limits:=false
+   safety_pos_margin:=0.15
+   safety_k_position:=20"
+  >
+    <xacro:include filename="$(find ur_description)/urdf/inc/ur_macro.xacro"/>
+    <xacro:ur_robot
+      prefix="${prefix}"
+      joint_limits_parameters_file="${joint_limits_parameters_file}"
+      kinematics_parameters_file="${kinematics_parameters_file}"
+      physical_parameters_file="${physical_parameters_file}"
+      visual_parameters_file="${visual_parameters_file}"
+      transmission_hw_interface="${transmission_hw_interface}"
+      safety_limits="${safety_limits}"
+      safety_pos_margin="${safety_pos_margin}"
+      safety_k_position="${safety_k_position}"
+    />
+  </xacro:macro>
+</robot>

File: ur_description/urdf/ur12e.xacro (robot description, xacro)
@@ -1 +1,18 @@
-ur10e.xacro
+<?xml version="1.0"?>
+<robot xmlns:xacro="http://wiki.ros.org/xacro" name="ur12e_robot">
+  <!--
+    This is a convenience top-level xacro which loads the macro for the ur12e
+    which defines the default values for the various "parameters files"
+    parameters for a ur12e.
+    This file is only useful when loading a stand-alone, completely isolated
+    robot with only default values for all parameters such as the kinematics,
+    visual and physical parameters and joint limits.
+    This file is not intended to be integrated into a larger scene or other
+    composite xacro.
+    Instead, xacro:include 'inc/ur12e_macro.xacro' and override the defaults
+    for the arguments to that macro.
+    Refer to 'inc/ur_macro.xacro' for more information.
+  -->
+  <xacro:include filename="$(find ur_description)/urdf/inc/ur12e_macro.xacro"/>
+  <xacro:ur12e_robot prefix="" />
+</robot>

File: ur_description/urdf/ur7e.xacro (robot description, xacro)
@@ -1 +1,18 @@
-ur5e.xacro
+<?xml version="1.0"?>
+<robot xmlns:xacro="http://wiki.ros.org/xacro" name="ur7e_robot">
+  <!--
+    This is a convenience top-level xacro which loads the macro for the ur7e
+    which defines the default values for the various "parameters files"
+    parameters for a ur7e.
+    This file is only useful when loading a stand-alone, completely isolated
+    robot with only default values for all parameters such as the kinematics,
+    visual and physical parameters and joint limits.
+    This file is not intended to be integrated into a larger scene or other
+    composite xacro.
+    Instead, xacro:include 'inc/ur7e_macro.xacro' and override the defaults
+    for the arguments to that macro.
+    Refer to 'inc/ur_macro.xacro' for more information.
+  -->
+  <xacro:include filename="$(find ur_description)/urdf/inc/ur7e_macro.xacro"/>
+  <xacro:ur7e_robot prefix="" />
+</robot>
